File: hubby.kicad_pcb (KiCad board)
At the start: 4 copper layers, 77 x 100 mm, 141 parts, among them IC1 FE2.1, J1 USB1, J13 USB2, J14 USB2, J16 JTAG_OUT, J19 STM_PROG_ENA, J2 USB2, J20 STM_EXT_IO, J21 Conn_01x08, J3 Barrel_Jack_Switch, J4 Conn_01x04, J5 Screw_Terminal_01x10, J6 Conn_02x06_Odd_Even, J7 UART_OUT, P1 USB_C_Plug_USB2.0, Q1 AO3401A, Q2 AO3401A, Q3 AO3401A, SW1 SW_Push, SW2 RotaryEncoder_Switch, SW3 RotaryEncoder_Switch, U1 USBLC6-2SC6, U10 TPS565208, U11 24LC00, U12 TPS565208, U13 AP1117-18, U14 AP1117-33, U15 USBLC6-2SC6, U16 USBLC6-2SC6, U17 USBLC6-2SC6, U18 USBLC6-2SC6, U19 INA181, U2 STM32F103RBTx, U20 24LC00, U21 SN74LVC2T45YZP, U22 AP1117-33, U3 INA181, U4 INA181, U5 INA181, U6 INA181, U7 FT2232HL, U8 INA181, U9 INA181, X1 ECS-2520MV-xxx-xx, Y1 6MHZ 2520, Y2 6MHZ 2520

Commit message: commiting before swapping MCUs
Parts:
- removed J19: STM_PROG_ENA, Connector_PinHeader_2.54mm:PinHeader_2x04_P2.54mm_Vertical
- removed P1: USB_C_Plug_USB2.0, Connector_USB:USB_C_Receptacle_GCT_USB4085
- removed Q1: AO3401A, Package_TO_SOT_SMD:SOT-23
- removed R6: 100k, Resistor_SMD:R_0603_1608Metric_Pad0.98x0.95mm_HandSolder
- added C47: 10u, Capacitor_SMD:C_0805_2012Metric, F.Cu at (166.6, 59.5)
- added C48: 100n, Capacitor_SMD:C_0402_1005Metric, F.Cu at (170.0, 54.2)
- added C49: 100n, Capacitor_SMD:C_0402_1005Metric, F.Cu at (169.0, 54.2)
- added C50: 100n, Capacitor_SMD:C_0402_1005Metric, F.Cu at (164.5, 55.0)
- added C51: 47uF, Capacitor_THT:CP_Radial_D5.0mm_P2.50mm, F.Cu at (161.0, 65.3)
- added C52: 100n, Capacitor_SMD:C_0402_1005Metric, F.Cu at (169.0, 90.7)
- added C53: 2.2u, Capacitor_SMD:C_0805_2012Metric, F.Cu at (182.2, 89.8)
- added C54: 10u, Capacitor_SMD:C_0805_2012Metric, F.Cu at (172.5, 93.8)
- added C55: 10u, Capacitor_SMD:C_0805_2012Metric, F.Cu at (170.5, 93.8)
- added C56: 47u, Capacitor_SMD:C_0805_2012Metric, F.Cu at (166.8, 97.0)
- added C57: 100n, Capacitor_SMD:C_0402_1005Metric, F.Cu at (157.2, 79.9)
- added C58: 10u, Capacitor_SMD:C_0805_2012Metric, F.Cu at (123.4, 104.9)
- added C59: SUPERCAP, Capacitor_THT:CP_Radial_D5.0mm_P2.50mm, F.Cu at (118.9, 96.0)
- added C60: 100n, Capacitor_SMD:C_0402_1005Metric, F.Cu at (135.5, 64.2)
- added C61: 100n, Capacitor_SMD:C_0402_1005Metric, F.Cu at (97.3, 45.9)
- added C62: 10u, Capacitor_SMD:C_0805_2012Metric, F.Cu at (142.3, 65.1)
- added C63: 10u, Capacitor_SMD:C_0805_2012Metric, F.Cu at (135.7, 74.2)
- added C64: 10u, Capacitor_SMD:C_0805_2012Metric, F.Cu at (135.7, 70.9)
- added C65: 100n, Capacitor_SMD:C_0402_1005Metric, F.Cu at (151.1, 67.1)
- added C66: 100n, Capacitor_SMD:C_0402_1005Metric, F.Cu at (153.5, 75.9)
- added C67: 100n, Capacitor_SMD:C_0402_1005Metric, F.Cu at (138.5, 75.2)
- added C68: 100n, Capacitor_SMD:C_0402_1005Metric, F.Cu at (128.0, 51.7)
- added C69: 100n, Capacitor_SMD:C_0402_1005Metric, F.Cu at (119.4, 59.0)
- added C70: 100n, Capacitor_SMD:C_0402_1005Metric, F.Cu at (124.6, 64.2)
- added C71: 100n, Capacitor_SMD:C_0402_1005Metric, F.Cu at (145.2, 80.8)
- added C72: 100n, Capacitor_SMD:C_0402_1005Metric, F.Cu at (148.6, 80.8)
- added C73: 100n, Capacitor_SMD:C_0402_1005Metric, F.Cu at (146.5, 65.8)
- added C74: 10u, Capacitor_SMD:C_0805_2012Metric, F.Cu at (120.3, 54.0)
- added C75: 100n, Capacitor_SMD:C_0402_1005Metric, F.Cu at (119.3, 57.2)
- added C76: 100n, Capacitor_SMD:C_0402_1005Metric, F.Cu at (131.8, 59.4)
- added C77: 100n, Capacitor_SMD:C_0402_1005Metric, F.Cu at (149.4, 101.2)
- added C78: 10u, Capacitor_SMD:C_0805_2012Metric, F.Cu at (130.7, 63.8)
- added C79: 100n, Capacitor_SMD:C_0402_1005Metric, F.Cu at (131.6, 86.7)
- added C80: 100n, Capacitor_SMD:C_0402_1005Metric, F.Cu at (131.8, 79.8)
- added C81: 100n, Capacitor_SMD:C_0402_1005Metric, F.Cu at (118.5, 88.9)
- added C82: 100n, Capacitor_SMD:C_0402_1005Metric, F.Cu at (119.2, 77.8)
- added C83: 100n, Capacitor_SMD:C_0402_1005Metric, F.Cu at (126.4, 91.1)
- added C84: 10u, Capacitor_SMD:C_0805_2012Metric, F.Cu at (163.0, 55.0)
- added C85: 100n, Capacitor_SMD:C_0402_1005Metric, F.Cu at (154.0, 72.8)
- added C86: 10u, Capacitor_SMD:C_0805_2012Metric, F.Cu at (167.0, 100.0)
- added C87: 10u, Capacitor_SMD:C_0805_2012Metric, F.Cu at (169.5, 100.0)
- added C88: 10u/16V, Capacitor_SMD:C_0805_2012Metric, F.Cu at (162.0, 100.0)
- added C89: 10u, Capacitor_SMD:C_0805_2012Metric, F.Cu at (164.5, 100.0)
- added C91: 100n, Capacitor_SMD:C_0402_1005Metric, F.Cu at (159.2, 95.0)
- added D3: D_Schottky, Diode_SMD:D_SMA, F.Cu at (160.2, 57.2)
- added D4: D_Schottky, Diode_SMD:D_SMA, F.Cu at (156.3, 59.7)
- added D5: D_Schottky, Diode_SMD:D_SMA, F.Cu at (177.5, 95.5)
- added J8: USB_C_Receptacle_USB2.0, Connector_USB:USB_C_Receptacle_GCT_USB4085, F.Cu at (110.5, 42.0)
- added J9: STM_PROG_ENA, Connector_PinHeader_2.54mm:PinHeader_2x04_P2.54mm_Vertical, F.Cu at (146.8, 90.2)
- added JP4: VPROG_SET_SRC, Connector_PinHeader_2.54mm:PinHeader_1x03_P2.54mm_Vertical, F.Cu at (158.4, 88.4)
- added L5: L_Iron, Inductor_SMD:L_1206_3216Metric_Pad1.42x1.75mm_HandSolder, F.Cu at (171.0, 97.0)
- added L6: L, Inductor_SMD:L_1206_3216Metric_Pad1.22x1.90mm_HandSolder, F.Cu at (130.0, 91.9)
- added R38: 100k, Resistor_SMD:R_0603_1608Metric_Pad0.98x0.95mm_HandSolder, F.Cu at (169.0, 88.0)
- added R39: 2k, Resistor_SMD:R_0603_1608Metric_Pad0.98x0.95mm_HandSolder, F.Cu at (165.2, 94.0)
- added R40: 3k, Resistor_SMD:R_0603_1608Metric_Pad0.98x0.95mm_HandSolder, F.Cu at (168.2, 94.0)
- added R41: 2k, Resistor_SMD:R_0603_1608Metric_Pad0.98x0.95mm_HandSolder, F.Cu at (166.8, 94.0)
- added R42: 100k, Resistor_SMD:R_0603_1608Metric_Pad0.98x0.95mm_HandSolder, F.Cu at (152.5, 53.2)
- added R43: 100k, Resistor_SMD:R_0603_1608Metric_Pad0.98x0.95mm_HandSolder, F.Cu at (156.0, 53.2)
- added R44: 100k, Resistor_SMD:R_0603_1608Metric_Pad0.98x0.95mm_HandSolder, F.Cu at (171.9, 74.9)
- added R45: 100k, Resistor_SMD:R_0603_1608Metric_Pad0.98x0.95mm_HandSolder, F.Cu at (175.7, 74.9)
- added R46: 100k, Resistor_SMD:R_0603_1608Metric_Pad0.98x0.95mm_HandSolder, F.Cu at (162.2, 75.3)
- added R47: 100k, Resistor_SMD:R_0603_1608Metric_Pad0.98x0.95mm_HandSolder, F.Cu at (165.8, 75.3)
- added R48: 3k, Resistor_SMD:R_0603_1608Metric_Pad0.98x0.95mm_HandSolder, F.Cu at (155.9, 82.3)
- added R49: 100k, Resistor_SMD:R_0603_1608Metric_Pad0.98x0.95mm_HandSolder, F.Cu at (162.8, 96.8)
- added R50: 100k, Resistor_SMD:R_0603_1608Metric_Pad0.98x0.95mm_HandSolder, F.Cu at (159.6, 96.7)
- added R51: 100k, Resistor_SMD:R_0603_1608Metric_Pad0.98x0.95mm_HandSolder, F.Cu at (139.4, 59.3)
- added R52: 100k, Resistor_SMD:R_0603_1608Metric_Pad0.98x0.95mm_HandSolder, F.Cu at (139.3, 60.8)
- added R53: 2k2, Resistor_SMD:R_0603_1608Metric_Pad0.98x0.95mm_HandSolder, F.Cu at (137.3, 57.2)
- added R54: 100k, Resistor_SMD:R_0603_1608Metric_Pad0.98x0.95mm_HandSolder, F.Cu at (139.3, 62.3)
- added R55: 470, Resistor_SMD:R_0603_1608Metric_Pad0.98x0.95mm_HandSolder, F.Cu at (113.9, 43.3)
- added REF**: ESP32-WROOM-32, RF_Module:ESP32-WROOM-32, F.Cu at (105.5, 73.5)
- added RV1: 10k, Potentiometer_THT:Potentiometer_Runtron_RM-065_Vertical, F.Cu at (166.8, 86.2)
- added TP1: RTC_OUT, TestPoint:TestPoint_Pad_D1.0mm, F.Cu at (116.4, 90.3)
- added TP2: GENERIC_PWM, TestPoint:TestPoint_Pad_D1.0mm, F.Cu at (116.9, 86.7)
- added TP3: STM_CLK_OUT, TestPoint:TestPoint_Pad_D1.0mm, F.Cu at (123.5, 76.3)
- added U23: SN74LVC2T45DCUR, Package_SO:VSSOP-8_2.4x2.1mm_P0.5mm, F.Cu at (150.6, 99.4)
- C1, C10, C11, C12, C13, C14, C17, C18, C2, C41, C45, C46, C5, C6, C7, C8: footprint Capacitor_SMD:C_1206_3216Metric_Pad1.33x1.80mm_HandSolder -> Capacitor_SMD:C_0805_2012Metric
- C15, C9: value C -> 10u; footprint Capacitor_SMD:C_1206_3216Metric_Pad1.33x1.80mm_HandSolder -> Capacitor_SMD:C_0805_2012Metric
- C16, C19, C20, C21, C22, C23, C24, C25, C26, C28, C29, C30, C35, C36, C37, C38, C39, C4, C40, C43, C44: footprint Capacitor_SMD:C_0603_1608Metric_Pad1.08x0.95mm_HandSolder -> Capacitor_SMD:C_0402_1005Metric
- C27: value 100n -> 10u; footprint Capacitor_SMD:C_0603_1608Metric_Pad1.08x0.95mm_HandSolder -> Capacitor_SMD:C_0805_2012Metric
- C3: footprint Capacitor_SMD:C_1206_3216Metric_Pad1.33x1.80mm_HandSolder -> Capacitor_THT:CP_Radial_D5.0mm_P2.50mm
- C31, C32, C33, C34: value 10u -> 20p; footprint Capacitor_SMD:C_1206_3216Metric_Pad1.33x1.80mm_HandSolder -> Capacitor_SMD:C_0402_1005Metric
- C42: footprint Capacitor_THT:C_Radial_D10.0mm_H12.5mm_P5.00mm -> Capacitor_THT:CP_Radial_D5.0mm_P2.50mm
- J4: footprint Connector_PinSocket_2.54mm:PinSocket_1x04_P2.54mm_Vertical -> Connector_PinHeader_2.00mm:PinHeader_1x04_P2.00mm_Vertical
- J5: value Screw_Terminal_01x10 -> Screw_Terminal_01x12; footprint TerminalBlock_Phoenix:TerminalBlock_Phoenix_MKDS-1,5-10-5.08_1x10_P5.08mm_Horizontal -> TerminalBlock_Phoenix:TerminalBlock_Phoenix_PT-1,5-12-5.0-H_1x12_P5.00mm_Horizontal
- L1: value L -> 2.2u; footprint Inductor_SMD:L_1206_3216Metric_Pad1.22x1.90mm_HandSolder -> Inductor_SMD:L_Vishay_IHLP-4040
- L2: value L -> L_Iron_Coupled; footprint Inductor_SMD:L_1206_3216Metric_Pad1.22x1.90mm_HandSolder -> Inductor_SMD:L_Wuerth_WE-DD-Typ-M-Typ-S
- R10: value 60k -> 100k
- R11, R12: value 40k -> 100k
- R27: value 100k -> 12k
- R9: value 100k -> 470
- U10: value TPS565208 -> MIC2405x; footprint Package_TO_SOT_SMD:SOT-23-6 -> Critbit_lib:QFN-28-3EP_5x6mm_MIC2045x
- U12: value TPS565208 -> ADP1612; footprint Package_TO_SOT_SMD:SOT-23-6 -> Package_SO:MSOP-8_3x3mm_P0.65mm
- U13: value AP1117-18 -> MCP6001U; footprint Package_TO_SOT_SMD:SOT-223-3_TabPin2 -> Package_TO_SOT_SMD:SOT-23-5
- U14: value AP1117-33 -> AZ1117-ADJ
- U20: value 24LC00 -> AZ1117-ADJ; footprint Package_SO:SOIC-8_3.9x4.9mm_P1.27mm -> Package_TO_SOT_SMD:SOT-223-3_TabPin2
- U21: value SN74LVC2T45YZP -> AZ1117-ADJ; footprint Package_BGA:Texas_DSBGA-8_0.9x1.9mm_Layout2x4_P0.5mm -> Package_TO_SOT_SMD:SOT-223-3_TabPin2
- U22: value AP1117-33 -> 93LCxxAxxOT; footprint Package_TO_SOT_SMD:SOT-223-3_TabPin2 -> Package_TO_SOT_SMD:SOT-23-6
- Y2: value 6MHZ 2520 -> 12MHZ 2520
- moved R13 188.9 mm to (102.6, 94.8)
- moved Q3 173.0 mm to (96.6, 98.9), turned to -90 degrees
- moved R10 161.6 mm to (127.3, 74.5), turned to 90 degrees
- moved U11 161.3 mm to (97.4, 49.4)
- moved U1 160.3 mm to (107.5, 45.5), turned to -90 degrees
- moved R14 159.1 mm to (99.2, 98.4), turned to 90 degrees
- moved Y1 155.8 mm to (121.0, 51.3), turned to 180 degrees
- moved U16 155.7 mm to (125.8, 50.9), turned to 90 degrees
- moved R30 150.3 mm to (118.7, 55.9)
- moved R15 150.2 mm to (102.5, 101.0)
- moved F1 149.5 mm to (97.2, 95.4), turned to 180 degrees
- moved C29 148.6 mm to (124.0, 99.8), turned to 90 degrees
- moved U15 146.5 mm to (113.0, 98.3), turned to -90 degrees
- moved R9 146.3 mm to (111.3, 44.2)
- moved C30 142.9 mm to (119.3, 92.0), turned to -90 degrees
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Connections:
- C15 pad 1: +VSW -> Net-(C15-Pad1)
- C16 pad 1: +3V3 -> VDDA
- C17 pad 1: /USBx_5V -> +5V
- C18 pad 1: /USBx_5V -> +5V
- C2 pad 1: /USBx_5V -> +5V
- C24 pad 1: Net-(C24-Pad1) -> VDD
- C27 pad 1: VDD -> Net-(C27-Pad1)
- C28 pad 1: +1V8 -> Net-(C28-Pad1)
- C36 pad 1: +3V3 -> VDD
- C37 pad 1: Net-(C37-Pad1) -> /ENC2_BUT
- C38 pad 1: Net-(C38-Pad1) -> /ENC1_A
- C39 pad 1: Net-(C39-Pad1) -> /ENC1_B
- C4 pad 1: +3V3 -> VDDA
- C40 pad 1: Net-(C40-Pad1) -> /ENC1_BUT
- C43 pad 1: Net-(C43-Pad1) -> /ENC2_A
- C44 pad 1: Net-(C44-Pad1) -> /ENC2_B
- C45 pad 1: +5V -> Net-(C45-Pad1)
- C9 pad 1: Net-(C9-Pad1) -> +VDC
- D1 pad 2: Net-(D1-Pad2) -> VDD
- D2 pad 2: Net-(D2-Pad2) -> VDD
- IC1 pad 15: VDD -> Net-(C27-Pad1)
- IC1 pad 20: VDD -> Net-(C27-Pad1)
- IC1 pad 21: unconnected-(IC1-Pad21) -> Net-(C28-Pad1)
- IC1 pad 25: unconnected-(IC1-Pad25) -> Net-(C28-Pad1)
- IC1 pad 26: VDD -> Net-(C27-Pad1)
- IC1 pad 28: +1V8 -> Net-(C28-Pad1)
- IC1 pad 31: VDD -> Net-(C27-Pad1)
- IC1 pad 36: VDD -> Net-(C27-Pad1)
- IC1 pad 42: VDD -> Net-(C27-Pad1)
- IC1 pad 6: +1V8 -> Net-(C28-Pad1)
- IC1 pad 9: unconnected-(IC1-Pad9) -> Net-(C27-Pad1)
- J13 pad 1: /USBx_5V -> +5V
- J14 pad 1: /USBx_5V -> +5V
- J2 pad 1: /USBx_5V -> +5V
- J20 pad 12: unconnected-(J20-Pad12) -> GND
- J20 pad 2: unconnected-(J20-Pad2) -> GND
- J20 pad 4: unconnected-(J20-Pad4) -> GND
- J5 pad 1: /EXT_PS_OUT -> GND
- J5 pad 10: GND -> /EXT_PS_OUT
- J5 pad 2: GND -> /VPROG_OUT
- J5 pad 3: /5V_OUT -> GND
- J5 pad 4: GND -> /1V8_OUT
- J5 pad 5: /3V3_OUT -> GND
- J5 pad 6: GND -> /3V3_OUT
- J5 pad 7: /1V8_OUT -> GND
- J5 pad 8: GND -> /5V_OUT
- J5 pad 9: /VPROG_OUT -> GND
- J6 pad 1: /EXT_PS_OUT -> /VPROG_OUT
- J6 pad 11: /VPROG_OUT -> /EXT_PS_OUT
- J6 pad 12: Net-(C42-Pad1) -> GND
- J6 pad 2: GND -> Net-(C42-Pad1)
- J6 pad 3: /5V_OUT -> /VPROG_OUT
- J6 pad 5: /3V3_OUT -> /1V8_OUT
- J6 pad 7: /1V8_OUT -> /3V3_OUT
- J6 pad 9: /VPROG_OUT -> /5V_OUT
- JP2 pad 1: Net-(JP2-Pad1) -> Net-(J9-Pad2)
- JP3 pad 3: Net-(JP3-Pad3) -> Net-(J9-Pad6)
- L1 pad 1: Net-(L1-Pad1) -> Net-(C48-Pad2)
- L1 pad 2: Net-(C9-Pad1) -> Net-(C50-Pad1)
- L2 pad 1: Net-(L2-Pad1) -> GND
- L2 pad 2: +VSW -> Net-(C53-Pad1)
- Q2 pad 3: Net-(C9-Pad1) -> Net-(C50-Pad1)
- Q3 pad 1: Net-(Q3-Pad1) -> /USB1_PWR_ENA
- Q3 pad 3: /USBx_5V -> /USB1_5V
- R1 pad 1: Net-(D1-Pad2) -> Net-(U7-Pad55)
- R1 pad 2: VDD -> Net-(D1-Pad1)
- R10 pad 1: Net-(R10-Pad1) -> /EXT_PS_CONV_PG
- R10 pad 2: +VSW -> VDD
- R11 pad 1: GND -> /EXT_PS_CONV_EN
- R11 pad 2: Net-(R10-Pad1) -> +VDC
- R12 pad 1: /VPROG_PWM -> Net-(C50-Pad2)
- R12 pad 2: Net-(R10-Pad1) -> Net-(C49-Pad2)
- R13 pad 1: Net-(Q3-Pad1) -> /USB1_PWR_ENA
- R14 pad 1: Net-(Q3-Pad1) -> /USB1_PWR_ENA
- R15 pad 1: Net-(Q1-Pad3) -> /USB1_5V
- R17 pad 1: Net-(C9-Pad1) -> Net-(C50-Pad1)
- R18 pad 2: +5V -> Net-(C50-Pad1)
- R20 pad 1: /VPROG_VLT -> Net-(C50-Pad2)
- R20 pad 2: +VSW -> Net-(C50-Pad1)
- R21 pad 2: /VPROG_VLT -> Net-(C50-Pad2)
- R3 pad 1: Net-(D2-Pad2) -> Net-(U7-Pad54)
- R3 pad 2: VDD -> Net-(D2-Pad1)
- R31 pad 1: Net-(C37-Pad1) -> /ENC2_BUT
- R32 pad 1: Net-(C38-Pad1) -> /ENC1_A
- R33 pad 1: Net-(C39-Pad1) -> /ENC1_B
- R34 pad 1: Net-(C40-Pad1) -> /ENC1_BUT
- R36 pad 1: Net-(C43-Pad1) -> /ENC2_A
- R37 pad 1: Net-(C44-Pad1) -> /ENC2_B
- R7 pad 2: +3V3 -> VBUS
- R9 pad 1: /EXT_PS_DET -> Net-(J8-PadA5)
- R9 pad 2: +5V -> GND
- RN1 pad 7: Net-(JP3-Pad3) -> Net-(J9-Pad6)
- RN2 pad 2: /TARG_TDO_SWDIO -> /TARG_TDI
- RN2 pad 3: /TARG_TDI -> /TARG_TDO_SWDIO
- RN2 pad 6: /TDI -> Net-(J9-Pad2)
- RN2 pad 7: Net-(JP2-Pad1) -> /TDI
- SW2 pad A: Net-(C38-Pad1) -> /ENC1_A
- SW2 pad B: Net-(C39-Pad1) -> /ENC1_B
- SW2 pad S1: Net-(C40-Pad1) -> /ENC1_BUT
- SW3 pad A: Net-(C43-Pad1) -> /ENC2_A
- SW3 pad B: Net-(C44-Pad1) -> /ENC2_B
- SW3 pad S1: Net-(C37-Pad1) -> /ENC2_BUT
- U1 pad 4: /USBIN_P -> /USBIN_M
- U1 pad 6: /USBIN_M -> /USBIN_P
- U10 pad 1: GND -> Net-(C15-Pad1)
- U10 pad 2: Net-(L1-Pad1) -> GND
- U10 pad 3: +VDC -> (no net)
- U10 pad 4: unconnected-(U10-Pad4) -> Net-(C48-Pad2)
- U10 pad 5: unconnected-(U10-Pad5) -> GND
- U10 pad 6: unconnected-(U10-Pad6) -> GND
- U12 pad 1: GND -> Net-(C52-Pad1)
- U12 pad 2: Net-(L2-Pad1) -> Net-(R39-Pad2)
- U12 pad 3: +5V -> /VPROG_EN
- U12 pad 4: Net-(R10-Pad1) -> GND
- U12 pad 5: unconnected-(U12-Pad5) -> Net-(C53-Pad2)
- U12 pad 6: unconnected-(U12-Pad6) -> +5V
- U13 pad 1: GND -> Net-(JP4-Pad2)
- U13 pad 2: +1V8 -> GND
- U13 pad 3: +5V -> Net-(R39-Pad1)
- U14 pad 1: GND -> Net-(R42-Pad1)
- U14 pad 2: +3V3 -> VDD
- U14 pad 3: +5V -> Net-(C45-Pad1)
- U15 pad 5: +5V -> Net-(C1-Pad1)
- U2 pad 2: unconnected-(U2-Pad2) -> /RTC_OUT
- U2 pad 3: unconnected-(U2-Pad3) -> /FE21_RST
- U2 pad 33: unconnected-(U2-Pad33) -> /EXT_PS_DET
- U2 pad 34: unconnected-(U2-Pad34) -> /VPROG_EN
- U2 pad 35: unconnected-(U2-Pad35) -> /EXT_PS_CONV_EN
- U2 pad 36: unconnected-(U2-Pad36) -> /EXT_PS_CONV_PG
- U2 pad 37: unconnected-(U2-Pad37) -> /ENC2_A
- U2 pad 38: unconnected-(U2-Pad38) -> /ENC2_B
- U2 pad 39: unconnected-(U2-Pad39) -> /ENC1_BUT
- U2 pad 4: unconnected-(U2-Pad4) -> /USB1_PWR_ENA
- U2 pad 40: unconnected-(U2-Pad40) -> /ENC2_BUT
- U2 pad 46: unconnected-(U2-Pad46) -> /STM_SWDIO
- U2 pad 49: unconnected-(U2-Pad49) -> /STM_SWCLK
- U2 pad 51: unconnected-(U2-Pad51) -> /FT2232_RST
- U2 pad 52: /LCD_BL -> /LCD_DC
- U2 pad 53: /LCD_DC -> /LCD_RST
- U2 pad 54: /LCD_RST -> /LCD_BL
- U2 pad 61: /STM_BUT1 -> /GENERIC_PWM
- U2 pad 62: /STM_BUT2 -> unconnected-(U2-Pad62)
- U20 pad 1: GND -> Net-(R44-Pad1)
- U20 pad 2: GND -> +3V3
- U20 pad 3: GND -> +5V
- U22 pad 1: GND -> Net-(R51-Pad1)
- U22 pad 2: VDD -> GND
- U22 pad 3: +5V -> Net-(R53-Pad2)
- U3 pad 3: Net-(C9-Pad1) -> Net-(C50-Pad1)
- U3 pad 6: +3V3 -> VDDA
- U7 pad 10: unconnected-(U7-Pad10) -> GND
- U7 pad 12: +1V8 -> Net-(C62-Pad1)
- U7 pad 13: unconnected-(U7-Pad13) -> GND
- U7 pad 37: +1V8 -> Net-(C62-Pad1)
- U7 pad 49: Net-(C24-Pad1) -> Net-(C62-Pad1)
- U7 pad 54: Net-(D2-Pad1) -> Net-(U7-Pad54)
- U7 pad 55: Net-(D1-Pad1) -> Net-(U7-Pad55)
- U7 pad 61: Net-(U20-Pad5) -> Net-(R53-Pad2)
- U7 pad 62: Net-(U20-Pad6) -> Net-(R52-Pad1)
- U7 pad 63: unconnected-(U7-Pad63) -> Net-(R54-Pad1)
- U7 pad 64: +1V8 -> Net-(C62-Pad1)
- U8 pad 3: Net-(Q1-Pad3) -> /USB1_5V
- U8 pad 6: +3V3 -> VDDA
Routing:
- net VDD: track 0.00 -> 150.4 mm, vias 0 -> 16
- net /EXT_PS_OUT: track 0.00 -> 97.9 mm, vias 0 -> 1
- net /VPROG_OUT: track 0.00 -> 95.3 mm, vias 0 -> 1
- net VBUS: track 0.00 -> 89.8 mm, vias 0 -> 2
- net GND: track 1.00 -> 89.1 mm, vias 0 -> 34
- net /5V_OUT: track 0.00 -> 83.2 mm, vias 0 -> 1
- net /3V3_OUT: track 0.00 -> 69.1 mm
- net /ENC2_B: track 0.00 -> 57.7 mm, vias 0 -> 2
- net /ENC2_A: track 0.00 -> 55.0 mm, vias 0 -> 1
- net /USB1_DP: track 0.00 -> 53.0 mm, vias 0 -> 2
- net /USB1_DM: track 0.00 -> 50.5 mm, vias 0 -> 1
- net /TXD: track 0.00 -> 45.4 mm, vias 0 -> 1
- net /STM_PULSE_CNT: track 0.00 -> 44.8 mm, vias 0 -> 2
- net +VDC: track 0.00 -> 44.0 mm
- net /1V8_OUT: track 0.00 -> 43.4 mm, vias 0 -> 1
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- added copper zone on B.Cu, net +1V8
- added copper zone on In2.Cu, net +5V
- added copper zone on In1.Cu, net GND
- added copper zone on In2.Cu, net VDD
- added copper zone on B.Cu, net VDDA
Other:
- board size 77 x 100 mm -> 100 x 77 mm

Commit message: commiting changes before large concept change
Parts:
- removed the C30 at (119.3, 92.0)
- removed the C51 at (161.0, 65.3)
- removed the C78 at (130.7, 63.8)
- removed the C79 at (131.6, 86.7)
- removed the C80 at (131.8, 79.8)
- removed the C81 at (118.5, 88.9)
- removed the C82 at (119.2, 77.8)
- removed the C83 at (126.4, 91.1)
- removed the J9 at (146.8, 90.2)
- removed the L6 at (130.0, 91.9)
- removed the R35 at (113.3, 88.1)
- removed REF**: ESP32-WROOM-32, RF_Module:ESP32-WROOM-32
- removed TP3: STM_CLK_OUT, TestPoint:TestPoint_Pad_D1.0mm
- removed the U2 at (124.3, 83.8)
- removed X1: ECS-2520MV-xxx-xx, Oscillator:Oscillator_SMD_ECS_2520MV-xxx-xx-4Pin_2.5x2.0mm
- added C1: 10u, Capacitor_SMD:C_0805_2012Metric, F.Cu at (130.4, 85.7)
- added C14: 100n, Capacitor_SMD:C_0402_1005Metric, F.Cu at (129.1, 98.0)
- added C22: 22u, Capacitor_SMD:C_0805_2012Metric, F.Cu at (170.8, 70.8)
- added C24: 22u, Capacitor_SMD:C_0805_2012Metric, F.Cu at (170.4, 67.0)
- added C5: 22u, Capacitor_SMD:C_0805_2012Metric, F.Cu at (102.5, 84.3)
- added C6: 22u, Capacitor_SMD:C_0805_2012Metric, F.Cu at (98.2, 84.3)
- added C8: 10u, Capacitor_SMD:C_0805_2012Metric, F.Cu at (131.9, 88.5)
- added F1: 1A, Resistor_SMD:R_1210_3225Metric_Pad1.30x2.65mm_HandSolder, F.Cu at (106.0, 46.1)
- added J8: Conn_02x02_Odd_Even, Connector_PinHeader_2.54mm:PinHeader_2x02_P2.54mm_Vertical, F.Cu at (144.3, 90.2)
- added JP1: GND_DOMAIN_BRG, Jumper:SolderJumper-2_P1.3mm_Bridged_Pad1.0x1.5mm, B.Cu at (128.2, 81.0)
- added JP2: 5V_FROM_USB_DIS, Connector_PinHeader_2.54mm:PinHeader_1x02_P2.54mm_Vertical, F.Cu at (158.6, 64.7)
- added L1: L, Inductor_SMD:L_1206_3216Metric_Pad1.22x1.90mm_HandSolder, F.Cu at (130.2, 81.0)
- added R24: 100k, Resistor_SMD:R_0603_1608Metric_Pad0.98x0.95mm_HandSolder, F.Cu at (172.9, 99.2)
- added R8: 100k, Resistor_SMD:R_0603_1608Metric_Pad0.98x0.95mm_HandSolder, F.Cu at (137.4, 79.2)
- added R9: 100k, Resistor_SMD:R_0603_1608Metric_Pad0.98x0.95mm_HandSolder, F.Cu at (134.0, 79.2)
- added U1: AZ1117-ADJ, Package_TO_SOT_SMD:SOT-223-3_TabPin2, F.Cu at (135.9, 83.7)
- added U3: MCP3208, Package_SO:SOIC-16_3.9x9.9mm_P1.27mm, F.Cu at (133.5, 94.9)
- added U5: ESP32-S3-WROOM-1, Espressif:ESP32-S3-WROOM-1, F.Cu at (105.8, 73.4)
- F2: renamed from F1; value Polyfuse -> 1A; footprint Resistor_SMD:R_1206_3216Metric_Pad1.30x1.75mm_HandSolder -> Resistor_SMD:R_1210_3225Metric_Pad1.30x2.65mm_HandSolder
- J7: renamed from J4; value Conn_01x04 -> USBEXT
- R5: value DNP -> 100k
- SW1: footprint Button_Switch_THT:SW_PUSH_6mm_H4.3mm -> Button_Switch_SMD:SW_SPST_TL3342
- TP1: value RTC_OUT -> TestPoint
- TP2: value GENERIC_PWM -> TestPoint
- moved TP1 75.5 mm to (171.0, 38.1), turned to 0 degrees
- moved U18 71.9 mm to (133.9, -12.6), turned to 90 degrees
- moved C61 67.1 mm to (130.4, -12.5), turned to -90 degrees
- moved TP2 50.5 mm to (162.1, 64.2), turned to 0 degrees
- moved R54 38.3 mm to (127.5, 65.7), turned to 90 degrees
- moved R12 38.0 mm to (163.0, 61.5), turned to 0 degrees
- moved F2 26.0 mm to (122.4, 102.0), turned to -90 degrees
- moved C2 19.6 mm to (118.4, 91.0), turned to -90 degrees
- moved C11 16.4 mm to (109.1, 84.3), turned to -90 degrees
- moved J7 16.3 mm to (113.3, 60.3), turned to 180 degrees
- moved R14 15.9 mm to (111.3, 84.3)
- moved R1 15.4 mm to (117.9, 88.3), turned to 90 degrees
- moved R55 13.4 mm to (102.6, 111.3), turned to 0 degrees
- moved R7 12.7 mm to (101.3, 41.4)
- moved R2 12.4 mm to (99.5, 46.5), turned to -90 degrees
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- renumbered C44 to C10, C38 to C11, C43 to C12, C9 to C13, C47 to C16, C48 to C18, C49 to C19, C40 to C2, C50 to C20, C84 to C21, C58 to C23, C10 to C25, C4 to C26, C52 to C27, C53 to C28, C20 to C29, C37 to C3, C21 to C30, C22 to C31, C54 to C32, C45 to C33, C12 to C34, C11 to C35, C55 to C36, C91 to C37, C6 to C38, C7 to C39, C29 to C4, C8 to C40, C56 to C41, C57 to C42, C86 to C43, C87 to C44, C23 to C45, C14 to C47, C13 to C48, C19 to C49, C59 to C50, C41 to C51, C5 to C52, C88 to C53, C42 to C54, C89 to C55, C60 to C56, C31 to C57, C24 to C58, C32 to C59, C33 to C60, C34 to C62, C62 to C63, C63 to C64, C64 to C65, C65 to C66, C35 to C67, C26 to C68, C66 to C69, C3 to C7, C25 to C70, C67 to C71, C27 to C72, C68 to C73, C69 to C74, C70 to C75, C85 to C76, C71 to C77, C72 to C78, C73 to C79, C74 to C80, C75 to C81, C76 to C82, C28 to C83, C36 to C84, C77 to C85, C1 to C86, C2 to C87, C17 to C88, C18 to C89, C39 to C9, C16 to C90, D3 to D1, D4 to D2, D5 to D3, D1 to D4, D2 to D5, J3 to J1, J2 to J10, J13 to J11, J14 to J12, J7 to J13, J16 to J14, J8 to J2, J21 to J3, J20 to J4, J6 to J5, J5 to J6, J1 to J9, JP4 to JP3, JP1 to JP4, JP2 to JP5, JP3 to JP6, L1 to L2, L2 to L3, L5 to L4, L4 to L5, L3 to L6, Q2 to Q1, Q3 to Q2, R34 to R1, R33 to R10, R37 to R11, R10 to R12, R11 to R13, R32 to R14, R36 to R15, R12 to R16, R4 to R17, R20 to R18, R21 to R19, R31 to R2, R7 to R20, R18 to R21, R19 to R22, R17 to R23, R38 to R25, R39 to R26, R40 to R27, R41 to R28, R23 to R29, R8 to R3, R24 to R30, R25 to R31, R42 to R32, R43 to R33, R44 to R34, R45 to R35, R46 to R36, R47 to R37, R48 to R38, R49 to R39, R16 to R4, R50 to R40, R26 to R41, R22 to R42, R51 to R43, R52 to R44, R53 to R45, R28 to R46, R54 to R47, R27 to R48, R29 to R49, R30 to R50, R1 to R51, R2 to R52, R3 to R53, R13 to R54, R14 to R55, R15 to R56, R9 to R6, R55 to R7, RN2 to RN1, RN1 to RN2, U9 to U10, U13 to U11, U14 to U12, U20 to U13, U21 to U14, U19 to U15, U4 to U16, U22 to U17, U11 to U18, U7 to U19, U1 to U2, U23 to U20, U15 to U21, U16 to U22, U17 to U23, U18 to U24, U8 to U25, U10 to U4, U3 to U6, U12 to U7, U5 to U8, U6 to U9
Connections:
- C26 pad 1: VDDA -> VDD
- C26 pad 2: GND -> GNDA
- C29 pad 2: GND -> GNDA
- C30 pad 2: GND -> GNDA
- C31 pad 2: GND -> GNDA
- C45 pad 2: GND -> GNDA
- C49 pad 2: GND -> GNDA
- C90 pad 2: GND -> GNDA
- F2 pad 2: Net-(F1-Pad2) -> Net-(F2-Pad2)
- IC1 pad 34: /STM_DM -> /USBEXT_DM
- IC1 pad 35: /STM_DP -> /USBEXT_DP
- IC1 pad 37: /USBEXT_DM -> /STM_DM
- IC1 pad 38: /USBEXT_DP -> /STM_DP
- IC1 pad 45: Net-(F1-Pad2) -> Net-(F2-Pad2)
- J1 pad 3: /EXT_PS_DET -> Net-(J1-Pad3)
- J2 pad A4: VBUS -> Net-(F1-Pad1)
- J2 pad A6: Net-(J8-PadA6) -> Net-(J2-PadA6)
- J2 pad A7: Net-(J8-PadA7) -> Net-(J2-PadA7)
- J2 pad A9: VBUS -> Net-(F1-Pad1)
- J2 pad B4: VBUS -> Net-(F1-Pad1)
- J2 pad B6: Net-(J8-PadA6) -> Net-(J2-PadA6)
- J2 pad B7: Net-(J8-PadA7) -> Net-(J2-PadA7)
- J2 pad B9: VBUS -> Net-(F1-Pad1)
- J4 pad 6: /STM_PULSE_CNT -> /EXT_IO0
- Q1 pad 1: /EXT_PS_DET -> Net-(JP2-Pad1)
- Q2 pad 2: Net-(F1-Pad2) -> Net-(F2-Pad2)
- R12 pad 2: VDD -> +VDC
- R20 pad 1: /EXT_PS_DET -> GND
- R20 pad 2: VBUS -> Net-(JP2-Pad1)
- R5 pad 1: /BOOT0 -> /STM_BUT_RST
- R55 pad 2: +5V -> Net-(F2-Pad2)
- TP1 pad 1: /RTC_OUT -> Net-(J1-Pad3)
- TP2 pad 1: /GENERIC_PWM -> /EXT_PS_CONV_PG
- U10 pad 2: GND -> GNDA
- U10 pad 5: GND -> GNDA
- U15 pad 2: GND -> GNDA
- U15 pad 5: GND -> GNDA
- U16 pad 2: GND -> GNDA
- U16 pad 5: GND -> GNDA
- U2 pad 1: Net-(J8-PadA6) -> Net-(J2-PadA7)
- U2 pad 3: Net-(J8-PadA7) -> Net-(J2-PadA6)
- U2 pad 4: /USBIN_M -> /USBIN_P
- U2 pad 5: VBUS -> Net-(F1-Pad1)
- U2 pad 6: /USBIN_P -> /USBIN_M
- U25 pad 2: GND -> GNDA
- U25 pad 5: GND -> GNDA
- U6 pad 6: VDDA -> VDD
- U8 pad 2: GND -> GNDA
- U8 pad 5: GND -> GNDA
- U9 pad 2: GND -> GNDA
- U9 pad 5: GND -> GNDA
Routing:
- net Net-(F1-Pad1): track 0.00 -> 94.3 mm, vias 0 -> 2
- net /EXT_PS_OUT_CURR: track 0.00 -> 94.1 mm, vias 0 -> 2
- net VBUS: track 89.8 -> 0.00 mm, vias 2 -> 0
- net VDD: track 150.4 -> 61.3 mm, vias 16 -> 12
- net /5V_OUT_CURR: track 0.00 -> 87.1 mm, vias 0 -> 2
- net /3V3_OUT_CURR: track 0.00 -> 79.1 mm, vias 0 -> 2
- net VDDA: track 9.28 -> 78.5 mm, vias 2 -> 3
- net /1V8_OUT_CURR: track 0.00 -> 69.0 mm, vias 0 -> 2
- net GNDA: track 0.00 -> 58.8 mm, vias 0 -> 6
- net /USB1_CURR: track 0.00 -> 56.2 mm, vias 0 -> 5
- net /VPROG_OUT_CURR: track 0.00 -> 53.7 mm, vias 0 -> 2
- net /ADC_CS: track 0.00 -> 51.5 mm, vias 0 -> 2
- net /STM_PULSE_CNT: track 44.8 -> 0.00 mm, vias 2 -> 0
- net /ADC_SCK: track 0.00 -> 44.2 mm, vias 0 -> 2
- net +5V: track 37.9 -> 80.7 mm, vias 7 -> 9
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- added copper zone on In1.Cu, net +3V3
- added copper zone on F.Cu, net GND
- added copper zone on B.Cu, net GNDA
- added copper zone on In2.Cu, net GNDA
- added copper zone on F.Cu, net Net-(F2-Pad2)
Other:
- outline, holes or cut-outs redrawn
