File: hubby.kicad_sch (KiCad schematic)
At the start: 112 parts, among them IC1 FE2.1, J1 USB1, J10 VPROG_OUT, J11 1V8_OUT, J12 VPROG_OUT, J13 USB2, J14 USB2, J15 UART_OUT, J16 JTAG_OUT, J17 EXT_PS_OUT, J18 EXT_PS_OUT, J2 USB2, J3 Barrel_Jack_Switch, J4 Conn_01x04, J5 3V3_OUT, J6 1V8_OUT, J7 5V_OUT, J8 5V_OUT, J9 3V3_OUT, P1 USB_C_Plug_USB2.0, Q1 AO3401A, Q2 AO3401A, Q3 AO3401A, U1 USBLC6-2SC6, U10 TPS565208, U11 24LC00, U12 TPS565208, U13 AP1117-18, U14 AP1117-33, U15 USBLC6-2SC6, U16 USBLC6-2SC6, U17 USBLC6-2SC6, U18 USBLC6-2SC6, U19 INA181, U2 STM32F103RBTx, U20 24LC00, U3 INA181, U4 INA181, U5 INA181, U6 INA181, U7 FT2232HL, U8 INA181, U9 INA181, X1 ECS-2520MV-xxx-xx

Commit message: commiting cause i'm terrified of kicad 5.99
Parts:
- removed C5, C6, C7, C8: 10u, Capacitor_SMD:C_1206_3216Metric_Pad1.33x1.80mm_HandSolder, symbol Device:C_Small
- removed DS1: OLED-128O064D, Display:OLED-128O064D, symbol Display_Graphic:OLED-128O064D
- removed R4, R5: 10k, Resistor_SMD:R_0603_1608Metric_Pad0.98x0.95mm_HandSolder, symbol Device:R_Small
- added C29, C37, C38, C39, C40: 1n, Capacitor_SMD:C_0603_1608Metric_Pad1.08x0.95mm_HandSolder, symbol Device:C_Small
- added C31, C32, C33, C34: 10u, Capacitor_SMD:C_1206_3216Metric_Pad1.33x1.80mm_HandSolder, symbol Device:C_Small
- added C35, C36: 100n, Capacitor_SMD:C_0603_1608Metric_Pad1.08x0.95mm_HandSolder, symbol Device:C_Small
- added J19: STM_PROG_ENA, Connector_PinSocket_2.54mm:PinSocket_2x04_P2.54mm_Vertical, symbol Connector_Generic:Conn_02x04_Counter_Clockwise
- added J20: STM_EXT_IO, Connector_PinSocket_2.54mm:PinSocket_2x06_P2.54mm_Vertical, symbol Connector_Generic:Conn_02x06_Odd_Even
- added J?: Conn_01x08, symbol Connector_Generic:Conn_01x08
- added JP2: TDO_VSHIFT, Connector_PinHeader_2.54mm:PinHeader_1x03_P2.54mm_Vertical, symbol Jumper:Jumper_3_Open
- added JP3: RXD_VSHIFT, Connector_PinHeader_2.54mm:PinHeader_1x03_P2.54mm_Vertical, symbol Jumper:Jumper_3_Open
- added L4: L, Inductor_SMD:L_1206_3216Metric_Pad1.22x1.90mm_HandSolder, symbol Device:L
- added R31, R32, R33, R34: 100k, Resistor_SMD:R_0603_1608Metric_Pad0.98x0.95mm_HandSolder, symbol Device:R_Small
- added R?: 0R, Resistor_SMD:R_0603_1608Metric_Pad0.98x0.95mm_HandSolder, symbol Device:R_Small
- added R?: DNP, Resistor_SMD:R_0603_1608Metric_Pad0.98x0.95mm_HandSolder, symbol Device:R_Small
- added RN1, RN2: 22, Resistor_SMD:R_Array_Convex_4x0603, symbol Device:R_Pack04
- added SW1: SW_Push, Button_Switch_THT:SW_PUSH_6mm_H4.3mm, symbol Switch:SW_Push
- added SW2: KB_ENC, Critbit_lib:RollerEncoder_Panasonic_EVQWGD001, symbol Device:RotaryEncoder_Switch
- added SW3: BUT_BACK, Button_Switch_THT:SW_PUSH_6mm_H4.3mm, symbol Switch:SW_Push
- added U21: SN74LVC2T45YZP, Package_BGA:Texas_DSBGA-8_0.9x1.9mm_Layout2x4_P0.5mm, symbol Logic_LevelTranslator:SN74LVC2T45YZP
- added Y1: 6MHZ 2520, Crystal:Crystal_SMD_2520-4Pin_2.5x2.0mm, symbol Device:Crystal_GND24
- C15, C3, C9: footprint (none) -> Capacitor_SMD:C_1206_3216Metric_Pad1.33x1.80mm_HandSolder
- C16, C19, C20, C21, C22, C23, C24, C25, C26, C27, C28, C4: footprint (none) -> Capacitor_SMD:C_0603_1608Metric_Pad1.08x0.95mm_HandSolder
- C30: renamed from C?; footprint (none) -> Capacitor_SMD:C_0603_1608Metric_Pad1.08x0.95mm_HandSolder
- F1, R15, R17, R22, R23, R24, R25, R26: footprint (none) -> Resistor_SMD:R_1206_3216Metric_Pad1.30x1.75mm_HandSolder
- J10, J17, J6, J7, J9: footprint TerminalBlock:TerminalBlock_bornier-2_P5.08mm -> TerminalBlock_MetzConnect:TerminalBlock_MetzConnect_Type086_RT03402HBLC_1x02_P3.81mm_Horizontal
- J16: footprint (none) -> Connector_PinSocket_2.54mm:PinSocket_2x04_P2.54mm_Vertical
- J3: footprint (none) -> Connector_BarrelJack:BarrelJack_CUI_PJ-102AH_Horizontal
- J4: footprint (none) -> Connector_PinSocket_2.54mm:PinSocket_1x04_P2.54mm_Vertical
- L1, L2, L3: footprint (none) -> Inductor_SMD:L_1206_3216Metric_Pad1.22x1.90mm_HandSolder
- U11, U20: footprint (none) -> Package_SO:SOIC-8_3.9x4.9mm_P1.27mm
- Y2: renamed from Y?; value Crystal_GND24 -> 6MHZ 2520; footprint (none) -> Crystal:Crystal_SMD_2520-4Pin_2.5x2.0mm
Connections:
- net STM32_DM is gone; now on net STM_DM: IC1.34 (DM6)
- net STM32_DP is gone; now on net STM_DP: IC1.35 (DP6)
- net +3V3: now also C36.1, J?.1 (Pin_1), L4.1, R31.2, R32.2, R33.2, R34.2, R?.2, U21.A1 (VCCA)
- net +VSW: now also J20.12 (Pin_12)
- net 5V_CURR: now also U2.8 (PC0); no longer U2.26 (PB0)
- net DTR: now also RN1.6 (R3.2); no longer J15.3 (Pin_3)
- net GND: now also U2.12 (VSSA), U2.18 (VSS), U2.31 (VSS), U2.47 (VSS), U2.63 (VSS), C29.2, C31.2, C32.2, C33.2, C34.2, C35.2, C36.2, C37.2, C38.2, C39.2, C40.2, J20.1 (Pin_1), J20.11 (Pin_11), J20.3 (Pin_3), J?.2 (Pin_2), R?.1, SW1.1, SW2.C, SW2.S2, SW3.1, U21.D1 (GND), U21.D2 (DIR), Y1.2, Y1.4
- net RTS: now also RN1.5 (R4.2); no longer J15.2 (Pin_2)
- net RXD: now also JP3.2 (C); no longer J15.4 (Pin_4)
- net TCK: now also RN2.5 (R4.2); no longer J16.1 (Pin_1)
- net TDI: now also R2.2, RN2.6 (R3.2); no longer J16.3 (Pin_3), JP1.1 (A)
- net TDO: now also JP1.1 (A), JP2.2 (C); no longer J16.5 (Pin_5), R2.2
- net TMS: now also RN2.8 (R1.2); no longer J16.7 (Pin_7)
- net TXD: now also RN1.8 (R1.2); no longer J15.8 (Pin_8)
- net USB1_CURR: now also U2.9 (PC1); no longer U2.27 (PB1)
- net VPROG_PWM: now also U2.37 (PC6); no longer U2.41 (PA8)
- net ADC_???: now reaches U2.10 (PC2)
- net STM_PROBE1: now reaches U2.24 (PC4)
- net STM_PROBE1: now also J20.2 (Pin_2)
- net STM_PROBE2: now reaches U2.25 (PC5)
- net STM_PROBE2: now also J20.4 (Pin_4)
- net EXT_IO3: now reaches U2.28 (PB2)
- net EXT_IO3: now also J20.8 (Pin_8)
- net EXT_IO4: now reaches U2.29 (PB10)
- net EXT_IO4: now also J20.9 (Pin_9)
- net EXT_IO5: now reaches U2.30 (PB11)
- net EXT_IO5: now also J20.10 (Pin_10)
- net STM_TXD: now reaches U2.42 (PA9)
- net STM_TXD: now also J19.6 (Pin_6)
- net STM_RXD: now reaches U2.43 (PA10)
- net STM_RXD: now also J19.4 (Pin_4)
- net STM_DM: now reaches U2.44 (PA11)
- net STM_DP: now reaches U2.45 (PA12)
- net STM_12MHZ: now reaches U2.5 (PD0)
- net STM_12MHZ: now also X1.3 (OUT)
- net STM_PULSE_CNT: now reaches U2.50 (PA15)
- net STM_PULSE_CNT: now also J20.6 (Pin_6)
- net LCD_RST: now reaches U2.54 (PD2)
- net LCD_RST: now also J?.7 (Pin_7)
- net LCD_CLK: now reaches U2.55 (PB3)
- net LCD_CLK: now also J?.4 (Pin_4)
- net LCD_CS: now reaches U2.56 (PB4)
- net LCD_CS: now also J?.5 (Pin_5)
- net LCD_MOSI: now reaches U2.57 (PB5)
- net LCD_MOSI: now also J?.3 (Pin_3)
- net ENC_A: now reaches U2.58 (PB6)
- net ENC_A: now also C38.1, R32.1, SW2.A
- net ENC_B: now reaches U2.59 (PB7)
- net ENC_B: now also C39.1, R33.1, SW2.B
- net at U2.60 (BOOT0): now also R?.1, R?.2
- net ENC_BUT: now reaches U2.61 (PB8)
- net STM_BUT_BACK: now reaches U2.62 (PB9)
- net STM_BUT_BACK: now also C37.1, R31.1, SW3.2
- net STM_BUT_RST: now reaches U2.7 (NRST)
- net STM_BUT_RST: now also C29.1, SW1.2
- net at U7.2 (OSCI): now also Y2.1, C33.1
- net at U7.3 (OSCO): now also Y2.3, C34.1
- net at C26.1, L3.2, U7.4 (VPHY): no longer U7.9 (VPLL)
- net at IC1.22 (XIN): now also C31.1, Y1.1
- net at IC1.23 (XOUT): now also C32.1, Y1.3
- new net: JP3.3 (B), RN1.7 (R2.2), U21.C2 (B2)
- new net: C35.1, L4.2, U7.9 (VPLL)
- new net: JP2.1 (A), RN2.7 (R2.2), U21.B2 (B1)
- new net: JP2.3 (B), U21.B1 (A1)
- new net: JP3.1 (A), U21.C1 (A2)
- new net ENC_SW: C40.1, R34.1, SW2.S1
- new net EXT_IO1: J20.5 (Pin_5), U2.26 (PB0)
- new net EXT_IO2: J20.7 (Pin_7), U2.27 (PB1)
- new net STM_CLK_OUT: U2.41 (PA8)
- new net STM_SWCLK: J19.7 (Pin_7)
- new net STM_SWDIO: J19.8 (Pin_8)
- new net TARG_DTR: J15.3 (Pin_3), RN1.3 (R3.1)
- new net TARG_RTS: J15.2 (Pin_2), RN1.4 (R4.1)
- new net TARG_RXD: J15.8 (Pin_8), J19.5 (Pin_5), RN1.1 (R1.1)
- new net TARG_TCK_SWCLK: J16.1 (Pin_1), J19.2 (Pin_2), RN2.4 (R4.1)
- new net TARG_TDI: J16.5 (Pin_5), RN2.3 (R3.1)
- new net TARG_TDO_SWDIO: J16.3 (Pin_3), J19.1 (Pin_1), RN2.2 (R2.1)
- new net TARG_TMS: J16.7 (Pin_7), RN2.1 (R1.1)
- new net TARG_TXD: J15.4 (Pin_4), J19.3 (Pin_3), RN1.2 (R2.1)
- no-connect marks 31 -> 24
Other:
- moved on the sheet: C24, C26, C30, D1, D2, J15, J16, JP1, L3, R1, R2, R27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

Commit message: another progress checkpoint
Parts:
- removed J10: VPROG_OUT, TerminalBlock_MetzConnect:TerminalBlock_MetzConnect_Type086_RT03402HBLC_1x02_P3.81mm_Horizontal, symbol Connector:Screw_Terminal_01x02
- removed J11: 1V8_OUT, Connector_PinSocket_2.54mm:PinSocket_1x02_P2.54mm_Vertical, symbol Connector_Generic:Conn_01x02
- removed J12: VPROG_OUT, Connector_PinSocket_2.54mm:PinSocket_1x02_P2.54mm_Vertical, symbol Connector_Generic:Conn_01x02
- removed J15: UART_OUT, Connector_PinSocket_2.54mm:PinSocket_2x04_P2.54mm_Vertical, symbol Connector_Generic:Conn_02x04_Top_Bottom
- removed J17: EXT_PS_OUT, TerminalBlock_MetzConnect:TerminalBlock_MetzConnect_Type086_RT03402HBLC_1x02_P3.81mm_Horizontal, symbol Connector:Screw_Terminal_01x02
- removed J18: EXT_PS_OUT, Connector_PinSocket_2.54mm:PinSocket_1x02_P2.54mm_Vertical, symbol Connector_Generic:Conn_01x02
- removed J5: 3V3_OUT, Connector_PinSocket_2.54mm:PinSocket_1x02_P2.54mm_Vertical, symbol Connector_Generic:Conn_01x02
- removed J6: 1V8_OUT, TerminalBlock_MetzConnect:TerminalBlock_MetzConnect_Type086_RT03402HBLC_1x02_P3.81mm_Horizontal, symbol Connector:Screw_Terminal_01x02
- removed J7: 5V_OUT, TerminalBlock_MetzConnect:TerminalBlock_MetzConnect_Type086_RT03402HBLC_1x02_P3.81mm_Horizontal, symbol Connector:Screw_Terminal_01x02
- removed J8: 5V_OUT, Connector_PinSocket_2.54mm:PinSocket_1x02_P2.54mm_Vertical, symbol Connector_Generic:Conn_01x02
- removed J9: 3V3_OUT, TerminalBlock_MetzConnect:TerminalBlock_MetzConnect_Type086_RT03402HBLC_1x02_P3.81mm_Horizontal, symbol Connector:Screw_Terminal_01x02
- removed SW3: BUT_BACK, Button_Switch_THT:SW_PUSH_6mm_H4.3mm, symbol Switch:SW_Push
- added C41: 10u/16V, Capacitor_SMD:C_1206_3216Metric_Pad1.33x1.80mm_HandSolder, symbol Device:C_Small
- added C42: 220u, Capacitor_THT:C_Radial_D10.0mm_H12.5mm_P5.00mm, symbol Device:C_Small
- added C43, C44: 1n, Capacitor_SMD:C_0603_1608Metric_Pad1.08x0.95mm_HandSolder, symbol Device:C_Small
- added C45, C46, C5, C6, C7, C8: 10u, Capacitor_SMD:C_1206_3216Metric_Pad1.33x1.80mm_HandSolder, symbol Device:C_Small
- added J5: Screw_Terminal_01x10, TerminalBlock_Phoenix:TerminalBlock_Phoenix_MKDS-1,5-10-5.08_1x10_P5.08mm_Horizontal, symbol Connector:Screw_Terminal_01x10
- added J6: Conn_02x06_Odd_Even, Connector_PinHeader_2.54mm:PinHeader_2x06_P2.54mm_Horizontal, symbol Connector_Generic:Conn_02x06_Odd_Even
- added J7: UART_OUT, Connector_PinHeader_2.54mm:PinHeader_2x04_P2.54mm_Horizontal, symbol Connector_Generic:Conn_02x04_Odd_Even
- added R36, R37, R4: 100k, Resistor_SMD:R_0603_1608Metric_Pad0.98x0.95mm_HandSolder, symbol Device:R_Small
- added SW3: RotaryEncoder_Switch, Rotary_Encoder:RotaryEncoder_Alps_EC12E-Switch_Vertical_H20mm_CircularMountingHoles, symbol Device:RotaryEncoder_Switch
- added U22: AP1117-33, Package_TO_SOT_SMD:SOT-223-3_TabPin2, symbol Regulator_Linear:AP1117-33
- J16: footprint Connector_PinSocket_2.54mm:PinSocket_2x04_P2.54mm_Vertical -> Connector_PinHeader_2.54mm:PinHeader_2x04_P2.54mm_Horizontal
- J19: footprint Connector_PinSocket_2.54mm:PinSocket_2x04_P2.54mm_Vertical -> Connector_PinHeader_2.54mm:PinHeader_2x04_P2.54mm_Vertical
- J20: footprint Connector_PinSocket_2.54mm:PinSocket_2x06_P2.54mm_Vertical -> Connector_PinHeader_2.54mm:PinHeader_2x06_P2.54mm_Horizontal
- J21: renamed from J?; footprint (none) -> Connector_PinSocket_2.54mm:PinSocket_1x08_P2.54mm_Vertical
- SW2: value KB_ENC -> RotaryEncoder_Switch; footprint Critbit_lib:RollerEncoder_Panasonic_EVQWGD001 -> Rotary_Encoder:RotaryEncoder_Alps_EC12E-Switch_Vertical_H20mm_CircularMountingHoles
- gave numbers to parts that had none: 2
Connections:
- net ADC_??? is gone; now on net VPROG_OUT_CURR: U2.10 (PC2)
- net +3V3: no longer C19.1, C20.1, C21.1, C22.1, C23.1, C27.1, C30.1, IC1.15 (VD33), IC1.20 (VD33), IC1.26 (VD33), IC1.31 (VD33), IC1.36 (VD33), IC1.42 (VD33), J21.1 (Pin_1), L3.1, L4.1, R1.2, R28.2, R29.2, R3.2, R31.2, R32.2, R33.2, R34.2, R5.2, U11.8 (VCC), U19.6 (V+), U2.1 (VBAT), U2.13 (VDDA), U2.19 (VDD), U2.32 (VDD), U2.48 (VDD), U2.64 (VDD), U20.8 (VCC), U4.6 (V+), U5.6 (V+), U6.6 (V+), U7.50 (VREGIN), U9.6 (V+), X1.4 (VDD)
- net +5V: now also C45.1, U22.3 (VI)
- net +VSW: no longer J20.12 (Pin_12)
- net 1V8_OUT_CURR: now also U2.23 (PA7); no longer U2.22 (PA6)
- net 3V3_OUT_CURR: now also U2.22 (PA6); no longer U2.21 (PA5)
- net 5V_OUT_CURR: now also U2.21 (PA5); no longer U2.20 (PA4)
- net 5V_VLT: now also U2.15 (PA1); no longer U2.14 (PA0)
- net EXT_PS_DET: now also Q2.1 (G), R9.1
- net EXT_PS_OUT_CURR: now also U2.20 (PA4); no longer U2.17 (PA3)
- net EXT_PS_VLT: now also U2.17 (PA3); no longer U2.16 (PA2)
- net GND: now also C41.2, C42.2, C43.2, C44.2, C45.2, C46.2, C5.2, C6.2, C7.2, C8.2, J5.10 (Pin_10), J5.2 (Pin_2), J5.4 (Pin_4), J5.6 (Pin_6), J5.8 (Pin_8), J6.10 (Pin_10), J6.2 (Pin_2), J6.4 (Pin_4), J6.6 (Pin_6), J6.8 (Pin_8), J7.4 (Pin_4), J7.6 (Pin_6), R4.1, SW3.C, SW3.S2, U22.1 (GND); no longer J20.1 (Pin_1), J20.11 (Pin_11), J20.3 (Pin_3)
- net LCD_RST: now also R4.2
- net STM_PROBE1: now also J20.1 (Pin_1); no longer J20.2 (Pin_2)
- net STM_PROBE2: now also J20.3 (Pin_3); no longer J20.4 (Pin_4)
- net TARG_DTR: now also J7.5 (Pin_5)
- net TARG_RTS: now also J7.3 (Pin_3)
- net TARG_RXD: now also J7.8 (Pin_8)
- net TARG_TXD: now also J7.7 (Pin_7)
- net UART_3V3: now also J7.1 (Pin_1)
- net UART_5V: now also J7.2 (Pin_2)
- net VBUS_SUCC_ENA: no longer Q2.1 (G), R9.1
- net VPROG_OUT_CURR: no longer U2.23 (PA7)
- net VPROG_PWM: now also U2.14 (PA0); no longer U2.37 (PC6)
- net VPROG_VLT: now also U2.16 (PA2); no longer U2.15 (PA1)
- net VPROG_OUT: now reaches R25.2, U9.4 (-)
- net VPROG_OUT: now also J20.11 (Pin_11), C8.1, J5.9 (Pin_9), J6.11 (Pin_11), J6.9 (Pin_9)
- net 3V3_OUT: now reaches R23.2, U5.4 (-)
- net 3V3_OUT: now also C6.1, J5.5 (Pin_5), J6.5 (Pin_5)
- net LCD_BL: now reaches U2.52 (PC11)
- net LCD_BL: now also J21.8 (Pin_8)
- net LCD_DC: now reaches U2.53 (PC12)
- net LCD_DC: now also J21.6 (Pin_6)
- net BOOT0: now reaches R35.2, R5.1, U2.60 (BOOT0)
- net 1V8_OUT: now reaches R24.2, U6.4 (-)
- net 1V8_OUT: now also C7.1, J5.7 (Pin_7), J6.7 (Pin_7)
- net 5V_OUT: now reaches R22.2, U4.4 (-)
- net 5V_OUT: now also C5.1, J5.3 (Pin_3), J6.3 (Pin_3)
- net EXT_PS_OUT: now reaches R26.2, U19.4 (-)
- net EXT_PS_OUT: now also C41.1, J5.1 (Pin_1), J6.1 (Pin_1)
- net ENC_A: no longer names the net of C38.1, R32.1, SW2.A
- net ENC_A: no longer U2.58 (PB6)
- net ENC_B: no longer names the net of C39.1, R33.1, SW2.B
- net ENC_B: no longer U2.59 (PB7)
- net ENC_BUT renamed STM_BUT1
- net ENC_SW: no longer names the net of C40.1, R34.1, SW2.S1
- net STM_BUT_BACK: no longer names the net of C37.1, R31.1
- net STM_BUT_BACK: now also SW3.S1; no longer U2.62 (PB9)
- net VCCIO_SEL renamed VDD
- net VDD: now also C27.1, C30.1, IC1.15 (VD33), IC1.20 (VD33), IC1.26 (VD33), IC1.31 (VD33), IC1.36 (VD33), IC1.42 (VD33), J21.1 (Pin_1), L3.1, L4.1, R1.2, R28.2, R29.2, R3.2, R31.2, R32.2, R33.2, R34.2, R5.2, U11.8 (VCC), U2.1 (VBAT), U2.19 (VDD), U2.32 (VDD), U2.48 (VDD), U2.64 (VDD), U20.8 (VCC), U7.50 (VREGIN), X1.4 (VDD), C46.1, R36.2, R37.2, U22.2 (VO)
- new net: C43.1, R36.1, SW3.A
- new net: C44.1, R37.1, SW3.B
- new net: C42.1, J6.12 (Pin_12)
- new net ENC1_A: U2.58 (PB6)
- new net ENC1_B: U2.59 (PB7)
- new net STM_BUT2: U2.62 (PB9)
- new net VDDA: C19.1, C20.1, C21.1, C22.1, C23.1, U19.6 (V+), U2.13 (VDDA), U4.6 (V+), U5.6 (V+), U6.6 (V+), U9.6 (V+)
Other:
- note added: "1.8V output Low current - no step-down needed"
- note added: "3.3V internal"
- note added: "3.3V output To be upgraded to step-down when silicon shortage is dealt with"
- moved on the sheet: C11, C12, C13, C14, C19, C20, C21, C22, C23, C29, C30, C37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

Commit message: commiting before swapping MCUs
Parts:
- removed C15, C9: C, Capacitor_SMD:C_1206_3216Metric_Pad1.33x1.80mm_HandSolder, symbol Device:C
- removed J19: STM_PROG_ENA, Connector_PinHeader_2.54mm:PinHeader_2x04_P2.54mm_Vertical, symbol Connector_Generic:Conn_02x04_Counter_Clockwise
- removed J5: Screw_Terminal_01x10, TerminalBlock_Phoenix:TerminalBlock_Phoenix_MKDS-1,5-10-5.08_1x10_P5.08mm_Horizontal, symbol Connector:Screw_Terminal_01x10
- removed L2: L, Inductor_SMD:L_1206_3216Metric_Pad1.22x1.90mm_HandSolder, symbol Device:L
- removed P1: USB_C_Plug_USB2.0, Connector_USB:USB_C_Receptacle_GCT_USB4085, symbol Connector:USB_C_Plug_USB2.0
- removed Q1: AO3401A, Package_TO_SOT_SMD:SOT-23, symbol Transistor_FET:AO3401A
- removed R6: 100k, Resistor_SMD:R_0603_1608Metric_Pad0.98x0.95mm_HandSolder, symbol Device:R_Small
- removed U10, U12: TPS565208, Package_TO_SOT_SMD:SOT-23-6, symbol Regulator_Switching:TPS565208
- removed U13: AP1117-18, Package_TO_SOT_SMD:SOT-223-3_TabPin2, symbol Regulator_Linear:AP1117-18
- removed U14, U22: AP1117-33, Package_TO_SOT_SMD:SOT-223-3_TabPin2, symbol Regulator_Linear:AP1117-33
- removed U20: 24LC00, Package_SO:SOIC-8_3.9x4.9mm_P1.27mm, symbol Memory_EEPROM:24LC00
- removed U21: SN74LVC2T45YZP, Package_BGA:Texas_DSBGA-8_0.9x1.9mm_Layout2x4_P0.5mm, symbol Logic_LevelTranslator:SN74LVC2T45YZP
- added C15, C47, C54, C55, C58, C62, C63, C64, C74, C78, C84, C86, C87, C89, C9: 10u, Capacitor_SMD:C_0805_2012Metric, symbol Device:C_Small
- added C48, C49, C50, C52, C57, C60, C61, C65, C66, C67, C68, C69, C70, C71, C72, C73, C75, C76, C77, C79, C80, C81, C82, C83, C85, C91: 100n, Capacitor_SMD:C_0402_1005Metric, symbol Device:C_Small
- added C51: 47uF, Capacitor_THT:CP_Radial_D5.0mm_P2.50mm, symbol Device:C_Polarized
- added C53: 2.2u, Capacitor_SMD:C_0805_2012Metric, symbol Device:C_Small
- added C56: 47u, Capacitor_SMD:C_0805_2012Metric, symbol Device:C_Small
- added C59: SUPERCAP, Capacitor_THT:CP_Radial_D5.0mm_P2.50mm, symbol Device:C_Polarized
- added C88: 10u/16V, Capacitor_SMD:C_0805_2012Metric, symbol Device:C_Small
- added D3, D4, D5: D_Schottky, Diode_SMD:D_SMA, symbol Device:D_Schottky
- added J5: Screw_Terminal_01x12, TerminalBlock_Phoenix:TerminalBlock_Phoenix_PT-1,5-12-5.0-H_1x12_P5.00mm_Horizontal, symbol Connector:Screw_Terminal_01x12
- added J8: USB_C_Receptacle_USB2.0, Connector_USB:USB_C_Receptacle_GCT_USB4085, symbol Connector:USB_C_Receptacle_USB2.0
- added J9: STM_PROG_ENA, Connector_PinHeader_2.54mm:PinHeader_2x04_P2.54mm_Vertical, symbol Connector_Generic:Conn_02x04_Odd_Even
- added JP4: VPROG_SET_SRC, Connector_PinHeader_2.54mm:PinHeader_1x03_P2.54mm_Vertical, symbol Jumper:Jumper_3_Open
- added L2: L_Iron_Coupled, Inductor_SMD:L_Wuerth_WE-DD-Typ-M-Typ-S, symbol Device:L_Iron_Coupled
- added L5: L_Iron, Inductor_SMD:L_1206_3216Metric_Pad1.42x1.75mm_HandSolder, symbol Device:L_Iron
- added L6: L, Inductor_SMD:L_1206_3216Metric_Pad1.22x1.90mm_HandSolder, symbol Device:L
- added R38, R42, R43, R44, R45, R46, R47, R49, R50, R51, R52, R54: 100k, Resistor_SMD:R_0603_1608Metric_Pad0.98x0.95mm_HandSolder, symbol Device:R_Small
- added R39, R41: 2k, Resistor_SMD:R_0603_1608Metric_Pad0.98x0.95mm_HandSolder, symbol Device:R_Small
- added R40, R48: 3k, Resistor_SMD:R_0603_1608Metric_Pad0.98x0.95mm_HandSolder, symbol Device:R_Small
- added R53: 2k2, Resistor_SMD:R_0603_1608Metric_Pad0.98x0.95mm_HandSolder, symbol Device:R_Small
- added R55: 470, Resistor_SMD:R_0603_1608Metric_Pad0.98x0.95mm_HandSolder, symbol Device:R_Small
- added RV1: 10k, Potentiometer_THT:Potentiometer_Runtron_RM-065_Vertical, symbol Device:R_Potentiometer
- added TP1: RTC_OUT, TestPoint:TestPoint_Pad_D1.0mm, symbol Connector:TestPoint_Flag
- added TP2: GENERIC_PWM, TestPoint:TestPoint_Pad_D1.0mm, symbol Connector:TestPoint_Flag
- added TP3: STM_CLK_OUT, TestPoint:TestPoint_Pad_D1.0mm, symbol Connector:TestPoint_Flag
- added U10: MIC2405x, Critbit_lib:QFN-28-3EP_5x6mm_MIC2045x, symbol Critbit_lib:MIC2405x
- added U12: ADP1612, Package_SO:MSOP-8_3x3mm_P0.65mm, symbol Critbit_lib:ADP1612
- added U13: MCP6001U, Package_TO_SOT_SMD:SOT-23-5, symbol Amplifier_Operational:MCP6001U
- added U14, U20, U21: AZ1117-ADJ, Package_TO_SOT_SMD:SOT-223-3_TabPin2, symbol Regulator_Linear:AZ1117-ADJ
- added U22: 93LCxxAxxOT, Package_TO_SOT_SMD:SOT-23-6, symbol Memory_EEPROM:93LCxxAxxOT
- added U23: SN74LVC2T45DCUR, Package_SO:VSSOP-8_2.4x2.1mm_P0.5mm, symbol Logic_LevelTranslator:SN74LVC2T45DCUR
- added U?: ESP32-S3-WROOM-1, Espressif:ESP32-S3-WROOM-1, symbol Espressif:ESP32-S3-WROOM-1
- C1, C10, C11, C12, C13, C14, C17, C18, C2, C41, C45, C46, C5, C6, C7, C8: footprint Capacitor_SMD:C_1206_3216Metric_Pad1.33x1.80mm_HandSolder -> Capacitor_SMD:C_0805_2012Metric
- C16, C19, C20, C21, C22, C23, C24, C25, C26, C28, C29, C30, C35, C36, C37, C38, C39, C4, C40, C43, C44: footprint Capacitor_SMD:C_0603_1608Metric_Pad1.08x0.95mm_HandSolder -> Capacitor_SMD:C_0402_1005Metric
- C27: value 100n -> 10u; footprint Capacitor_SMD:C_0603_1608Metric_Pad1.08x0.95mm_HandSolder -> Capacitor_SMD:C_0805_2012Metric
- C3: footprint Capacitor_SMD:C_1206_3216Metric_Pad1.33x1.80mm_HandSolder -> Capacitor_THT:CP_Radial_D5.0mm_P2.50mm
- C31, C32, C33, C34: value 10u -> 20p; footprint Capacitor_SMD:C_1206_3216Metric_Pad1.33x1.80mm_HandSolder -> Capacitor_SMD:C_0402_1005Metric
- C42: footprint Capacitor_THT:C_Radial_D10.0mm_H12.5mm_P5.00mm -> Capacitor_THT:CP_Radial_D5.0mm_P2.50mm
- J4: footprint Connector_PinSocket_2.54mm:PinSocket_1x04_P2.54mm_Vertical -> Connector_PinHeader_2.00mm:PinHeader_1x04_P2.00mm_Vertical
- L1: value L -> 2.2u; footprint Inductor_SMD:L_1206_3216Metric_Pad1.22x1.90mm_HandSolder -> Inductor_SMD:L_Vishay_IHLP-4040
- R10: value 60k -> 100k
- R11, R12: value 40k -> 100k
- R27: value 100k -> 12k
- R9: value 100k -> 470
- Y2: value 6MHZ 2520 -> 12MHZ 2520
Connections:
- net +1V8: now also C77.1, R46.2, U21.2 (VO), U23.8 (VCCB); no longer C28.1, IC1.28 (VD18), IC1.6 (VD18), U7.12 (VCORE), U7.37 (VCORE), U7.64 (VCORE)
- net +3V3: now also R44.2, U20.2 (VO); no longer C16.1, C36.1, C4.1, R7.2, U3.6 (V+), U8.6 (V+)
- net +5V: now also C17.1, C18.1, C2.1, J13.1 (VBUS), J14.1 (VBUS), J2.1 (VBUS), C91.1, D4.2 (A), L2.3, U12.6 (VIN), U12.7 (FREQ), U13.5 (V+), U20.3 (VI), U21.3 (VI); no longer C45.1, R18.2, R9.2, U15.5 (+)
- net +VDC: now also R11.2, C47.1, C9.1, J5.12 (Pin_12), U10.13 (PVIN), U10.14 (PVIN), U10.15 (PVIN), U10.16 (PVIN), U10.17 (PVIN), U10.18 (PVIN), U10.19 (PVIN), U10.27 (VIN)
- net +VSW: now also C55.1, C56.1, L5.2, R40.2, R49.2; no longer R10.2, R20.2
- net 1V8_OUT: now also J6.5 (Pin_5), C87.1, J5.4 (Pin_4); no longer J6.7 (Pin_7)
- net 3V3_OUT: now also J6.7 (Pin_7), C86.1, J5.6 (Pin_6); no longer J6.5 (Pin_5)
- net 5V_OUT: now also J6.9 (Pin_9), C89.1, J5.8 (Pin_8); no longer J6.3 (Pin_3)
- net ENC1_A: now also C38.1, R32.1, SW2.A
- net ENC1_B: now also C39.1, R33.1, SW2.B
- net EXT_PS_DET: now also U2.33 (PB12); no longer R9.1
- net EXT_PS_OUT: now also J6.11 (Pin_11), C88.1, J5.10 (Pin_10); no longer J6.1 (Pin_1)
- net FE21_RST: now also U2.3 (PC14)
- net FT2232_RST: now also U2.51 (PC10)
- net GND: now also J20.12 (Pin_12), J20.2 (Pin_2), J20.4 (Pin_4), J6.12 (Pin_12), R9.2, U7.10 (AGND), U7.13 (TEST), C15.2, C47.2, C51.2, C54.2, C55.2, C56.2, C57.2, C58.2, C59.1, C60.2, C61.2, C62.2, C63.2, C64.2, C65.2, C66.2, C67.2, C68.2, C69.2, C70.2, C71.2, C72.2, C73.2, C74.2, C75.2, C76.2, C77.2, C78.2, C79.2, C80.2, C81.2, C82.2, C83.2, C85.2, C86.2, C87.2, C88.2, C89.2, C9.2, C91.2, J5.1 (Pin_1), J5.11 (Pin_11), J5.3 (Pin_3), J5.5 (Pin_5), J5.7 (Pin_7), J5.9 (Pin_9), J8.A1 (GND), J8.A12 (GND), J8.B1 (GND), J8.B12 (GND), J8.S1 (SHIELD), L2.1, R38.1, R41.1, R43.1, R45.1, R47.1, R50.1, R55.2, RV1.3, U10.2 (PGND), U10.21 (PGND), U10.23 (SGND), U10.5 (PGND), U10.6 (PGND), U10.7 (PGND), U10.8 (PGND), U12.4 (GND), U13.2 (V-), U22.2 (GND), U23.4 (GND), U23.5 (DIR); no longer J6.2 (Pin_2), R11.1
- net LCD_BL: now also U2.54 (PD2); no longer U2.52 (PC11)
- net LCD_DC: now also U2.52 (PC11); no longer U2.53 (PC12)
- net LCD_RST: now also U2.53 (PC12); no longer U2.54 (PD2)
- net STM_CLK_OUT: now also TP3.1
- net STM_RXD: now also J9.8 (Pin_8)
- net STM_SWCLK: now also U2.49 (PA14), J9.3 (Pin_3)
- net STM_SWDIO: now also U2.46 (PA13), J9.1 (Pin_1)
- net STM_TXD: now also J9.5 (Pin_5)
- net TARG_TDI: now also RN2.2 (R2.1); no longer RN2.3 (R3.1)
- net TARG_TDO_SWDIO: now also RN2.3 (R3.1); no longer RN2.2 (R2.1)
- net TCK: now also J9.4 (Pin_4)
- net TDI: now also RN2.7 (R2.2); no longer RN2.6 (R3.2)
- net TXD: now also J9.7 (Pin_7)
- net USB1_PWR_ENA: now also Q3.1 (G), R13.1, R14.1, U2.4 (PC15)
- net USBIN_M: now also U1.4 (I/O2); no longer U1.6 (I/O1)
- net USBIN_P: now also U1.6 (I/O1); no longer U1.4 (I/O2)
- net VBUS: now also R7.2, J8.A4 (VBUS), J8.A9 (VBUS), J8.B4 (VBUS), J8.B9 (VBUS)
- net VDD: now also C24.1, C36.1, D1.2 (A), D2.2 (A), R10.2, C59.2, C60.1, C61.1, C71.1, C72.1, C73.1, C78.1, C79.1, C80.1, C81.1, C82.1, C85.1, L6.1, R42.2, R51.2, R52.2, R54.2, RV1.1, U14.2 (VO), U22.6 (VCC), U23.1 (VCCA); no longer C27.1, IC1.15 (VD33), IC1.20 (VD33), IC1.26 (VD33), IC1.31 (VD33), IC1.36 (VD33), IC1.42 (VD33), R1.2, R3.2
- net VDDA: now also C16.1, C4.1, U3.6 (V+), U8.6 (V+), C83.1, L6.2
- net VPROG_OUT: now also J6.1 (Pin_1), J6.3 (Pin_3), C58.1, J5.2 (Pin_2); no longer J6.11 (Pin_11), J6.9 (Pin_9)
- net VPROG_PWM: now also R48.1; no longer R12.1
- net VPROG_VLT: now also R49.1, R50.2; no longer R20.1, R21.2
- net at L1.2, Q2.3 (D), R17.1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: now also R18.2, R20.2, C50.1, C51.1, C84.1
- net USB1_5V: now reaches R15.1, U8.3 (+)
- net USB1_5V: now also Q3.3 (D)
- net at C1.1, J1.1 (VBUS), R15.2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: now also U15.5 (+)
- net at JP3.3 (B), RN1.7 (R2.2): now also J9.6 (Pin_6), U23.6 (B2)
- net RTC_OUT: now reaches U2.2 (PC13)
- net RTC_OUT: now also TP1.1
- net VPROG_EN: now reaches U2.34 (PB13)
- net VPROG_EN: now also U12.3 (EN)
- net EXT_PS_CONV_EN: now reaches U2.35 (PB14)
- net EXT_PS_CONV_EN: now also R11.1, U10.26 (EN)
- net EXT_PS_CONV_PG: now reaches U2.36 (PB15)
- net EXT_PS_CONV_PG: now also R10.1, U10.25 (PG)
- net ENC2_A: now reaches U2.37 (PC6)
- net ENC2_A: now also C43.1, R36.1, SW3.A
- net ENC2_B: now reaches U2.38 (PC7)
- net ENC2_B: now also C44.1, R37.1, SW3.B
- net ENC1_BUT: now reaches U2.39 (PC8)
- net ENC1_BUT: now also C40.1, R34.1, SW2.S1
- net ENC2_BUT: now reaches U2.40 (PC9)
- net ENC2_BUT: now also C37.1, R31.1, SW3.S1
- net at L1.1: now also C48.2, C49.1, U10.10 (SW), U10.11 (SW), U10.12 (SW), U10.22 (CS), U10.4 (SW), U10.9 (SW)
- net at U7.61 (EEDATA): now also R53.2, U22.3 (DI)
- net at U7.62 (EECLK): now also R52.1, U22.4 (CLK)
- net at C26.1, L3.2, U7.4 (VPHY): now also C64.1
- net at U7.49 (VREGOUT): now also U7.12 (VCORE), U7.37 (VCORE), U7.64 (VCORE), C62.1, C65.1, C66.1, C67.1; no longer C24.1
- net at U7.54 (BCBUS3): now also R3.1; no longer D2.1 (K)
- net at U7.55 (BCBUS4): now also R1.1; no longer D1.1 (K)
- net at U7.63 (EECS): now also R54.1, U22.5 (CS)
- net at C35.1, L4.2, U7.9 (VPLL): now also C63.1
- net at C42.1: now also J6.2 (Pin_2); no longer J6.12 (Pin_12)
- net at JP2.1 (A): now also RN2.6 (R3.2), J9.2 (Pin_2), U23.7 (B1); no longer RN2.7 (R2.2)
- net at JP2.3 (B): now also U23.2 (A1)
- net at JP3.1 (A): now also U23.3 (A2)
- net at U1.3 (I/O2): now also J8.A7 (D-), J8.B7 (D-)
- net at U1.1 (I/O1): now also J8.A6 (D+), J8.B6 (D+)
- net at IC1.21 (VD_PLL): now also C28.1, IC1.25 (VD18_0), IC1.28 (VD18), IC1.6 (VD18), C74.1, C75.1, C76.1
- net at IC1.9 (VD33_O): now also C27.1, IC1.15 (VD33), IC1.20 (VD33), IC1.26 (VD33), IC1.31 (VD33), IC1.36 (VD33), IC1.42 (VD33), C68.1, C69.1, C70.1
- net STM_BUT1 renamed GENERIC_PWM
- net GENERIC_PWM: now also TP2.1
- net STM_BUT2: no longer names the net of U2.62 (PB9)
- removed net USBx_5V: C17.1, C18.1, C2.1, J13.1 (VBUS), J14.1 (VBUS), J2.1 (VBUS), Q3.3 (D)
- new net: C15.1, D3.2 (A), U10.1 (PVDD), U10.28 (VDD)
- new net: C48.1, D3.1 (K), U10.20 (BST)
- new net: C50.2, C84.2, R12.1, R20.1, R21.2, U10.24 (FB)
- new net: R42.1, R43.2, U14.1 (ADJ)
- new net: C45.1, D4.1 (K), U14.3 (VI)
- new net: R46.1, R47.2, U21.1 (ADJ)
- new net: J8.A5 (CC1), R9.1
- new net: C57.1, JP4.3 (B), R48.2
- new net: J8.B5 (CC2), R55.1
- new net: JP4.1 (A), RV1.2
- new net: C49.2, R12.2
- new net: R51.1, R53.1, U22.1 (DO)
- new net: R39.2, R40.1, R41.2, U12.2 (FB)
- new net: C52.2, R38.2
- new net: C53.1, D5.2 (A), L2.2
- new net: C53.2, L2.4, U12.5 (SW)
- new net: R44.1, R45.2, U20.1 (ADJ)
- new net: JP4.2 (C), U13.1 (+)
- new net: D2.1 (K), R3.2
- new net: R39.1, U13.3 (-), U13.4
- new net: D1.1 (K), R1.2
- new net: C52.1, U12.1 (COMP)
- new net: C54.1, D5.1 (K), L5.1
- no-connect marks 24 -> 38
Other:
- note added: "1.8V output expected to be low current - no step-down needed"
- note added: "3.3v eeprom"
- note added: "4.8V - STM 0V 2V - STM 1.9V 0V - STM 1.6V https://tinyurl.com/y2o7nnj4"
- note added: "FT2232 stuff"
- note added: "LiPo-emulating cap->"
- note added: "OSCI may be driven by CMOS-compatible oscillator"
- note added: "Power supply outputs"
- note added: "Relatively small resistance helps mitigating ripple"
- note added: "STM32"
- note added: "TODO: decide if this should be replaced by separate LDO"
- note added: "there's already large cap at VSW output"
- note removed: "1.8V output Low current - no step-down needed"
- note removed: "4.8V - STM 0V 2V - STM 1.9V 0V - STM 1.6V https://tinyurl.com/y2ouna7q"
- note removed: "fb 1.2v"
- note removed: "range 0v-3.3v"
- note removed: "range 1.2v-4.8v"
- note removed: "voltage?"
- moved on the sheet: C10, C11, C12, C13, C14, C19, C20, C21, C22, C23, C24, C25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
