File: hubby.kicad_sch (KiCad schematic)
At the start: 213 parts, among them IC1 FE2.1, J1 USB1, J13 USB2, J14 USB2, J16 JTAG_OUT, J2 USB2, J20 STM_EXT_IO, J21 Conn_01x08, J3 Barrel_Jack_Switch, J4 Conn_01x04, J5 Screw_Terminal_01x12, J6 Conn_02x06_Odd_Even, J7 UART_OUT, J8 USB_C_Receptacle_USB2.0, J9 STM_PROG_ENA, Q2 AO3401A, Q3 AO3401A, SW1 SW_Push, SW2 RotaryEncoder_Switch, SW3 RotaryEncoder_Switch, U1 USBLC6-2SC6, U10 MIC2405x, U11 24LC00, U12 ADP1612, U13 MCP6001U, U14 AZ1117-ADJ, U15 USBLC6-2SC6, U16 USBLC6-2SC6, U17 USBLC6-2SC6, U18 USBLC6-2SC6, U19 INA181, U2 STM32F103RBTx, U20 AZ1117-ADJ, U21 AZ1117-ADJ, U22 93LCxxAxxOT, U23 SN74LVC2T45DCUR, U3 INA181, U4 INA181, U5 INA181, U6 INA181, U7 FT2232HL, U8 INA181, U9 INA181, X1 ECS-2520MV-xxx-xx, Y1 6MHZ 2520, Y2 12MHZ 2520

Commit message: commiting changes before large concept change
Parts:
- removed C30: 1n, Capacitor_SMD:C_0402_1005Metric, symbol Device:C_Small
- removed C51: 47uF, Capacitor_THT:CP_Radial_D5.0mm_P2.50mm, symbol Device:C_Polarized
- removed C78: 10u, Capacitor_SMD:C_0805_2012Metric, symbol Device:C_Small
- removed C79, C80, C81, C82, C83: 100n, Capacitor_SMD:C_0402_1005Metric, symbol Device:C_Small
- removed J9: STM_PROG_ENA, Connector_PinHeader_2.54mm:PinHeader_2x04_P2.54mm_Vertical, symbol Connector_Generic:Conn_02x04_Odd_Even
- removed L6: L, Inductor_SMD:L_1206_3216Metric_Pad1.22x1.90mm_HandSolder, symbol Device:L
- removed R35: 0R, Resistor_SMD:R_0603_1608Metric_Pad0.98x0.95mm_HandSolder, symbol Device:R_Small
- removed TP1: RTC_OUT, TestPoint:TestPoint_Pad_D1.0mm, symbol Connector:TestPoint_Flag
- removed TP2: GENERIC_PWM, TestPoint:TestPoint_Pad_D1.0mm, symbol Connector:TestPoint_Flag
- removed TP3: STM_CLK_OUT, TestPoint:TestPoint_Pad_D1.0mm, symbol Connector:TestPoint_Flag
- removed U2: STM32F103RBTx, Package_QFP:LQFP-64_10x10mm_P0.5mm, symbol MCU_ST_STM32F1:STM32F103RBTx
- removed X1: ECS-2520MV-xxx-xx, Oscillator:Oscillator_SMD_ECS_2520MV-xxx-xx-4Pin_2.5x2.0mm, symbol Oscillator:ECS-2520MV-xxx-xx
- added C1, C8: 10u, Capacitor_SMD:C_0805_2012Metric, symbol Device:C_Small
- added C14: 100n, Capacitor_SMD:C_0402_1005Metric, symbol Device:C_Small
- added C22, C24, C5, C6: 22u, Capacitor_SMD:C_0805_2012Metric, symbol Device:C_Small
- added F1: 1A, Resistor_SMD:R_1210_3225Metric_Pad1.30x2.65mm_HandSolder, symbol Device:Polyfuse
- added J8: Conn_02x02_Odd_Even, Connector_PinHeader_2.54mm:PinHeader_2x02_P2.54mm_Vertical, symbol Connector_Generic:Conn_02x02_Odd_Even
- added JP1: GND_DOMAIN_BRG, Jumper:SolderJumper-2_P1.3mm_Bridged_Pad1.0x1.5mm, symbol Jumper:SolderJumper_2_Bridged
- added JP2: 5V_FROM_USB_DIS, Connector_PinHeader_2.54mm:PinHeader_1x02_P2.54mm_Vertical, symbol Jumper:Jumper_2_Open
- added L1: L, Inductor_SMD:L_1206_3216Metric_Pad1.22x1.90mm_HandSolder, symbol Device:L
- added R24, R8, R9: 100k, Resistor_SMD:R_0603_1608Metric_Pad0.98x0.95mm_HandSolder, symbol Device:R_Small
- added TP1, TP2: TestPoint, TestPoint:TestPoint_Pad_D1.0mm, symbol Connector:TestPoint
- added U1: AZ1117-ADJ, Package_TO_SOT_SMD:SOT-223-3_TabPin2, symbol Regulator_Linear:AZ1117-ADJ
- added U3: MCP3208, Package_SO:SOIC-16_3.9x9.9mm_P1.27mm, symbol Analog_ADC:MCP3208
- F2: renamed from F1; value Polyfuse -> 1A; footprint Resistor_SMD:R_1206_3216Metric_Pad1.30x1.75mm_HandSolder -> Resistor_SMD:R_1210_3225Metric_Pad1.30x2.65mm_HandSolder
- J7: renamed from J4; value Conn_01x04 -> USBEXT
- R5: value DNP -> 100k
- SW1: footprint Button_Switch_THT:SW_PUSH_6mm_H4.3mm -> Button_Switch_SMD:SW_SPST_TL3342
- gave numbers to parts that had none: 1
- renumbered C44 to C10, C38 to C11, C43 to C12, C9 to C13, C47 to C16, C48 to C18, C49 to C19, C40 to C2, C50 to C20, C84 to C21, C58 to C23, C10 to C25, C4 to C26, C52 to C27, C53 to C28, C20 to C29, C37 to C3, C21 to C30, C22 to C31, C54 to C32, C45 to C33, C12 to C34, C11 to C35, C55 to C36, C91 to C37, C6 to C38, C7 to C39, C29 to C4, C8 to C40, C56 to C41, C57 to C42, C86 to C43, C87 to C44, C23 to C45, C14 to C47, C13 to C48, C19 to C49, C59 to C50, C41 to C51, C5 to C52, C88 to C53, C42 to C54, C89 to C55, C60 to C56, C31 to C57, C24 to C58, C32 to C59, C33 to C60, C34 to C62, C62 to C63, C63 to C64, C64 to C65, C65 to C66, C35 to C67, C26 to C68, C66 to C69, C3 to C7, C25 to C70, C67 to C71, C27 to C72, C68 to C73, C69 to C74, C70 to C75, C85 to C76, C71 to C77, C72 to C78, C73 to C79, C74 to C80, C75 to C81, C76 to C82, C28 to C83, C36 to C84, C77 to C85, C1 to C86, C2 to C87, C17 to C88, C18 to C89, C39 to C9, C16 to C90, D3 to D1, D4 to D2, D5 to D3, D1 to D4, D2 to D5, J3 to J1, J2 to J10, J13 to J11, J14 to J12, J7 to J13, J16 to J14, J8 to J2, J21 to J3, J20 to J4, J6 to J5, J5 to J6, J1 to J9, JP4 to JP3, JP1 to JP4, JP2 to JP5, JP3 to JP6, L1 to L2, L2 to L3, L5 to L4, L4 to L5, L3 to L6, Q2 to Q1, Q3 to Q2, R34 to R1, R33 to R10, R37 to R11, R10 to R12, R11 to R13, R32 to R14, R36 to R15, R12 to R16, R4 to R17, R20 to R18, R21 to R19, R31 to R2, R7 to R20, R18 to R21, R19 to R22, R17 to R23, R38 to R25, R39 to R26, R40 to R27, R41 to R28, R23 to R29, R8 to R3, R24 to R30, R25 to R31, R42 to R32, R43 to R33, R44 to R34, R45 to R35, R46 to R36, R47 to R37, R48 to R38, R49 to R39, R16 to R4, R50 to R40, R26 to R41, R22 to R42, R51 to R43, R52 to R44, R53 to R45, R28 to R46, R54 to R47, R27 to R48, R29 to R49, R30 to R50, R1 to R51, R2 to R52, R3 to R53, R13 to R54, R14 to R55, R15 to R56, R9 to R6, R55 to R7, RN2 to RN1, RN1 to RN2, U9 to U10, U13 to U11, U14 to U12, U20 to U13, U21 to U14, U19 to U15, U4 to U16, U22 to U17, U11 to U18, U7 to U19, U1 to U2, U23 to U20, U15 to U21, U16 to U22, U17 to U23, U18 to U24, U8 to U25, U10 to U4, U3 to U6, U12 to U7, U5 to U8, U6 to U9
Connections:
- net BOOT0 is gone; now on net STM_BUT_RST: R5.1
- net STM_PULSE_CNT is gone; now on net EXT_IO0: J4.6 (Pin_6)
- net +5V: now also L1.1; no longer R55.2
- net +VDC: now also R12.2
- net 1V8_OUT_CURR: now also U3.6 (CH5)
- net 3V3_OUT_CURR: now also U3.5 (CH4)
- net 5V_CURR: now also U5.4 (GPIO4/TOUCH4/ADC1_CH3)
- net 5V_OUT_CURR: now also U3.4 (CH3)
- net 5V_VLT: now also U5.5 (GPIO5/TOUCH5/ADC1_CH4)
- net ENC1_A: now also U5.34 (MTDI/GPIO41/CLK_OUT1)
- net ENC1_B: now also U5.35 (MTMS/GPIO42)
- net ENC1_BUT: now also U5.27 (GPIO0/BOOT)
- net ENC2_A: now also U5.39 (GPIO1/TOUCH1/ADC1_CH0)
- net ENC2_B: now also U5.38 (GPIO2/TOUCH2/ADC1_CH1)
- net ENC2_BUT: now also U5.16 (GPIO46)
- net EXT_IO1: now also U5.12 (GPIO8/TOUCH8/ADC1_CH7/SUBSPICS1)
- net EXT_IO2: now also U5.11 (GPIO18/U1RXD/ADC2_CH7/CLK_OUT3)
- net EXT_IO3: now also U5.10 (GPIO17/U1TXD/ADC2_CH6)
- net EXT_IO4: now also U5.9 (GPIO16/U0CTS/ADC2_CH5/XTAL_32K_NH5)
- net EXT_IO5: now also U5.8 (GPIO15/U0RTS/ADC2_CH4/XTAL_32K_P)
- net EXT_PS_CONV_EN: now also U5.32 (MTCK/GPIO39/CLK_OUT3/SUBSPICS1)
- net EXT_PS_CONV_PG: now also TP2.1
- net EXT_PS_DET: no longer J1.3, Q1.1 (G), R20.1
- net EXT_PS_OUT_CURR: now also U3.3 (CH2)
- net EXT_PS_VLT: now also U5.7 (GPIO7/TOUCH7/ADC1_CH6)
- net FE21_RST: now also U5.33 (MTDO/GPIO40/CLK_OUT2)
- net FT2232_RST: now also U5.15 (GPIO3/TOUCH3/ADC1_CH2)
- net GND: now also R20.1, U5.1 (GND), U5.40 (GND), U5.41 (GND), C1.2, C22.2, C24.2, C5.2, C6.2, JP1.1 (A), R24.1; no longer C26.2, C29.2, C30.2, C31.2, C45.2, C49.2, C90.2, U10.2 (GND), U10.5 (REF), U15.2 (GND), U15.5 (REF), U16.2 (GND), U16.5 (REF), U25.2 (GND), U25.5 (REF), U8.2 (GND), U8.5 (REF), U9.2 (GND), U9.5 (REF)
- net LCD_BL: now also U5.17 (GPIO9/TOUCH9/ADC1_CH8/FSPIHD/SUBSPIHD)
- net LCD_CLK: now also U5.21 (GPIO13/TOUCH13/ADC2_CH2/FSPIQ/FSPIIO7/SUBSPIQ)
- net LCD_CS: now also U5.20 (GPIO12/TOUCH11/ADC2_CH0/FSPICS0/FSPIIO4/SUBSPICS0)
- net LCD_DC: now also U5.19 (GPIO11/TOUCH11/ADC2_CH0/FSPICS0/FSPIIO4/SUBSPICS0)
- net LCD_MOSI: now also U5.22 (GPIO14/TOUCH14/ADC2_CH3/FSPIWP/FSPIDQS/SUBSPIWP)
- net LCD_RST: now also U5.18 (GPIO10/TOUCH10/ADC1_CH9/FSPICS0/FSPIIO4/SUBSPICS0)
- net STM_BUT_RST: now also U5.3 (EN)
- net STM_DM: now also IC1.37 (DM7), U5.13 (GPIO19/U1RTS/ADC2_CH8/CLK_OUT2/USB_D-); no longer IC1.34 (DM6)
- net STM_DP: now also IC1.38 (DP7), U5.14 (GPIO20/U1CTS/ADC2_CH9/CLK_OUT1/USB_D+); no longer IC1.35 (DP6)
- net STM_PROBE1: now also U3.1 (CH0)
- net STM_PROBE2: now also U3.2 (CH1)
- net STM_RXD: now also U5.36 (U0RXD/GPIO44/CLK_OUT2), J8.3 (Pin_3)
- net STM_TXD: now also U5.37 (U0TXD/GPIO43/CLK_OUT1), J8.2 (Pin_2)
- net TXD: now also J8.4 (Pin_4)
- net USB1_CURR: now also U3.7 (CH6)
- net USB1_PWR_ENA: now also U5.23 (GPIO21)
- net USBEXT_DM: now also IC1.34 (DM6); no longer IC1.37 (DM7)
- net USBEXT_DP: now also IC1.35 (DP6); no longer IC1.38 (DP7)
- net USBIN_M: now also U2.6 (I/O1); no longer U2.4 (I/O2)
- net USBIN_P: now also U2.4 (I/O2); no longer U2.6 (I/O1)
- net VBUS: now also F1.2, JP2.2 (B); no longer J2.A4 (VBUS), J2.A9 (VBUS), J2.B4 (VBUS), J2.B9 (VBUS), R20.2, U2.5 (+)
- net VDD: now also C26.1, U5.2 (3V3), U6.6 (V+), C5.1, C6.1; no longer R12.2
- net VDDA: now also C14.1, C8.1, R8.2, U1.2 (VO), U3.15 (Vref), U3.16 (Vdd); no longer C26.1, U6.6 (V+)
- net VPROG_EN: now also U5.26 (GPIO45), R24.2
- net VPROG_OUT_CURR: now also U3.8 (CH7)
- net VPROG_PWM: now also U5.24 (GPIO47/SPICLK_P/SUBSPICLK_P_DIFF)
- net VPROG_VLT: now also U5.6 (GPIO6/TOUCH6/ADC1_CH5)
- net at C20.1, C21.1, L2.2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: now also C22.1, C24.1
- net at JP6.3 (B), RN2.7 (R2.2), U20.6 (B2): now also J8.1 (Pin_1)
- net at J2.A6 (D+), J2.B6 (D+): now also U2.3 (I/O2); no longer U2.1 (I/O1)
- net at J2.A7 (D-), J2.B7 (D-): now also U2.1 (I/O1); no longer U2.3 (I/O2)
- net EXT_IO0: now reaches U5.25 (GPIO48/SPICLK_N/SUBSPICLK_N_DIFF)
- net ADC_MOSI: now reaches U5.28 (SPIIO6/GPIO35/FSPID/SUBSPID)
- net ADC_MOSI: now also U3.11 (Din)
- net ADC_MISO: now reaches U5.29 (SPIIO7/GPIO36/FSPICLK/SUBSPICLK)
- net ADC_MISO: now also U3.12 (Dout)
- net ADC_SCK: now reaches U5.30 (SPIDQS/GPIO37/FSPIQ/SUBSPIQ)
- net ADC_SCK: now also U3.13 (CLK)
- net ADC_CS: now reaches U5.31 (GPIO38/FSPIWP/SUBSPIWP)
- net ADC_CS: now also U3.10 (~{CS}/SHDN)
- net at F2.2, IC1.45 (OVCJ1), Q2.2 (S): now also R55.2
- new net: R8.1, R9.2, U1.1 (ADJ)
- new net: JP2.1 (A), Q1.1 (G), R20.2
- new net: C1.1, L1.2, U1.3 (VI)
- new net: F1.1, J2.A4 (VBUS), J2.A9 (VBUS), J2.B4 (VBUS), J2.B9 (VBUS), U2.5 (+)
- new net: J1.3, TP1.1
- new net GNDA: C14.2, C26.2, C29.2, C30.2, C31.2, C45.2, C49.2, C8.2, C90.2, JP1.2 (B), R9.1, U10.2 (GND), U10.5 (REF), U15.2 (GND), U15.5 (REF), U16.2 (GND), U16.5 (REF), U25.2 (GND), U25.5 (REF), U3.14 (AGND), U3.9 (DGND), U8.2 (GND), U8.5 (REF), U9.2 (GND), U9.5 (REF)
- no-connect marks 38 -> 34
Other:
- note added: "From my experience, voltage on USB HUBs tends to sag a lot, in some cases to unacceptable values (like 4.6v). The DC/DC below may supply stable 5V. This voltage may leak back into the PC's USB system via Q1's body diode, which may or may not be a bad thing, implying the DC/DC works properly. This section should be remade if this ever becomes viable product"
- note added: "IO0: PU/PD -> SPI/DWNL boot"
- note added: "IO3: PU -> boot from USB"
- note added: "IO45: PD -> 3V3 flash"
- note added: "IO46: PD -> boot conf"
- note added: "MCP3208"
- note added: "Routing VDDA/GNDA to this area is too hard. Next rev?"
- note added: "This signal will probably be useless as we already sample VBUS"
- note removed: "STM32"
- moved on the sheet: C10, C11, C12, C2, C23, C29, C3, C30, C31, C38, C39, C4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
