File: rev_1/butter-board/butter-board.kicad_sch (KiCad schematic)
At the start: 78 parts, among them J1 JTAG_OUT, J2 Conn_02x02_Odd_Even, J3 Conn_02x30_Top_Bottom, J4 UART_OUT, J5 Conn_01x04, J6 STM_EXT_IO, J7 Conn_01x08, J8 Conn_02x06_Odd_Even, SW1 SW_Push, SW2 RotaryEncoder_Switch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

Commit message: moving to new pc
Parts:
- added JP?: VPROG_SET_SRC, Connector_PinHeader_2.54mm:PinHeader_1x03_P2.54mm_Vertical, symbol Jumper:Jumper_3_Open
- added RV?: 10k, Potentiometer_THT:Potentiometer_Runtron_RM-065_Vertical, symbol Device:R_Potentiometer
Connections:
- net GND: now also RV?.3
- net VDD: now also RV?.1
- net VPROG_PWM: now also JP?.2 (C); no longer U1.4 (GPIO4/TOUCH4/ADC1_CH3)
- new net: JP?.1 (A), RV?.2
- new net ESP_VPROG_PWM: JP?.3 (B), U1.4 (GPIO4/TOUCH4/ADC1_CH3)
Changed lines of the file:
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@@
     (stroke (width 0) (type default) (color 0 0 0 0))
   )
+  (wire (pts (xy 153.67 165.1) (xy 139.7 165.1))
+    (stroke (width 0) (type default) (color 0 0 0 0))
+  )
   (wire (pts (xy 502.92 45.72) (xy 502.92 78.74))
     (stroke (width 0) (type default) (color 0 0 0 0))
@@
     (stroke (width 0) (type default) (color 0 0 0 0))
   )
+  (wire (pts (xy 139.7 181.61) (xy 139.7 186.69))
+    (stroke (width 0) (type default) (color 0 0 0 0))
+  )
   (wire (pts (xy 408.94 71.12) (xy 408.94 69.85))
     (stroke (width 0) (type default) (color 0 0 0 0))
@@
     (stroke (width 0) (type default) (color 0 0 0 0))
   )
+  (wire (pts (xy 127 175.26) (xy 135.89 175.26))
+    (stroke (width 0) (type default) (color 0 0 0 0))
+  )
   (wire (pts (xy 318.77 144.78) (xy 318.77 146.05))
     (stroke (width 0) (type default) (color 0 0 0 0))
@@
     (stroke (width 0) (type default) (color 0 0 0 0))
   )
+  (wire (pts (xy 139.7 186.69) (xy 157.48 186.69))
+    (stroke (width 0) (type default) (color 0 0 0 0))
+  )
   (wire (pts (xy 97.79 243.84) (xy 80.01 243.84))
     (stroke (width 0) (type default) (color 0 0 0 0))
@@
     (stroke (width 0) (type default) (color 0 0 0 0))
   )
+  (wire (pts (xy 157.48 158.75) (xy 157.48 161.29))
+    (stroke (width 0) (type default) (color 0 0 0 0))
+  )
   (wire (pts (xy 245.11 107.95) (xy 245.11 110.49))
     (stroke (width 0) (type default) (color 0 0 0 0))
@@
     (stroke (width 0) (type default) (color 0 0 0 0))
   )
+  (wire (pts (xy 139.7 165.1) (xy 139.7 168.91))
+    (stroke (width 0) (type default) (color 0 0 0 0))
+  )
   (wire (pts (xy 369.57 194.31) (xy 369.57 196.85))
     (stroke (width 0) (type default) (color 0 0 0 0))
@@
     (stroke (width 0) (type default) (color 0 0 0 0))
   )
+  (wire (pts (xy 157.48 168.91) (xy 157.48 171.45))
+    (stroke (width 0) (type default) (color 0 0 0 0))
+  )
   (wire (pts (xy 204.47 240.03) (xy 205.74 240.03))
     (stroke (width 0) (type default) (color 0 0 0 0))
@@
     (effects (font (size 1.27 1.27)) (justify right bottom))
   )
+  (label "ESP_VPROG_PWM" (at 148.59 186.69 0)
+    (effects (font (size 1.27 1.27)) (justify left bottom))
+  )
   (label "VPROG_VLT" (at 34.29 80.01 180)
     (effects (font (size 1.27 1.27)) (justify right bottom))
@@
     (effects (font (size 1.27 1.27)) (justify right bottom))
   )
-  (label "VPROG_PWM" (at 110.49 64.77 180)
+  (label "ESP_VPROG_PWM" (at 110.49 64.77 180)
     (effects (font (size 1.27 1.27)) (justify right bottom))
   )
@@
     (effects (font (size 1.27 1.27)) (justify left bottom))
   )
+  (label "VPROG_PWM" (at 127 175.26 180)
+    (effects (font (size 1.27 1.27)) (justify right bottom))
+  )
   (label "RFU_IO2" (at 33.02 95.25 180)
     (effects (font (size 1.27 1.27)) (justify right bottom))
@@
     (pin "1")
   )
+  (symbol (lib_id "Device:R_Potentiometer") (at 157.48 165.1 0) (mirror y) (unit 1)
+    (in_bom yes) (on_board yes) (fields_autoplaced)
+    (property "Reference" "RV?" (id 0) (at 159.258 164.1915 0)
+      (effects (font (size 1.27 1.27)) (justify right))
+    )
+    (property "Value" "10k" (id 1) (at 159.258 166.9666 0)
+      (effects (font (size 1.27 1.27)) (justify right))
+    )
+    (property "Footprint" "Potentiometer_THT:Potentiometer_Runtron_RM-065_Vertical" (id 2) (at 157.48 165.1 0)
+      (effects (font (size 1.27 1.27)) hide)
+    )
+    (property "Datasheet" "~" (id 3) (at 157.48 165.1 0)
+      (effects (font (size 1.27 1.27)) hide)
+    )
+    (pin "1")
+    (pin "2")
+    (pin "3")
+  )
   (symbol (lib_id "power:GND") (at 344.17 102.87 0) (unit 1)
     (in_bom yes) (on_board yes) (fields_autoplaced)
@@
     (pin "2")
   )
+  (symbol (lib_id "power:VDD") (at 157.48 158.75 0) (unit 1)
+    (in_bom yes) (on_board yes) (fields_autoplaced)
+    (property "Reference" "#PWR?" (id 0) (at 157.48 162.56 0)
+      (effects (font (size 1.27 1.27)) hide)
+    )
+    (property "Value" "VDD" (id 1) (at 157.48 155.1455 0))
+    (property "Footprint" "" (id 2) (at 157.48 158.75 0)
+      (effects (font (size 1.27 1.27)) hide)
+    )
+    (property "Datasheet" "" (id 3) (at 157.48 158.75 0)
+      (effects (font (size 1.27 1.27)) hide)
+    )
+    (pin "1")
+  )
   (symbol (lib_id "power:GND") (at 353.06 45.72 0) (mirror y) (unit 1)
     (in_bom yes) (on_board yes) (fields_autoplaced)
@@
     (pin "1")
   )
+  (symbol (lib_id "power:GND") (at 157.48 171.45 0) (mirror y) (unit 1)
+    (in_bom yes) (on_board yes) (fields_autoplaced)
+    (property "Reference" "#PWR?" (id 0) (at 157.48 177.8 0)
+      (effects (font (size 1.27 1.27)) hide)
+    )
+    (property "Value" "GND" (id 1) (at 157.48 176.0124 0)
+      (effects (font (size 1.27 1.27)) hide)
+    )
+    (property "Footprint" "" (id 2) (at 157.48 171.45 0)
+      (effects (font (size 1.27 1.27)) hide)
+    )
+    (property "Datasheet" "" (id 3) (at 157.48 171.45 0)
+      (effects (font (size 1.27 1.27)) hide)
+    )
+    (pin "1")
+  )
   (symbol (lib_id "power:GND") (at 341.63 203.2 0) (unit 1)
     (in_bom yes) (on_board yes) (fields_autoplaced)
@@
     (pin "1")
   )
+  (symbol (lib_id "Jumper:Jumper_3_Open") (at 139.7 175.26 270) (unit 1)
+    (in_bom yes) (on_board yes)
+    (property "Reference" "JP?" (id 0) (at 141.8342 174.3515 90)
+      (effects (font (size 1.27 1.27)) (justify left))
+    )
+    (property "Value" "VPROG_SET_SRC" (id 1) (at 141.8342 177.1266 90)
+      (effects (font (size 1.27 1.27)) (justify left))
+    )
+    (property "Footprint" "Connector_PinHeader_2.54mm:PinHeader_1x03_P2.54mm_Vertical" (id 2) (at 139.7 175.26 0)
+      (effects (font (size 1.27 1.27)) hide)
+    )
+    (property "Datasheet" "~" (id 3) (at 139.7 175.26 0)
+      (effects (font (size 1.27 1.27)) hide)
+    )
+    (pin "1")
+    (pin "2")
+    (pin "3")
+  )
   (symbol (lib_id "Device:C_Small") (at 306.07 95.25 0) (mirror y) (unit 1)
     (in_bom yes) (on_board yes) (fields_autoplaced)
@@
       (reference "#PWR084") (unit 1) (value "GND") (footprint "")
     )
+    (path "/30640b3e-fc6e-4501-b0e2-163297e96389"
+      (reference "#PWR?") (unit 1) (value "VDD") (footprint "")
+    )
+    (path "/467b4061-0036-4f37-bc11-2c9e5580407c"
+      (reference "#PWR?") (unit 1) (value "GND") (footprint "")
+    )
     (path "/b8bd1d9d-1628-40de-927c-a1f6680aaada"
       (reference "C1") (unit 1) (value "1n") (footprint "Capacitor_SMD:C_0402_1005Metric")
@@
       (reference "JP4") (unit 1) (value "IOEXP_ADDR") (footprint "Jumper:SolderJumper-2_P1.3mm_Bridged2Bar_RoundedPad1.0x1.5mm")
     )
+    (path "/6055532a-24fb-434b-9bbc-cffd4eac4612"
+      (reference "JP?") (unit 1) (value "VPROG_SET_SRC") (footprint "Connector_PinHeader_2.54mm:PinHeader_1x03_P2.54mm_Vertical")
+    )
     (path "/ab2fa1df-848b-4d66-9e53-ccd0a45e8039"
       (reference "L1") (unit 1) (value "L_Ferrite") (footprint "Inductor_SMD:L_0805_2012Metric")
@@
       (reference "RN2") (unit 1) (value "22") (footprint "Resistor_SMD:R_Array_Convex_4x0603")
     )
+    (path "/08b67bcf-72a4-4cb2-89cf-2d3abed391df"
+      (reference "RV?") (unit 1) (value "10k") (footprint "Potentiometer_THT:Potentiometer_Runtron_RM-065_Vertical")
+    )
     (path "/c4305a8b-d08d-445c-9c47-aaaf383e244e"
