File: rev_1/butter-board/butter-board.kicad_pcb (KiCad board)
At the start: 4 copper layers, 90 x 58.6 mm, 78 parts, among them J1 JTAG_OUT, J2 Conn_02x02_Odd_Even, J3 Conn_02x30_Top_Bottom, J4 UART_OUT, J5 Conn_01x04, J6 STM_EXT_IO, J7 Conn_01x08, J8 Conn_02x06_Odd_Even, SW1 SW_Push, SW2 RotaryEncoder_Switch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

Commit message: checkpoint before yet another project structure change
Parts:
- moved J5 4.28 mm to (125.5, 84.0), turned to 0 degrees
- moved R12 2.73 mm to (121.5, 84.0), turned to 180 degrees
- moved L1 1.61 mm to (144.5, 84.0), turned to 90 degrees
Routing:
- net /MCU_TXD: track 74.8 -> 78.0 mm
- net /MCU_RXD: track 71.3 -> 74.4 mm
- net /USBEXT_DM: track 12.7 -> 9.93 mm
- net /I2C_SCL: track 69.0 -> 70.5 mm
- net /USBEXT_DP: track 12.3 -> 11.0 mm, vias 1 -> 0
- net +5V: track 6.30 -> 7.15 mm
- removed copper zone on B.Cu, net +5V
Other:
- outline, holes or cut-outs redrawn
