File: rev_1/bread-board/bread-board.kicad_pcb (KiCad board)
At the start: 4 copper layers, 100 x 77 mm, 160 parts, among them IC1 FE2.1, J1 USB_C_Receptacle_USB2.0, J2 USB_C_Receptacle_USB2.0, J3 Barrel_Jack_Switch, J4 USB2, J5 Conn_02x30_Top_Bottom, J6 USB2, J7 USB1, J8 USB2, J9 Screw_Terminal_01x12, Q1 AO3401A, SW1 SW_SP3T, U1 AZ1117-ADJ, U10 USBLC6-2SC6, U11 FSUSB30MUX, U12 AZ1117-ADJ, U13 INA181, U14 ADP1612, U15 INA181, U16 MIC2405x, U17 MCP6001U, U18 INA181, U19 INA181, U2 LB66200, U20 USBLC6-2SC6, U21 USBLC6-2SC6, U22 USBLC6-2SC6, U23 24LC00, U24 USBLC6-2SC6, U25 MCP3208, U3 LB66200, U4 USBLC6-2SC6, U5 INA181, U6 INA181, U7 AZ1117-ADJ, U8 INA181, U9 AZ1117-ADJ, Y1 6MHZ 2520

Commit message: moving to new pc
Parts:
- JP3: value VPROG_SET_SRC -> TEST_POT_ENA; footprint Connector_PinHeader_2.54mm:PinHeader_1x03_P2.54mm_Vertical -> Jumper:SolderJumper-2_P1.3mm_Open_RoundedPad1.0x1.5mm
- L1: value L -> L_Ferrite; footprint Inductor_SMD:L_1206_3216Metric_Pad1.22x1.90mm_HandSolder -> Inductor_SMD:L_0805_2012Metric
- RV1: value 10k -> 10k/DNP; footprint Potentiometer_THT:Potentiometer_Runtron_RM-065_Vertical -> Potentiometer_SMD:Potentiometer_Bourns_TC33X_Vertical
- moved R32 82.9 mm to (143.7, 88.6)
- moved TP2 75.9 mm to (144.0, 60.9)
- moved TP3 67.8 mm to (142.6, 57.5)
- moved U23 31.7 mm to (116.3, 90.3), turned to 0 degrees
- moved C56 29.0 mm to (117.2, 86.8), turned to 180 degrees
- moved C12 27.0 mm to (98.5, 70.0)
- moved TP1 26.1 mm to (96.9, 79.6)
- moved C52 25.4 mm to (139.9, 100.6), turned to 90 degrees
- moved TP4 23.5 mm to (101.5, 82.9)
- moved JP2 22.7 mm to (85.5, 81.1)
- moved RV1 15.5 mm to (136.4, 87.6), turned to 0 degrees
- moved C4 14.4 mm to (124.2, 92.3), turned to 180 degrees
- moved C55 13.6 mm to (134.1, 109.9), turned to 0 degrees
- moved R1 11.3 mm to (127.8, 91.8), turned to 180 degrees
- moved C2 11.1 mm to (148.7, 52.2), turned to -90 degrees
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- renumbered C11 to C10, C12 to C11, C13 to C12, C14 to C13, C15 to C14, C16 to C15, C17 to C16, C18 to C17, C19 to C18, C20 to C19, C21 to C20, C22 to C21, C23 to C22, C24 to C23, C25 to C24, C26 to C25, C27 to C26, C28 to C27, C29 to C28, C30 to C29, C31 to C30, C32 to C31, C33 to C32, C34 to C33, C35 to C34, C36 to C35, C37 to C36, C38 to C37, C39 to C38, C40 to C39, C41 to C40, C42 to C41, C43 to C42, C44 to C43, C45 to C44, C46 to C45, C47 to C46, C48 to C47, C49 to C48, C50 to C49, C6 to C5, C51 to C50, C52 to C51, C53 to C52, C54 to C53, C55 to C54, C56 to C55, C57 to C56, C58 to C57, C59 to C58, C60 to C59, C7 to C6, C61 to C60, C8 to C7, C9 to C8, C10 to C9, R34 to R32, R32 to R33, R33 to R34
Connections:
- C41 pad 1: Net-(C42-Pad1) -> Net-(C41-Pad1)
- JP3 pad 1: Net-(JP3-Pad1) -> /VPROG_PWM
- R32 pad 2: Net-(C42-Pad1) -> Net-(C41-Pad1)
- RV1 pad 2: Net-(JP3-Pad1) -> Net-(JP3-Pad2)
- U17 pad 1: Net-(JP3-Pad2) -> Net-(C41-Pad1)
Routing:
- net Net-(F1-Pad2): track 37.3 -> 3.28 mm, vias 0 -> 2
- net Net-(F2-Pad2): track 19.7 -> 1.87 mm, vias 0 -> 1
- net +5V: track 0.00 -> 14.4 mm, vias 0 -> 3
- net Net-(F2-Pad1): track 0.00 -> 11.1 mm
- net Net-(JP1-Pad1): track 0.00 -> 7.17 mm, vias 0 -> 3
- net Net-(C23-Pad2): track 0.00 -> 4.21 mm
- net Net-(C23-Pad1): track 0.00 -> 3.81 mm
- net GND: track 5.35 -> 8.70 mm, vias 3 -> 4
- net VBUS: track 0.00 -> 2.22 mm
- net Net-(C33-Pad1): track 0.00 -> 1.95 mm
- net VDD: track 0.00 -> 1.75 mm
- net /FT2232_DM: track 24.2 -> 23.7 mm
- net /USBEXT_DM: track 27.3 -> 26.8 mm
- added copper zone on In2.Cu, net +5V
- added copper zone on In1.Cu, net GND
- added copper zone on B.Cu, net Net-(F1-Pad2)
- added copper zone on B.Cu, net Net-(F2-Pad2)
- added copper zone on In2.Cu, net Net-(JP1-Pad1)

Commit message: checkpoint before yet another project structure change
Parts:
- removed the C14 at (143.7, 97.7)
- removed the C19 at (148.7, 97.7)
- removed the C30 at (151.2, 97.7)
- removed the C6 at (146.2, 97.7)
- L1: renamed from L4; footprint Inductor_SMD:L_Vishay_IHLP-4040 -> Inductor_SMD:L_Taiyo-Yuden_NR-80xx_HandSoldering
- moved U1 37.1 mm to (153.0, 100.4)
- moved U16 31.7 mm to (168.4, 98.0), turned to 0 degrees
- moved C33 30.4 mm to (169.2, 103.0), turned to 0 degrees
- moved L3 28.5 mm to (161.0, 102.0), turned to -90 degrees
- moved R32 26.8 mm to (163.2, 96.2), turned to 90 degrees
- moved C41 25.2 mm to (165.4, 103.0), turned to 0 degrees
- moved D3 25.1 mm to (136.4, 82.7), turned to 180 degrees
- moved R33 24.1 mm to (163.2, 99.7), turned to 90 degrees
- moved R2 23.2 mm to (152.0, 59.4), turned to -90 degrees
- moved L2 22.9 mm to (136.4, 88.7), turned to 0 degrees
- moved R1 22.8 mm to (153.0, 63.0)
- moved C28 22.4 mm to (136.4, 94.8), turned to 0 degrees
- moved C56 21.7 mm to (181.9, 91.1), turned to 90 degrees
- moved R35 20.1 mm to (145.1, 74.6), turned to -90 degrees
- moved C35 19.0 mm to (146.8, 74.5), turned to 90 degrees
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- renumbered C40 to C1, C32 to C10, C56 to C11, C53 to C12, C43 to C13, C33 to C14, C44 to C15, C45 to C16, C34 to C17, C46 to C18, C35 to C19, C60 to C2, C36 to C20, C47 to C21, C48 to C22, C25 to C23, C49 to C24, C50 to C25, C2 to C26, C23 to C28, C20 to C29, C37 to C3, C3 to C30, C7 to C31, C10 to C32, C16 to C33, C21 to C34, C31 to C35, C22 to C36, C41 to C37, C4 to C38, C8 to C39, C26 to C4, C11 to C40, C17 to C41, C51 to C42, C54 to C43, C59 to C44, C55 to C45, C1 to C46, C9 to C47, C15 to C48, C24 to C49, C38 to C5, C39 to C50, C52 to C51, C5 to C52, C13 to C53, C18 to C54, C29 to C55, C42 to C56, C57 to C6, C12 to C7, C58 to C8, C28 to C9, D3 to D1, D1 to D2, D2 to D3, J3 to J1, J1 to J2, J2 to J3, J5 to J4, J4 to J5, J8 to J7, J9 to J8, J7 to J9, JP4 to JP1, JP1 to JP2, JP2 to JP3, JP3 to JP4, L3 to L2, L1 to L3, L2 to L4, R29 to R1, R33 to R10, R31 to R11, R35 to R12, R19 to R13, R38 to R14, R41 to R15, R4 to R16, R6 to R17, R40 to R18, R28 to R19, R30 to R2, R39 to R20, R27 to R21, R25 to R22, R22 to R23, R26 to R24, R32 to R25, R1 to R26, R5 to R27, R9 to R28, R10 to R29, R7 to R3, R12 to R30, R13 to R31, R16 to R32, R17 to R33, R20 to R34, R21 to R35, R2 to R36, R11 to R37, R18 to R38, R23 to R39, R14 to R4, R36 to R40, R37 to R41, R8 to R5, R15 to R6, R24 to R7, R34 to R8, R3 to R9, TP5 to TP1, TP6 to TP2, TP1 to TP3, TP2 to TP5, TP3 to TP6, U25 to U1, U6 to U10, U14 to U11, U17 to U12, U1 to U13, U7 to U14, U9 to U15, U12 to U16, U20 to U17, U21 to U18, U24 to U19, U4 to U2, U22 to U20, U5 to U21, U8 to U22, U13 to U23, U15 to U24, U18 to U25, U19 to U26, U10 to U3, U16 to U4, U11 to U5, U23 to U6, U2 to U7, U3 to U9
Connections:
- C10 pad 1: Net-(C28-Pad2) (its old number) -> /VDC_SW
- C14 pad 1: Net-(C33-Pad1) (its old number) -> /5V_FROM_VDC
- C17 pad 1: Net-(C33-Pad1) (its old number) -> /5V_FROM_VDC
- C19 pad 1: Net-(C33-Pad1) (its old number) -> /5V_FROM_VDC
- C20 pad 1: Net-(C33-Pad1) (its old number) -> /5V_FROM_VDC
- C9 pad 2: Net-(C28-Pad2) (its old number) -> /VDC_SW
- L1 pad 1: Net-(C28-Pad2) (its old number) -> /VDC_SW
- L1 pad 2: Net-(C33-Pad1) (its old number) -> /5V_FROM_VDC
- R11 pad 2: Net-(C33-Pad1) (its old number) -> /5V_FROM_VDC
- U4 pad 10: Net-(C28-Pad2) (its old number) -> /VDC_SW
- U4 pad 11: Net-(C28-Pad2) (its old number) -> /VDC_SW
- U4 pad 12: Net-(C28-Pad2) (its old number) -> /VDC_SW
- U4 pad 22: Net-(C28-Pad2) (its old number) -> /VDC_SW
- U4 pad 4: Net-(C28-Pad2) (its old number) -> /VDC_SW
- U4 pad 9: Net-(C28-Pad2) (its old number) -> /VDC_SW
- U9 pad 6: Net-(C33-Pad1) (its old number) -> /5V_FROM_VDC
Routing:
- net GND: track 8.70 -> 54.6 mm, vias 4 -> 14
- net /5V_FROM_VDC: track 0.00 -> 34.4 mm, vias 0 -> 8
- net +VDC: track 0.00 -> 27.3 mm, vias 0 -> 3
- net Net-(C4-Pad1): track 0.00 -> 17.3 mm
- net /VPROG_PWM: track 0.00 -> 16.6 mm
- net +VSW: track 0.00 -> 14.2 mm
- net Net-(C9-Pad1): track 0.00 -> 14.1 mm
- net /VDC_SW: track 0.00 -> 13.2 mm, vias 0 -> 1
- net Net-(C28-Pad1): track 3.81 -> 15.6 mm
- net /EXT_PS_CONV_PG: track 0.00 -> 9.37 mm, vias 0 -> 2
- net +5V: track 14.4 -> 21.9 mm, vias 3 -> 8
- net Net-(R22-Pad2): track 0.00 -> 7.44 mm
- net Net-(C30-Pad1): track 0.00 -> 6.17 mm
- net /EXT_PS_CONV_EN: track 0.00 -> 5.59 mm
- net /VPROG_EN: track 0.00 -> 5.19 mm
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- added copper zone on F.Cu, net +VDC
- added copper zone on B.Cu, net /5V_FROM_VDC
- added copper zone on F.Cu, net /VDC_SW
- added copper zone on B.Cu, net GNDA
- added copper zone on In2.Cu, net VDDA

Commit message: adding yeast^WcubeMX project, working on pcb
Parts:
- added C57: 20p, Capacitor_SMD:C_0402_1005Metric, F.Cu at (150.7, 78.5)
- added C58: 100n, Capacitor_SMD:C_0402_1005Metric, F.Cu at (143.4, 86.1)
- added C59: 100n, Capacitor_SMD:C_0402_1005Metric, F.Cu at (132.6, 82.2)
- added C60: 100n, Capacitor_SMD:C_0402_1005Metric, F.Cu at (122.5, 53.5)
- added C61: 100n, Capacitor_SMD:C_0402_1005Metric, F.Cu at (129.6, 53.4)
- added C62: 100n, Capacitor_SMD:C_0402_1005Metric, F.Cu at (136.6, 53.4)
- added C63: 100n, Capacitor_SMD:C_0402_1005Metric, F.Cu at (147.2, 76.2)
- added C64: 100n, Capacitor_SMD:C_0402_1005Metric, F.Cu at (143.0, 71.4)
- added C65: 100n, Capacitor_SMD:C_0402_1005Metric, F.Cu at (136.5, 71.4)
- added C66: 100n, Capacitor_SMD:C_0402_1005Metric, F.Cu at (82.3, 69.7)
- added JP5: MCU_USB_MUX_ENA, Jumper:SolderJumper-2_P1.3mm_Open_RoundedPad1.0x1.5mm, F.Cu at (83.0, 66.9)
- added Q10: BC847, Package_TO_SOT_SMD:SOT-23, F.Cu at (122.4, 60.3)
- added Q11: BC847, Package_TO_SOT_SMD:SOT-23, F.Cu at (129.6, 60.3)
- added Q12: BC847, Package_TO_SOT_SMD:SOT-23, F.Cu at (136.6, 60.3)
- added Q2: AO3401A, Package_TO_SOT_SMD:SOT-23, F.Cu at (125.9, 60.3)
- added Q3: AO3401A, Package_TO_SOT_SMD:SOT-23, F.Cu at (133.1, 60.3)
- added Q4: AO3401A, Package_TO_SOT_SMD:SOT-23, F.Cu at (140.1, 60.3)
- added Q5: AO3401A, Package_TO_SOT_SMD:SOT-23, F.Cu at (136.8, 136.3)
- added Q6: AO3401A, Package_TO_SOT_SMD:SOT-23, F.Cu at (176.0, 61.5)
- added Q7: BC847, Package_TO_SOT_SMD:SOT-23, F.Cu at (175.8, 65.3)
- added Q8: BC847, Package_TO_SOT_SMD:SOT-23, F.Cu at (176.0, 58.0)
- added Q9: BC847, Package_TO_SOT_SMD:SOT-23, F.Cu at (140.3, 136.3)
- added R42: 10k, Resistor_SMD:R_0603_1608Metric_Pad0.98x0.95mm_HandSolder, F.Cu at (140.3, 86.3)
- added R43: 100mR, Resistor_SMD:R_1206_3216Metric_Pad1.30x1.75mm_HandSolder, F.Cu at (125.9, 55.8)
- added R44: 100mR, Resistor_SMD:R_1206_3216Metric_Pad1.30x1.75mm_HandSolder, F.Cu at (133.1, 55.7)
- added R45: 100mR, Resistor_SMD:R_1206_3216Metric_Pad1.30x1.75mm_HandSolder, F.Cu at (140.1, 55.8)
- added R46: 10k, Resistor_SMD:R_0603_1608Metric_Pad0.98x0.95mm_HandSolder, F.Cu at (173.1, 68.7)
- added R47: 10k, Resistor_SMD:R_0603_1608Metric_Pad0.98x0.95mm_HandSolder, F.Cu at (173.3, 61.5)
- added R48: 3k, Resistor_SMD:R_0603_1608Metric_Pad0.98x0.95mm_HandSolder, F.Cu at (173.1, 65.3)
- added R49: 3k, Resistor_SMD:R_0603_1608Metric_Pad0.98x0.95mm_HandSolder, F.Cu at (173.3, 58.0)
- added R50: 10k, Resistor_SMD:R_0603_1608Metric_Pad0.98x0.95mm_HandSolder, F.Cu at (140.3, 133.5)
- added R51: 10k, Resistor_SMD:R_0603_1608Metric_Pad0.98x0.95mm_HandSolder, F.Cu at (125.9, 63.0)
- added R52: 10k, Resistor_SMD:R_0603_1608Metric_Pad0.98x0.95mm_HandSolder, F.Cu at (133.1, 63.0)
- added R53: 10k, Resistor_SMD:R_0603_1608Metric_Pad0.98x0.95mm_HandSolder, F.Cu at (140.1, 63.0)
- added R54: 3k, Resistor_SMD:R_0603_1608Metric_Pad0.98x0.95mm_HandSolder, F.Cu at (143.2, 142.0)
- added R55: 3k, Resistor_SMD:R_0603_1608Metric_Pad0.98x0.95mm_HandSolder, F.Cu at (122.4, 63.0)
- added R56: 3k, Resistor_SMD:R_0603_1608Metric_Pad0.98x0.95mm_HandSolder, F.Cu at (129.6, 63.0)
- added R57: 3k, Resistor_SMD:R_0603_1608Metric_Pad0.98x0.95mm_HandSolder, F.Cu at (136.6, 63.0)
- added TP7: STM_BOOT0, TestPoint:TestPoint_Pad_D1.0mm, F.Cu at (86.7, 66.7)
- added U27: INA181, Package_TO_SOT_SMD:SOT-23-6, F.Cu at (130.1, 56.1)
- added U28: INA181, Package_TO_SOT_SMD:SOT-23-6, F.Cu at (137.1, 56.1)
- added U8: INA181, Package_TO_SOT_SMD:SOT-23-6, F.Cu at (123.0, 56.1)
- added Y2: 6MHZ 2520, Crystal:Crystal_SMD_2520-4Pin_2.5x2.0mm, F.Cu at (149.1, 80.2)
- C2: value 100n -> 20p
- J6: value USB2 -> USB3
- J7: value USB2 -> USB4
- JP1: value GND_DOMAIN_BRG -> FUSE_BYP; footprint Jumper:SolderJumper-2_P1.3mm_Bridged_Pad1.0x1.5mm -> Jumper:SolderJumper-2_P1.3mm_Open_RoundedPad1.0x1.5mm; moved to F.Cu
- R36, R37, R38, R40: value 0.5R -> 50mR
- R39: value 0.5R -> 200mR
- R41: value 0.5R -> 100mR
- SW1: value SW_SP3T -> PCM13
- U1: value MCP3208 -> STM32F103RFTx; footprint Package_SO:SOIC-16_3.9x9.9mm_P1.27mm -> Package_QFP:LQFP-64_10x10mm_P0.5mm
- moved JP1 81.3 mm to (145.2, 134.4), turned to 180 degrees
- moved R16 78.5 mm to (143.2, 64.2), turned to 90 degrees
- moved JP3 63.7 mm to (145.9, 61.0), turned to 180 degrees
- moved Q1 55.8 mm to (175.8, 68.8), turned to 0 degrees
- moved C51 43.3 mm to (139.8, 143.9), turned to 180 degrees
- moved F3 42.6 mm to (145.9, 136.7), turned to 0 degrees
- moved C45 34.0 mm to (137.0, 144.4)
- moved R41 34.0 mm to (136.2, 140.8)
- moved U26 34.0 mm to (139.2, 141.2)
- moved R5 30.3 mm to (115.0, 39.2), turned to -90 degrees
- moved R3 29.6 mm to (113.4, 39.2), turned to -90 degrees
- moved R20 27.7 mm to (111.0, 81.4), turned to 90 degrees
- moved C35 27.5 mm to (155.1, 100.8), turned to 0 degrees
- moved R35 26.4 mm to (155.1, 99.0), turned to 180 degrees
- moved U1 25.3 mm to (139.9, 78.7)
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Connections:
- net /RFU_IO1 renamed /RFU_HSIO2
- net /RFU_IO2 renamed /RFU_HSIO1
- net Net-(F1-Pad2) renamed /VBUSIN_1
- net Net-(F2-Pad2) renamed /VBUSIN_2
- net Net-(JP2-Pad1) renamed /VBUSIN_COM
- C2 pad 1: VDDA -> Net-(C2-Pad1)
- C2 pad 2: GNDA -> GND
- C42 pad 1: +5V -> Net-(R43-Pad2)
- C43 pad 1: +5V -> Net-(U18-Pad5)
- C44 pad 1: +5V -> Net-(R45-Pad2)
- F3 pad 1: +5V -> Net-(Q5-Pad2)
- F3 pad 2: Net-(F3-Pad2) -> +5V
- IC1 pad 34: /FT2232_DM -> /STM32_DM
- IC1 pad 35: /FT2232_DP -> /STM32_DP
- IC1 pad 37: /USBEXT_DM -> /FT2232_DM
- IC1 pad 38: /USBEXT_DP -> /FT2232_DP
- IC1 pad 45: Net-(F3-Pad2) -> +5V
- J4 pad 11: /USB_OC_DET -> unconnected-(J4-Pad11)
- J4 pad 12: /USBIN_SEL -> unconnected-(J4-Pad12)
- J4 pad 13: /FE21_RST -> unconnected-(J4-Pad13)
- J4 pad 14: /VPROG_EN -> unconnected-(J4-Pad14)
- J4 pad 15: /VPROG_PWM -> unconnected-(J4-Pad15)
- J4 pad 17: /VPROG_VLT -> unconnected-(J4-Pad17)
- J4 pad 18: /USBIN2_CC2 -> unconnected-(J4-Pad18)
- J4 pad 19: /USBIN2_CC1 -> unconnected-(J4-Pad19)
- J4 pad 20: /USBIN1_CC2 -> unconnected-(J4-Pad20)
- J4 pad 21: /USBIN1_CC1 -> unconnected-(J4-Pad21)
- J4 pad 39: /RFU_CS -> unconnected-(J4-Pad39)
- J4 pad 46: /PS_SDA -> /PS_SCL
- J4 pad 47: /PS_SCL -> /PS_SDA
- J4 pad 48: /RFU_IO4 -> /CON_GPIO1
- J4 pad 49: /RFU_IO3 -> /CON_GPIO2
- J4 pad 50: /EXT_PS_CONV_EN -> /CON_GPIO3
- J4 pad 51: /EXT_PS_CONV_PG -> /CON_GPIO4
- J5 pad 1: +5V -> Net-(R43-Pad2)
- J6 pad 1: +5V -> Net-(U18-Pad5)
- J7 pad 1: +5V -> Net-(R45-Pad2)
- JP1 pad 1: GND -> +5V
- JP1 pad 2: GNDA -> Net-(Q5-Pad2)
- Q1 pad 1: /USB_OC_DET -> Net-(Q1-Pad1)
- Q1 pad 2: Net-(F3-Pad2) -> +5V
- Q1 pad 3: /USB1_5V -> Net-(R36-Pad1)
- R13 pad 2: /USBIN_SEL -> Net-(R13-Pad2)
- R18 pad 1: /USB_OC_DET -> Net-(R18-Pad1)
- R20 pad 1: /USB_OC_DET -> Net-(R18-Pad1)
- R20 pad 2: Net-(F3-Pad2) -> +5V
- R36 pad 1: +5V -> Net-(R36-Pad1)
- R37 pad 1: +VDC -> Net-(R37-Pad1)
- R41 pad 1: /USB1_5V -> Net-(Q5-Pad3)
- U1 pad 1: /EXT_PS_VLT -> VDD
- U1 pad 10: /ADC_CS -> /1V8_OUT_CURR
- U1 pad 11: /ADC_MOSI -> /VPROG_OUT_CURR
- U1 pad 12: /ADC_MISO -> GND
- U1 pad 13: /ADC_SCK -> VDDA
- U1 pad 14: GNDA -> /5V_CURR
- U1 pad 15: VDDA -> /EXT_PS_OUT_CURR
- U1 pad 16: VDDA -> /5V_OUT_CURR
- U1 pad 2: /5V_CURR -> unconnected-(U1-Pad2)
- U1 pad 3: /EXT_PS_OUT_CURR -> /EXT_PS_CONV_EN
- U1 pad 4: /5V_OUT_CURR -> /EXT_PS_CONV_PG
- U1 pad 5: /3V3_OUT_CURR -> Net-(C2-Pad1)
- U1 pad 6: /1V8_OUT_CURR -> Net-(C57-Pad1)
- U1 pad 7: /USB1_CURR -> Net-(U1-Pad7)
- U1 pad 8: /VPROG_OUT_CURR -> /EXT_PS_VLT
- U1 pad 9: GNDA -> /VPROG_VLT
- U17 pad 5: +5V -> Net-(R43-Pad2)
- U18 pad 5: +5V -> Net-(U18-Pad5)
- U19 pad 5: +5V -> Net-(R45-Pad2)
- U21 pad 3: +5V -> Net-(R36-Pad1)
- U22 pad 3: +VDC -> Net-(R37-Pad1)
- U26 pad 3: /USB1_5V -> Net-(Q5-Pad3)
- U5 pad 1: /USBIN_SEL -> Net-(R13-Pad2)
Routing:
- net /USBEXT_DM: track 26.8 -> 0.00 mm, vias 2 -> 0
- net /USBEXT_DP: track 26.1 -> 0.00 mm, vias 2 -> 0
- net /STM32_DM: track 0.00 -> 24.7 mm, vias 0 -> 1
- net /STM32_DP: track 0.00 -> 24.6 mm, vias 0 -> 1
- net /VPROG_PWM: track 16.6 -> 0.00 mm
- net /USBIN1_CC2: track 0.00 -> 9.19 mm
- net /USBIN1_CC1: track 0.00 -> 9.03 mm
- net +5V: track 21.9 -> 14.2 mm, vias 8 -> 5
- net Net-(C30-Pad1): track 6.17 -> 0.28 mm
- net Net-(C2-Pad1): track 0.00 -> 4.10 mm
- net Net-(C57-Pad1): track 0.00 -> 4.03 mm
- net Net-(C28-Pad1): track 15.6 -> 13.7 mm
- net Net-(JP4-Pad2): track 1.90 -> 0.00 mm
- net GND: track 54.6 -> 52.9 mm, vias 14 -> 13
- net Net-(J2-PadA7): track 3.09 -> 4.79 mm
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
Commit message: routing AAAAAAAAAAAAAAA
Parts:
- added D10: LED, LED_SMD:LED_0603_1608Metric, F.Cu at (177.6, 110.8)
- added D11: LED, LED_SMD:LED_0603_1608Metric, F.Cu at (175.4, 110.8)
- added D12: LED, LED_SMD:LED_0603_1608Metric, F.Cu at (171.2, 110.8)
- added D4: LED, LED_SMD:LED_0603_1608Metric, F.Cu at (183.9, 110.8)
- added D5: LED, LED_SMD:LED_0603_1608Metric, F.Cu at (173.3, 110.8)
- added D6: LED, LED_SMD:LED_0603_1608Metric, F.Cu at (179.7, 110.8)
- added D7: LED, LED_SMD:LED_0603_1608Metric, F.Cu at (166.9, 110.8)
- added D8: LED, LED_SMD:LED_0603_1608Metric, F.Cu at (181.8, 110.8)
- added D9: LED, LED_SMD:LED_0603_1608Metric, F.Cu at (169.1, 110.8)
- added J10: Conn_01x03, Connector_PinHeader_2.54mm:PinHeader_1x03_P2.54mm_Vertical, F.Cu at (76.0, 57.7)
- added JP6: X, Jumper:SolderJumper-2_P1.3mm_Open_RoundedPad1.0x1.5mm, F.Cu at (147.0, 72.4)
- added JP7: X, Jumper:SolderJumper-2_P1.3mm_Open_RoundedPad1.0x1.5mm, F.Cu at (115.5, 86.3)
- added JP8: X, Jumper:SolderJumper-2_P1.3mm_Open_RoundedPad1.0x1.5mm, F.Cu at (112.6, 86.3)
- added R58: 2k, Resistor_SMD:R_0603_1608Metric_Pad0.98x0.95mm_HandSolder, F.Cu at (166.5, 94.5)
- added R59: 3k, Resistor_SMD:R_0603_1608Metric_Pad0.98x0.95mm_HandSolder, F.Cu at (173.2, 54.5)
- added R60: 2k, Resistor_SMD:R_0603_1608Metric_Pad0.98x0.95mm_HandSolder, F.Cu at (166.5, 97.8)
- added R61: 2k, Resistor_SMD:R_0603_1608Metric_Pad0.98x0.95mm_HandSolder, F.Cu at (160.4, 94.5)
- added R62: 2k, Resistor_SMD:R_0603_1608Metric_Pad0.98x0.95mm_HandSolder, F.Cu at (170.5, 97.8)
- added R63: 2k, Resistor_SMD:R_0603_1608Metric_Pad0.98x0.95mm_HandSolder, F.Cu at (160.4, 97.8)
- added R64: 2k, Resistor_SMD:R_0603_1608Metric_Pad0.98x0.95mm_HandSolder, F.Cu at (170.5, 94.5)
- added R65: 2k, Resistor_SMD:R_0603_1608Metric_Pad0.98x0.95mm_HandSolder, F.Cu at (162.4, 97.8)
- added R66: 2k, Resistor_SMD:R_0603_1608Metric_Pad0.98x0.95mm_HandSolder, F.Cu at (162.4, 94.5)
- added R67: 2k, Resistor_SMD:R_0603_1608Metric_Pad0.98x0.95mm_HandSolder, F.Cu at (168.5, 94.5)
- added R68: 2k, Resistor_SMD:R_0603_1608Metric_Pad0.98x0.95mm_HandSolder, F.Cu at (164.4, 97.8)
- added R69: 2k, Resistor_SMD:R_0603_1608Metric_Pad0.98x0.95mm_HandSolder, F.Cu at (168.5, 97.8)
- added R70: 2k, Resistor_SMD:R_0603_1608Metric_Pad0.98x0.95mm_HandSolder, F.Cu at (164.4, 94.5)
- added R71: 3k, Resistor_SMD:R_0603_1608Metric_Pad0.98x0.95mm_HandSolder, F.Cu at (156.4, 97.8)
- added R72: 100k, Resistor_SMD:R_0603_1608Metric_Pad0.98x0.95mm_HandSolder, F.Cu at (156.3, 94.5)
- added R73: 100k, Resistor_SMD:R_0603_1608Metric_Pad0.98x0.95mm_HandSolder, F.Cu at (158.4, 97.8)
- added SW2: BUT_SMD, Button_Switch_SMD:SW_SPST_TL3342, F.Cu at (134.6, 67.2)
- added SW3: BUT_SMD, Button_Switch_SMD:SW_SPST_TL3342, F.Cu at (143.2, 67.2)
- added SW4: PCM13, Button_Switch_SMD:SW_SP3T_PCM13, F.Cu at (146.8, 110.8)
- added TP8: RFUPAD, TestPoint:TestPoint_Pad_D1.0mm, F.Cu at (141.3, 89.1)
- C13, C17, C19, C20, C21, C23, C28, C29, C3, C30, C31, C32, C33, C34, C36, C38, C39, C4, C40, C41, C42, C43, C44, C45, C5, C52, C53, C54, C55, C56: footprint Capacitor_SMD:C_0805_2012Metric -> Capacitor_SMD:C_0603_1608Metric
- TP5: value ID2_CTRL -> RFUPAD
- moved JP5 66.7 mm to (147.0, 85.7), turned to 90 degrees
- moved TP7 57.1 mm to (139.3, 89.0)
- moved JP1 53.5 mm to (123.0, 85.7)
- moved F3 52.7 mm to (123.2, 89.2)
- moved R54 51.1 mm to (129.1, 92.9), turned to 90 degrees
- moved C45 47.6 mm to (114.6, 102.5), turned to 90 degrees
- moved C66 47.3 mm to (129.6, 67.2), turned to 90 degrees
- moved R13 46.3 mm to (158.4, 94.5)
- moved Q5 46.2 mm to (121.4, 92.8)
- moved Q9 46.2 mm to (124.9, 92.8)
- moved U26 46.2 mm to (123.9, 97.7)
- moved R41 46.2 mm to (120.8, 97.3)
- moved C51 46.2 mm to (124.4, 100.4)
- moved R50 42.6 mm to (127.5, 92.9), turned to 90 degrees
- moved C38 40.9 mm to (160.5, 80.8), turned to 0 degrees
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Connections:
- J4 pad 11: unconnected-(J4-Pad11) -> /EXT_PS_CONV_EN
- J4 pad 12: unconnected-(J4-Pad12) -> /EXT_PS_CONV_PG
- J4 pad 13: unconnected-(J4-Pad13) -> /VPROG_PWM
- J4 pad 14: unconnected-(J4-Pad14) -> /STM_UART_TX
- J4 pad 15: unconnected-(J4-Pad15) -> /STM_UART_RX
- J4 pad 20: unconnected-(J4-Pad20) -> /SWDIO
- J4 pad 21: unconnected-(J4-Pad21) -> /SWCLK
- J4 pad 41: /ADC_MOSI -> /ADC_SCK
- J4 pad 44: /ADC_SCK -> /ADC_MOSI
- TP5 pad 1: Net-(R16-Pad2) -> Net-(U1-Pad54)
- U1 pad 2: unconnected-(U1-Pad2) -> /USBIN_SEL
- U1 pad 4: /EXT_PS_CONV_PG -> Net-(U1-Pad4)
- U1 pad 42: /UART_LOG -> /STM_UART_TX
- U1 pad 43: /USBIN_SEL -> /STM_UART_RX
- U1 pad 52: unconnected-(U1-Pad52) -> /FE21_EEPROM_SDA
- U1 pad 53: unconnected-(U1-Pad53) -> /FE21_EEPROM_SCL
- U1 pad 54: unconnected-(U1-Pad54) -> Net-(U1-Pad54)
- U1 pad 55: unconnected-(U1-Pad55) -> /STM_LED1
- U1 pad 56: unconnected-(U1-Pad56) -> /STM_LED2
- U1 pad 57: unconnected-(U1-Pad57) -> /STM_LED3
- U1 pad 61: unconnected-(U1-Pad61) -> Net-(U1-Pad61)
- U6 pad 5: Net-(IC1-Pad2) -> /FE21_EEPROM_SDA
- U6 pad 6: Net-(IC1-Pad3) -> /FE21_EEPROM_SCL
- U6 pad 7: unconnected-(U6-Pad7) -> GND
- U7 pad 3: /VBUSIN_1 -> /VBUSIN_2
- U7 pad 6: /VBUSIN_2 -> /VBUSIN_1
Routing:
- net /VPROG_PWM: track 0.00 -> 41.7 mm, vias 0 -> 3
- net Net-(C44-Pad1): track 0.00 -> 29.4 mm, vias 0 -> 1
- net /FE21_EEPROM_SDA: track 0.00 -> 27.5 mm
- net GND: track 52.9 -> 78.1 mm, vias 13 -> 21
- net /PS_SDA: track 0.00 -> 23.8 mm, vias 0 -> 2
- net /VBUSIN_2: track 1.87 -> 24.3 mm, vias 1 -> 0
- net /PS_SCL: track 0.00 -> 22.1 mm, vias 0 -> 2
- net Net-(C43-Pad1): track 0.00 -> 17.4 mm, vias 0 -> 1
- net /FE21_EEPROM_SCL: track 0.00 -> 17.0 mm
- net /LOADSW_USB1: track 0.00 -> 15.8 mm, vias 0 -> 2
- net /STM_LED1: track 0.00 -> 14.1 mm, vias 0 -> 2
- net /STM_LED2: track 0.00 -> 12.6 mm, vias 0 -> 2
- net VDD: track 1.75 -> 12.7 mm, vias 0 -> 4
- net /ADC_CS: track 0.00 -> 9.85 mm
- net /ADC_SCK: track 0.00 -> 9.85 mm
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- added copper zone on B.Cu, net VDD
- added copper zone on B.Cu, net VDDA
- removed copper zone on B.Cu, net GNDA
- removed copper zone on In2.Cu, net VDDA
Other:
- outline, holes or cut-outs redrawn
- board text added: "5V"
- board text added: "beat"
- board text added: "debug"
- board text added: "status"
- board text added: "vbus1"
- board text added: "vbus2"
- board text added: "vdc"
- board text added: "vdd"
- board text added: "vprog"

Commit message: WIP commit
Parts:
- moved SW1 75.1 mm to (93.8, 74.4), turned to -90 degrees
- moved JP5 49.3 mm to (98.2, 78.8), turned to -90 degrees
- moved J4 25.1 mm to (141.0, 92.0), turned to 0 degrees
- moved C30 24.9 mm to (141.6, 68.0), turned to 90 degrees
- moved U13 24.9 mm to (141.6, 68.0), turned to 180 degrees
- moved C57 23.8 mm to (129.9, 65.5), turned to 45 degrees
- moved JP6 23.8 mm to (123.5, 68.2), turned to 180 degrees
- moved C2 23.1 mm to (133.2, 65.7), turned to 135 degrees
- moved C38 21.6 mm to (140.7, 72.2), turned to 180 degrees
- moved Y2 21.2 mm to (131.6, 67.1), turned to 135 degrees
- moved C63 19.8 mm to (128.1, 69.0), turned to 0 degrees
- moved C64 19.3 mm to (122.8, 73.2), turned to -90 degrees
- moved C28 18.6 mm to (151.8, 107.8), turned to -90 degrees
- moved D2 18.2 mm to (147.8, 67.9), turned to -90 degrees
- moved R16 16.9 mm to (122.7, 76.3), turned to 90 degrees
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Routing:
- net /VPROG_PWM: track 41.7 -> 2.47 mm, vias 3 -> 1
- net /FE21_EEPROM_SDA: track 27.5 -> 2.73 mm
- net /PS_SDA: track 23.8 -> 3.74 mm, vias 2 -> 1
- net /PS_SCL: track 22.1 -> 3.49 mm, vias 2 -> 1
- net /FE21_EEPROM_SCL: track 17.0 -> 0.00 mm
- net /LOADSW_USB1: track 15.8 -> 1.85 mm, vias 2 -> 1
- net /STM_LED1: track 14.1 -> 2.26 mm
- net Net-(C28-Pad1): track 13.7 -> 3.81 mm
- net /ADC_CS: track 9.85 -> 0.00 mm
- net /ADC_SCK: track 9.85 -> 0.00 mm
- net /ADC_MOSI: track 9.66 -> 0.00 mm
- net /ADC_MISO: track 9.65 -> 0.00 mm
- net /STM_LED2: track 12.6 -> 3.35 mm
- net /CON_GPIO4: track 9.03 -> 0.00 mm
- net /CON_GPIO3: track 9.03 -> 0.00 mm
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Other:
- board size 100 x 77 mm -> 106.6 x 77 mm
