File: rev_1/bread-board/bread-board.kicad_pcb (KiCad board)
At the start: 4 copper layers, 106.6 x 77 mm, 232 parts, among them IC1 FE2.1, J1 Barrel_Jack_Switch, J10 Conn_01x03, J2 USB_C_Receptacle_USB2.0, J3 USB_C_Receptacle_USB2.0, J4 Conn_02x30_Top_Bottom, J5 USB2, J6 USB3, J7 USB4, J8 Screw_Terminal_01x12, J9 USB1, Q1 AO3401A, Q10 BC847, Q11 BC847, Q12 BC847, Q2 AO3401A, Q3 AO3401A, Q4 AO3401A, Q5 AO3401A, Q6 AO3401A, Q7 BC847, Q8 BC847, Q9 BC847, SW1 PCM13, SW2 BUT_SMD, SW3 BUT_SMD, SW4 PCM13, U1 STM32F103RFTx, U10 INA181, U11 ADP1612, U12 MCP6001U, U13 AZ1117-ADJ, U14 AZ1117-ADJ, U15 AZ1117-ADJ, U16 AZ1117-ADJ, U17 USBLC6-2SC6, U18 USBLC6-2SC6, U19 USBLC6-2SC6, U2 USBLC6-2SC6, U20 USBLC6-2SC6, U21 INA181, U22 INA181, U23 INA181, U24 INA181, U25 INA181, U26 INA181, U27 INA181, U28 INA181, U3 USBLC6-2SC6, U4 MIC2405x, U5 FSUSB30MUX, U6 24LC00, U7 LB66200, U8 INA181, U9 LB66200, Y1 6MHZ 2520, Y2 6MHZ 2520

Commit message: another schematic refactor smh
Changed lines of the file:
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@@
       ))
   )
-  (gr_line (start 167.12 108.02) (end 167.6 108.46) (layer "F.SilkS") (width 0.2))
-  (gr_line (start 167.6 108.46) (end 167.19 108.82) (layer "F.SilkS") (width 0.2))
-  (gr_arc (start 166.86 108.97) (mid 166.587191 108.706209) (end 166.85406 108.43641) (layer "F.SilkS") (width 0.2))
-  (gr_arc (start 167.18 108.83) (mid 167.03386 108.931681) (end 166.86 108.97) (layer "F.SilkS") (width 0.2))
-  (gr_arc (start 166.85406 108.43641) (mid 166.590822 108.170201) (end 166.86 107.91) (layer "F.SilkS") (width 0.2))
-  (gr_arc (start 166.864086 107.902837) (mid 167.004816 107.933519) (end 167.12 108.02) (layer "F.SilkS") (width 0.2))
+  (gr_line (start 167.420293 108.342599) (end 167.448577 108.993137) (layer "F.SilkS") (width 0.2))
+  (gr_line (start 167.448577 108.993137) (end 166.904105 108.957782) (layer "F.SilkS") (width 0.2))
+  (gr_arc (start 166.564693 108.830503) (mid 166.558314 108.451012) (end 166.937798 108.448998) (layer "F.SilkS") (width 0.2))
+  (gr_arc (start 166.889963 108.957782) (mid 166.714734 108.926334) (end 166.564693 108.830503) (layer "F.SilkS") (width 0.2))
+  (gr_arc (start 166.937798 108.448998) (mid 166.939867 108.074632) (end 167.314227 108.08097) (layer "F.SilkS") (width 0.2))
+  (gr_arc (start 167.322181 108.078794) (mid 167.4 108.2) (end 167.420293 108.342599) (layer "F.SilkS") (width 0.2))
   (gr_line (start 143.550001 -63.7) (end 143.550001 -32.7) (layer "Dwgs.User") (width 0.15))
   (gr_line (start 96.550001 -32.7) (end 96.55 -63.7) (layer "Dwgs.User") (width 0.15))
@@
   (gr_circle (center 189 109.05) (end 186.6 105.85) (layer "F.CrtYd") (width 0.05) (fill none))
   (gr_circle (center 179 52) (end 176.6 48.8) (layer "F.CrtYd") (width 0.05) (fill none))
-  (gr_text "vdd" (at 173.2 107.68 90) (layer "F.SilkS")
+  (gr_text "vdd" (at 174.2 107.9 45) (layer "F.SilkS")
     (effects (font (size 1.2 1.2) (thickness 0.2)))
   )
-  (gr_text "5V" (at 177.66 108.01 90) (layer "F.SilkS")
+  (gr_text "5V" (at 178.3 108.1 45) (layer "F.SilkS")
     (effects (font (size 1.2 1.2) (thickness 0.2)))
   )
-  (gr_text "vbus2" (at 181.63 106.57 90) (layer "F.SilkS")
+  (gr_text "vbus2" (at 183.215 107 45) (layer "F.SilkS")
     (effects (font (size 1.2 1.2) (thickness 0.2)))
   )
-  (gr_text "status" (at 168.89 106.38 90) (layer "F.SilkS")
+  (gr_text "status" (at 170.7 107 45) (layer "F.SilkS")
     (effects (font (size 1.2 1.2) (thickness 0.2)))
   )
-  (gr_text "debug" (at 171.05 106.42 90) (layer "F.SilkS")
+  (gr_text "debug" (at 173 107.1 45) (layer "F.SilkS")
     (effects (font (size 1.2 1.2) (thickness 0.2)))
   )
-  (gr_text "beat" (at 166.9 105.91 90) (layer "F.SilkS")
+  (gr_text "beat" (at 168.756724 106.69504 45) (layer "F.SilkS")
     (effects (font (size 1.2 1.2) (thickness 0.2)))
   )
-  (gr_text "vprog" (at 175.32 106.66 90) (layer "F.SilkS")
+  (gr_text "vprog" (at 176.7 107.2 45) (layer "F.SilkS")
     (effects (font (size 1.2 1.2) (thickness 0.2)))
   )
-  (gr_text "vbus1" (at 179.53 106.57 90) (layer "F.SilkS")
+  (gr_text "vbus1" (at 181 107 45) (layer "F.SilkS")
     (effects (font (size 1.2 1.2) (thickness 0.2)))
   )
-  (gr_text "vdc" (at 183.74 107.59 90) (layer "F.SilkS")
+  (gr_text "vdc" (at 184.6 107.9 45) (layer "F.SilkS")
     (effects (font (size 1.2 1.2) (thickness 0.2)))
   )
@@
     (connect_pads (clearance 0))
     (min_thickness 0.254)
-    (keepout (tracks allowed) (vias allowed) (pads allowed ) (copperpour allowed) (footprints allowed))
+    (keepout (tracks allowed) (vias allowed) (pads allowed) (copperpour allowed) (footprints allowed))
     (fill (thermal_gap 0.508) (thermal_bridge_width 0.508))
     (polygon
@@
     (connect_pads (clearance 0))
     (min_thickness 0.254)
-    (keepout (tracks allowed) (vias allowed) (pads allowed ) (copperpour allowed) (footprints not_allowed))
+    (keepout (tracks allowed) (vias allowed) (pads allowed) (copperpour allowed) (footprints not_allowed))
     (fill (thermal_gap 0.508) (thermal_bridge_width 0.508))
     (polygon
