File: rev_1/bread-board/bread-board.kicad_sch (KiCad schematic)
At the start: 160 parts, among them IC1 FE2.1, J1 USB_C_Receptacle_USB2.0, J2 USB_C_Receptacle_USB2.0, J3 Barrel_Jack_Switch, J4 USB2, J5 Conn_02x30_Top_Bottom, J6 USB2, J7 USB1, J8 USB2, J9 Screw_Terminal_01x12, Q1 AO3401A, SW1 SW_SP3T, U1 AZ1117-ADJ, U10 USBLC6-2SC6, U11 FSUSB30MUX, U12 AZ1117-ADJ, U13 INA181, U14 ADP1612, U15 INA181, U16 MIC2405x, U17 MCP6001U, U18 INA181, U19 INA181, U2 LB66200, U20 USBLC6-2SC6, U21 USBLC6-2SC6, U22 USBLC6-2SC6, U23 24LC00, U24 USBLC6-2SC6, U25 MCP3208, U3 LB66200, U4 USBLC6-2SC6, U5 INA181, U6 INA181, U7 AZ1117-ADJ, U8 INA181, U9 AZ1117-ADJ, Y1 6MHZ 2520

Commit message: moving to new pc
Parts:
- removed JP3: VPROG_SET_SRC, Connector_PinHeader_2.54mm:PinHeader_1x03_P2.54mm_Vertical, symbol Jumper:Jumper_3_Open
- added JP3: TEST_POT_ENA, Jumper:SolderJumper-2_P1.3mm_Open_RoundedPad1.0x1.5mm, symbol Jumper:SolderJumper_2_Open
- RV1: value 10k -> 10k/DNP; footprint Potentiometer_THT:Potentiometer_Runtron_RM-065_Vertical -> Potentiometer_SMD:Potentiometer_Bourns_TC33X_Vertical
- gave numbers to parts that had none: 1
- renumbered C11 to C10, C12 to C11, C13 to C12, C14 to C13, C15 to C14, C16 to C15, C17 to C16, C18 to C17, C19 to C18, C20 to C19, C21 to C20, C22 to C21, C23 to C22, C24 to C23, C25 to C24, C26 to C25, C27 to C26, C28 to C27, C29 to C28, C30 to C29, C31 to C30, C32 to C31, C33 to C32, C34 to C33, C35 to C34, C36 to C35, C37 to C36, C38 to C37, C39 to C38, C40 to C39, C41 to C40, C42 to C41, C43 to C42, C44 to C43, C45 to C44, C46 to C45, C47 to C46, C48 to C47, C49 to C48, C50 to C49, C6 to C5, C51 to C50, C52 to C51, C53 to C52, C54 to C53, C55 to C54, C56 to C55, C57 to C56, C58 to C57, C59 to C58, C60 to C59, C7 to C6, C61 to C60, C8 to C7, C9 to C8, C10 to C9, R34 to R32, R32 to R33, R33 to R34
Connections:
- net VPROG_PWM: now also JP3.1 (A)
- net at C41.1, R32.2: now also U17.1 (+)
- net at RV1.2: now also JP3.2 (B)
Other:
- note added: "Generic SMD pot, like VG039NCHXTB503 Better one on top board"
- note removed: "Power supply outputs"
- moved on the sheet: C41, R32, RV1

Commit message: checkpoint before yet another project structure change
Parts:
- removed C14: 10u/16V, Capacitor_SMD:C_0805_2012Metric, symbol Device:C_Small
- removed C19, C30, C6: 10u, Capacitor_SMD:C_0805_2012Metric, symbol Device:C_Small
- L1: renamed from L4; footprint Inductor_SMD:L_Vishay_IHLP-4040 -> Inductor_SMD:L_Taiyo-Yuden_NR-80xx_HandSoldering
- R36: renamed from R2; value 0.5R -> 50mR
- R37: renamed from R11; value 0.5R -> 50mR
- R38: renamed from R18; value 0.5R -> 50mR
- R39: renamed from R23; value 0.5R -> 200mR
- R40: renamed from R36; value 0.5R -> 50mR
- R41: renamed from R37; value 0.5R -> 100mR
- renumbered C40 to C1, C32 to C10, C56 to C11, C53 to C12, C43 to C13, C33 to C14, C44 to C15, C45 to C16, C34 to C17, C46 to C18, C35 to C19, C60 to C2, C36 to C20, C47 to C21, C48 to C22, C25 to C23, C49 to C24, C50 to C25, C2 to C26, C23 to C28, C20 to C29, C37 to C3, C3 to C30, C7 to C31, C10 to C32, C16 to C33, C21 to C34, C31 to C35, C22 to C36, C41 to C37, C4 to C38, C8 to C39, C26 to C4, C11 to C40, C17 to C41, C51 to C42, C54 to C43, C59 to C44, C55 to C45, C1 to C46, C9 to C47, C15 to C48, C24 to C49, C38 to C5, C39 to C50, C52 to C51, C5 to C52, C13 to C53, C18 to C54, C29 to C55, C42 to C56, C57 to C6, C12 to C7, C58 to C8, C28 to C9, D3 to D1, D1 to D2, D2 to D3, J3 to J1, J1 to J2, J2 to J3, J5 to J4, J4 to J5, J8 to J7, J9 to J8, J7 to J9, JP4 to JP1, JP1 to JP2, JP2 to JP3, JP3 to JP4, L3 to L2, L1 to L3, L2 to L4, R29 to R1, R33 to R10, R31 to R11, R35 to R12, R19 to R13, R38 to R14, R41 to R15, R4 to R16, R6 to R17, R40 to R18, R28 to R19, R30 to R2, R39 to R20, R27 to R21, R25 to R22, R22 to R23, R26 to R24, R32 to R25, R1 to R26, R5 to R27, R9 to R28, R10 to R29, R7 to R3, R12 to R30, R13 to R31, R16 to R32, R17 to R33, R20 to R34, R21 to R35, R14 to R4, R8 to R5, R15 to R6, R24 to R7, R34 to R8, R3 to R9, TP5 to TP1, TP6 to TP2, TP1 to TP3, TP2 to TP5, TP3 to TP6, U25 to U1, U6 to U10, U14 to U11, U17 to U12, U1 to U13, U7 to U14, U9 to U15, U12 to U16, U20 to U17, U21 to U18, U24 to U19, U4 to U2, U22 to U20, U5 to U21, U8 to U22, U13 to U23, U15 to U24, U18 to U25, U19 to U26, U10 to U3, U16 to U4, U11 to U5, U23 to U6, U2 to U7, U3 to U9
Connections:
- net VDC_SW: now reaches C10.1, C9.2, L1.1, U4.10 (SW), U4.11 (SW), U4.12 (SW), U4.22 (CS), U4.4 (SW), U4.9 (SW)
- net 5V_FROM_VDC: now reaches C14.1, C17.1, C19.1, C20.1, L1.2, R11.2, U9.6 (VIN2)
Other:
- note added: "INA181A2 dI_max = 0.1V R=U/I"
- note added: "Imax = 1A"
- note added: "Imax = 2A"
- note added: "Imax = 500mA"
- note added: "NRS8030T2R2NJGJ"
- note added: "SRF0703-150M SRF0703A-150M"

Commit message: adding yeast^WcubeMX project, working on pcb
Parts:
- removed JP1: GND_DOMAIN_BRG, Jumper:SolderJumper-2_P1.3mm_Bridged_Pad1.0x1.5mm, symbol Jumper:SolderJumper_2_Bridged
- removed U1: MCP3208, Package_SO:SOIC-16_3.9x9.9mm_P1.27mm, symbol Analog_ADC:MCP3208
- added C57: 20p, Capacitor_SMD:C_0402_1005Metric, symbol Device:C_Small
- added C58, C59, C60, C61, C62, C63, C64, C65, C66: 100n, Capacitor_SMD:C_0402_1005Metric, symbol Device:C_Small
- added JP1, JP5: (no value), Jumper:SolderJumper-2_P1.3mm_Open_RoundedPad1.0x1.5mm, symbol Jumper:SolderJumper_2_Open
- added Q10, Q12, Q7, Q8, Q9: BC847, Package_TO_SOT_SMD:SOT-23, symbol Transistor_BJT:BC847
- added Q11: (no value), symbol Transistor_BJT:BC847
- added Q2, Q3, Q4, Q5, Q6: AO3401A, Package_TO_SOT_SMD:SOT-23, symbol Transistor_FET:AO3401A
- added R42, R52: (no value), Resistor_SMD:R_0603_1608Metric_Pad0.98x0.95mm_HandSolder, symbol Device:R_Small
- added R43, R44, R45: 100mR, Resistor_SMD:R_1206_3216Metric_Pad1.30x1.75mm_HandSolder, symbol Device:R
- added R46, R47, R50, R51, R53: 10k, Resistor_SMD:R_0603_1608Metric_Pad0.98x0.95mm_HandSolder, symbol Device:R_Small
- added R48, R49, R54, R55, R56, R57: 3k, Resistor_SMD:R_0603_1608Metric_Pad0.98x0.95mm_HandSolder, symbol Device:R_Small
- added SW2: (no value), symbol Switch:SW_Push
- added TP7: (no value), TestPoint:TestPoint_Pad_D1.0mm, symbol Connector:TestPoint
- added U1: STM32F103RFTx, Package_QFP:LQFP-64_10x10mm_P0.5mm, symbol MCU_ST_STM32F1:STM32F103RFTx
- added U27, U28, U8: INA181, Package_TO_SOT_SMD:SOT-23-6, symbol Amplifier_Current:INA181
- added Y2: 6MHZ 2520, Crystal:Crystal_SMD_2520-4Pin_2.5x2.0mm, symbol Device:Crystal_GND24
- C13, C17, C19, C20, C21, C23, C28, C29, C3, C30, C31, C32, C33, C34, C36, C38, C39, C4, C40, C41, C42, C43, C44, C45, C5, C52, C53, C54, C55, C56: footprint Capacitor_SMD:C_0805_2012Metric -> (none)
- C2: value 100n -> 20p
- J6: value USB2 -> USB3
- J7: value USB2 -> USB4
- SW1: value SW_SP3T -> (none)
Connections:
- net +5V: now also F3.2, IC1.45 (OVCJ1), Q1.2 (S), R20.2, JP1.1 (A), Q2.2 (S), Q3.2 (S), Q4.2 (S), R46.2, R50.2, R51.2, R52.2, R53.2; no longer C42.1, C43.1, C44.1, F3.1, J5.1 (VBUS), J6.1 (VBUS), J7.1 (VBUS), R36.1, U17.5 (+), U18.5 (+), U19.5 (+), U21.3 (+)
- net +VDC: now also Q6.2 (S), R47.2; no longer R37.1, U22.3 (+)
- net 1V8_OUT_CURR: now also U1.10 (PC2)
- net 3V3_OUT_CURR: now also U1.17 (PA3)
- net 5V_CURR: now also U1.14 (PA0)
- net 5V_OUT_CURR: now also U1.16 (PA2)
- net ADC_CS: now also U1.33 (PB12)
- net ADC_MISO: now also U1.35 (PB14)
- net ADC_MOSI: now also U1.36 (PB15)
- net ADC_SCK: now also U1.34 (PB13)
- net EXT_PS_CONV_EN: now also U1.3 (PC14); no longer J4.50 (Pin_50)
- net EXT_PS_CONV_PG: now also U1.4 (PC15); no longer J4.51 (Pin_51)
- net EXT_PS_OUT_CURR: now also U1.15 (PA1)
- net EXT_PS_VLT: now also U1.8 (PC0)
- net FE21_RST: now also U1.41 (PA8); no longer J4.13 (Pin_13)
- net FT2232_DM: now also IC1.37 (DM7); no longer IC1.34 (DM6)
- net FT2232_DP: now also IC1.38 (DP7); no longer IC1.35 (DP6)
- net GND: now also C2.2, C57.2, C58.1, C59.2, C63.2, C64.1, C65.1, C66.2, Q10.2 (E), Q11.2 (E), Q12.2 (E), Q7.2 (E), Q8.2 (E), Q9.2 (E), R42.1, SW2.1, U1.12 (VSSA), U1.18 (VSS), U1.31 (VSS), U1.47 (VSS), U1.63 (VSS), Y2.2, Y2.4
- net GNDA: now also C60.2, C61.2, C62.2, U27.2 (GND), U27.5 (REF), U28.2 (GND), U28.5 (REF), U8.2 (GND), U8.5 (REF); no longer C2.2
- net PS_SCL: now also J4.46 (Pin_46), U1.58 (PB6); no longer J4.47 (Pin_47)
- net PS_SDA: now also J4.47 (Pin_47), U1.59 (PB7); no longer J4.46 (Pin_46)
- net USB1_CURR: now also U1.21 (PA5)
- net USBEXT_DM: no longer IC1.37 (DM7)
- net USBEXT_DP: no longer IC1.38 (DP7)
- net USBIN1_CC1: now also U1.25 (PC5); no longer J4.21 (Pin_21)
- net USBIN1_CC2: now also U1.24 (PC4); no longer J4.20 (Pin_20)
- net USBIN2_CC1: now also U1.20 (PA4); no longer J4.19 (Pin_19)
- net USBIN2_CC2: now also U1.27 (PB1); no longer J4.18 (Pin_18)
- net USBIN_SEL: now also JP5.2 (B), U1.43 (PA10); no longer J4.12 (Pin_12), R13.2, U5.1 (S)
- net VDD: now also C58.2, C59.1, C64.2, C65.2, U1.1 (VBAT), U1.19 (VDD), U1.32 (VDD), U1.48 (VDD), U1.64 (VDD)
- net VDDA: now also C60.1, C61.1, C62.1, C63.1, U1.13 (VDDA), U27.6 (V+), U28.6 (V+), U8.6 (V+); no longer C2.1
- net VPROG_EN: now also U1.62 (PB9); no longer J4.14 (Pin_14)
- net VPROG_OUT_CURR: now also U1.11 (PC3)
- net VPROG_PWM: now also U1.50 (PA15); no longer J4.15 (Pin_15)
- net VPROG_VLT: now also U1.9 (PC1); no longer J4.17 (Pin_17)
- net VBUSIN_COM: now reaches JP2.1 (A), JP3.2 (B), U7.2 (VOUT), U7.7 (VOUT), U9.3 (VIN1)
- net VBUSIN_1: now reaches F1.2, JP2.2 (B), U7.3 (VIN1)
- net VBUSIN_2: now reaches F2.2, U7.6 (VIN2)
- net RFU_CS: no longer names the net of J4.39 (Pin_39)
- net RFU_IO1 renamed RFU_HSIO2
- net RFU_IO2 renamed RFU_HSIO1
- net RFU_IO3 renamed CON_GPIO2
- net CON_GPIO2: now also U1.38 (PC7)
- net RFU_IO4 renamed CON_GPIO1
- net CON_GPIO1: now also U1.37 (PC6)
- net USB1_5V: no longer names the net of R41.1, U26.3 (+)
- net USB1_5V: now also Q5.3 (D); no longer Q1.3 (D)
- net USB_OC_DET: no longer names the net of R18.1, R20.1
- net USB_OC_DET: no longer J4.11 (Pin_11), Q1.1 (G)
- new net: Q1.1 (G), Q7.3 (C), R46.1
- new net: C43.1, J6.1 (VBUS), R44.2, U18.5 (+), U27.4 (-)
- new net: Q11.1 (B), R56.2
- new net: Q8.1 (B), R49.2
- new net: C42.1, J5.1 (VBUS), R43.2, U17.5 (+), U8.4 (-)
- new net: Q12.3 (C), Q4.1 (G), R53.1
- new net: Q4.3 (D), R45.1, U28.3 (+)
- new net: Q12.1 (B), R57.2
- new net: JP5.1 (A), R13.2, U5.1 (S)
- new net: Q7.1 (B), R48.2
- new net: Q10.3 (C), Q2.1 (G), R51.1
- new net: Q2.3 (D), R43.1, U8.3 (+)
- new net: C2.1, U1.5 (PD0), Y2.1
- new net: C44.1, J7.1 (VBUS), R45.2, U19.5 (+), U28.4 (-)
- new net: Q3.3 (D), R44.1, U27.3 (+)
- new net: R42.2, TP7.1, U1.60 (BOOT0)
- new net: Q1.3 (D), R36.1, U21.3 (+)
- new net: Q11.3 (C), Q3.1 (G), R52.1
- new net: Q6.1 (G), Q8.3 (C), R47.1
- new net: Q6.3 (D), R37.1, U22.3 (+)
- new net: Q9.1 (B), R54.2
- new net: C57.1, U1.6 (PD1), Y2.3
- new net: C66.1, SW2.2, U1.7 (NRST)
- new net: Q5.1 (G), Q9.3 (C), R50.1
- new net: Q10.1 (B), R55.2
- new net: F3.1, JP1.2 (B), Q5.2 (S)
- new net CON_GPIO3: J4.50 (Pin_50), U1.39 (PC8)
- new net CON_GPIO4: J4.51 (Pin_51), U1.40 (PC9)
- new net LOADSW_5V: R48.1
- new net LOADSW_USB1: R54.1, U1.51 (PC10)
- new net LOADSW_USB2: R55.1, U1.28 (PB2)
- new net LOADSW_USB3: R56.1, U1.29 (PB10)
- new net LOADSW_USB4: R57.1, U1.30 (PB11)
- new net LOADSW_VDC: R49.1
- new net STM32_DM: IC1.34 (DM6), U1.44 (PA11)
- new net STM32_DP: IC1.35 (DP6), U1.45 (PA12)
- new net SWCLK: U1.49 (PA14)
- new net SWDIO: U1.46 (PA13)
- new net UART_LOG: U1.42 (PA9)
- new net USB2_CURR: U1.22 (PA6), U8.1
- new net USB3_CURR: U1.23 (PA7), U27.1
- new net USB4_CURR: U1.26 (PB0), U28.1
- no-connect marks 12 -> 14
Other:
- note added: "From my experience, voltage on USB HUBs tends to sag a lot, in some cases to unacceptable values (like 4.6v)."
- note added: "The multiplexer can be controlled: * via ideal diode status pin * manually overriden by switch * overriden strongly by MCU output"
- note removed: "From my experience, voltage on USB HUBs tends to sag a lot, in some cases to unacceptable values (like 4.6v). The DC/DC below may supply stable 5V. This voltage may leak back into the PC's USB system via Q1's body diode, which may or may not be a bad thing, implying the DC/DC works properly. This section should be remade if this ever becomes viable product"
- moved on the sheet: C11, C12, C13, C15, C16, C18, C21, C22, C24, C25, C42, C43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

Commit message: adding some goodies to shcematic
Parts:
- removed TP5: ID2_CTRL, TestPoint:TestPoint_Pad_D1.0mm, symbol Connector:TestPoint
- added D? (x8): LED, symbol Device:LED
- added D?: (no value), symbol Device:LED
- added JP? (x2): (no value), Jumper:SolderJumper-2_P1.3mm_Open_RoundedPad1.0x1.5mm, symbol Jumper:SolderJumper_2_Open
- added JP?: X, Jumper:SolderJumper-2_P1.3mm_Open_RoundedPad1.0x1.5mm, symbol Jumper:SolderJumper_2_Open
- added R? (x9): 2k, Resistor_SMD:R_0603_1608Metric_Pad0.98x0.95mm_HandSolder, symbol Device:R_Small
- added R? (x4): (no value), Resistor_SMD:R_0603_1608Metric_Pad0.98x0.95mm_HandSolder, symbol Device:R_Small
- added SW?: (no value), Button_Switch_SMD:SW_SPST_TL3342, symbol Switch:SW_Push
- added TP?: (no value), TestPoint:TestPoint_Pad_D1.0mm, symbol Connector:TestPoint
- added TP?: RFUPAD, TestPoint:TestPoint_Pad_D1.0mm, symbol Connector:TestPoint
Connections:
- net UART_LOG is gone; now on net STM_UART_TX: U1.42 (PA9)
- net +5V: now also D?.2 (A)
- net +VDC: now also D?.2 (A)
- net +VSW: now also D?.2 (A)
- net 5V_FROM_VDC: now also SW?.2
- net EXT_PS_CONV_EN: now also J4.11 (Pin_11)
- net EXT_PS_CONV_PG: now also J4.12 (Pin_12), JP?.1 (A); no longer U1.4 (PC15)
- net GND: now also U6.7 (WP), R?.1, R?.1, R?.1, R?.1, R?.1, R?.1, R?.1, R?.1, R?.1, R?.1, R?.1, R?.1, R?.1
- net USBIN_SEL: now also U1.2 (PC13); no longer U1.43 (PA10)
- net VBUSIN_1: now also U7.6 (VIN2), D?.2 (A); no longer U7.3 (VIN1)
- net VBUSIN_2: now also U7.3 (VIN1), D?.2 (A); no longer U7.6 (VIN2)
- net VDD: now also D?.2 (A)
- net VPROG_PWM: now also J4.13 (Pin_13)
- net at R16.2, U9.4 (~{ON): now also SW?.1
- net FE21_EEPROM_SDA: now reaches U1.52 (PC11)
- net FE21_EEPROM_SDA: now also U6.5 (SDA), JP?.1 (A)
- net FE21_EEPROM_SCL: now reaches U1.53 (PC12)
- net FE21_EEPROM_SCL: now also U6.6 (SCL), JP?.1 (A)
- net at U1.54 (PD2): now also TP?.1
- net STM_LED1: now reaches U1.55 (PB3)
- net STM_LED1: now also D?.2 (A)
- net STM_LED2: now reaches U1.56 (PB4)
- net STM_LED2: now also D?.2 (A)
- net STM_LED3: now reaches U1.57 (PB5)
- net STM_LED3: now also D?.2 (A)
- net at U1.61 (PB8): now also TP?.1
- net STM_UART_TX: now reaches J4.14 (Pin_14)
- net STM_UART_RX: now reaches J4.15 (Pin_15)
- net STM_UART_RX: now also U1.43 (PA10)
- net at IC1.2 (TESTJ): now also JP?.2 (B); no longer U6.5 (SDA)
- net at IC1.3 (LED1): now also JP?.2 (B); no longer U6.6 (SCL)
- new net: D?.1 (K), R?.2, R?.2 (x4)
- new net: D?.1 (K), R?.2 (x5)
- new net: JP?.2 (B), U1.4 (PC15)
- no-connect marks 14 -> 13
Other:
- note added: "HSD1* when S=LOW"
- note added: "LOW when powered from VBUSIN_1 (VIN2 pin)"
- note added: "Lines crossed for compatibility with FSUSB30MUX"
- note removed: "Connect with PG?"
- note removed: "FSUSB30"
- moved on the sheet: C11, C2, C57, C58, C59, C6, C63, C64, C65, C66, C8, J4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

Commit message: routing AAAAAAAAAAAAAAA
Parts:
- added J10: Conn_01x03, Connector_PinHeader_2.54mm:PinHeader_1x03_P2.54mm_Vertical, symbol Connector_Generic:Conn_01x03
- added R71: 3k, Resistor_SMD:R_0603_1608Metric_Pad0.98x0.95mm_HandSolder, symbol Device:R_Small
- added R72, R73: 100k, Resistor_SMD:R_0603_1608Metric_Pad0.98x0.95mm_HandSolder, symbol Device:R_Small
- added SW4: PCM13, Button_Switch_SMD:SW_SP3T_PCM13, symbol Switch:SW_SP3T
- C13, C17, C19, C20, C21, C23, C28, C29, C3, C30, C31, C32, C33, C34, C36, C38, C39, C4, C40, C41, C42, C43, C44, C45, C5, C52, C53, C54, C55, C56: footprint (none) -> Capacitor_SMD:C_0603_1608Metric
- D10, D11, D12, D5, D6, D7, D8, D9: renamed from D?; footprint (none) -> LED_SMD:LED_0603_1608Metric
- D4: renamed from D?; value (none) -> LED; footprint (none) -> LED_SMD:LED_0603_1608Metric
- JP1: value (none) -> FUSE_BYP
- JP5: value (none) -> MCU_USB_MUX_ENA
- JP7, JP8: renamed from JP?; value (none) -> X
- Q11: value (none) -> BC847; footprint (none) -> Package_TO_SOT_SMD:SOT-23
- R42, R52: value (none) -> 10k
- R59: renamed from R?; value (none) -> 3k
- R62, R64, R67: renamed from R?; value (none) -> 2k
- SW1: value (none) -> PCM13
- SW2: value (none) -> BUT_SMD; footprint (none) -> Button_Switch_SMD:SW_SPST_TL3342
- SW3: renamed from SW?; value (none) -> BUT_SMD
- TP5: renamed from TP?; value (none) -> RFUPAD
- TP7: value (none) -> STM_BOOT0
- gave numbers to parts that had none: 11
Connections:
- net +5V: now also R67.2; no longer D10.2 (A)
- net +VDC: now also R59.2; no longer D4.2 (A)
- net +VSW: now also R69.2; no longer D11.2 (A)
- net ADC_MOSI: now also J4.44 (Pin_44); no longer J4.41 (Pin_41)
- net ADC_SCK: now also J4.41 (Pin_41); no longer J4.44 (Pin_44)
- net CON_GPIO1: now also R72.1, SW4.1
- net CON_GPIO2: now also R73.1, SW4.2
- net GND: now also D10.1 (K), D11.1 (K), D12.1 (K), D4.1 (K), D5.1 (K), D6.1 (K), D7.1 (K), D8.1 (K), D9.1 (K), J10.3 (Pin_3), R71.1; no longer R58.1, R59.1, R60.1, R61.1, R62.1, R63.1, R64.1, R65.1, R66.1, R67.1, R68.1, R69.1, R70.1
- net STM_LED1: now also R61.2, R63.2; no longer D7.2 (A)
- net STM_LED2: now also R65.2, R66.2; no longer D9.2 (A)
- net STM_LED3: now also R68.2, R70.2; no longer D12.2 (A)
- net SWCLK: now also J4.21 (Pin_21), J10.2 (Pin_2)
- net SWDIO: now also J4.20 (Pin_20), J10.1 (Pin_1)
- net VBUSIN_1: now also R62.2; no longer D6.2 (A)
- net VBUSIN_2: now also R64.2; no longer D8.2 (A)
- net VDD: now also R58.2, R60.2, R72.2, R73.2; no longer D5.2 (A)
- new net: D5.2 (A), R58.1, R60.1
- new net: D6.2 (A), R62.1
- new net: D12.2 (A), R68.1, R70.1
- new net: D10.2 (A), R67.1
- new net: R71.2, SW4.3
- new net: D7.2 (A), R61.1, R63.1
- new net: D8.2 (A), R64.1
- new net: D4.2 (A), R59.1
- new net: D11.2 (A), R69.1
- new net: D9.2 (A), R65.1, R66.1
- no-connect marks 13 -> 14
Other:
- moved on the sheet: C2, C57, D10, D11, D12, D4, D5, D6, D7, D8, D9, J4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

Commit message: another schematic refactor smh
Parts:
- removed C1: C, Capacitor_SMD:C_1210_3225Metric, symbol Device:C
- removed C10, C14, C26, C27, C35, C37, C7, C9: 100n, Capacitor_SMD:C_0402_1005Metric, symbol Device:C_Small
- removed C17, C23, C29, C3, C30, C31, C32, C33, C34, C38, C39, C4, C40, C41, C5: 10u, Capacitor_SMD:C_0603_1608Metric, symbol Device:C_Small
- removed C19, C20: 22u, Capacitor_SMD:C_0603_1608Metric, symbol Device:C_Small
- removed C28: 2.2u, Capacitor_SMD:C_0603_1608Metric, symbol Device:C_Small
- removed C36: 47u, Capacitor_SMD:C_0603_1608Metric, symbol Device:C_Small
- removed D1, D2, D3: D_Schottky, Diode_SMD:D_SMA, symbol Device:D_Schottky
- removed F1, F2: 1A, Resistor_SMD:R_1210_3225Metric_Pad1.30x2.65mm_HandSolder, symbol Device:Polyfuse
- removed J1: Barrel_Jack_Switch, Connector_BarrelJack:BarrelJack_CUI_PJ-102AH_Horizontal, symbol Connector:Barrel_Jack_Switch
- removed J2, J3: USB_C_Receptacle_USB2.0, Connector_USB:USB_C_Receptacle_GCT_USB4085, symbol Connector:USB_C_Receptacle_USB2.0
- removed JP2: USB1_PWR_BYP, Jumper:SolderJumper-2_P1.3mm_Open_RoundedPad1.0x1.5mm, symbol Jumper:SolderJumper_2_Open
- removed JP3: 5V_BYP, Jumper:SolderJumper-2_P1.3mm_Open_RoundedPad1.0x1.5mm, symbol Jumper:SolderJumper_2_Open
- removed JP4: TEST_POT_ENA, Jumper:SolderJumper-2_P1.3mm_Open_RoundedPad1.0x1.5mm, symbol Jumper:SolderJumper_2_Open
- removed JP5: MCU_USB_MUX_ENA, Jumper:SolderJumper-2_P1.3mm_Open_RoundedPad1.0x1.5mm, symbol Jumper:SolderJumper_2_Open
- removed L1: 2.2u, Inductor_SMD:L_Taiyo-Yuden_NR-80xx_HandSoldering, symbol Device:L
- removed L2: L_Iron_Coupled, Inductor_SMD:L_Wuerth_WE-DD-Typ-M-Typ-S, symbol Device:L_Iron_Coupled
- removed L3: L_Ferrite, Inductor_SMD:L_0805_2012Metric, symbol Device:L_Ferrite
- removed L4: L_Iron, Inductor_SMD:L_1206_3216Metric_Pad1.42x1.75mm_HandSolder, symbol Device:L_Iron
- removed R1: 470k, Resistor_SMD:R_0603_1608Metric_Pad0.98x0.95mm_HandSolder, symbol Device:R_Small
- removed R10, R11, R12, R16, R19, R2, R21, R26, R27, R28, R29, R30, R31, R32, R33, R34, R35, R7, R8, R9: 100k, Resistor_SMD:R_0603_1608Metric_Pad0.98x0.95mm_HandSolder, symbol Device:R_Small
- removed R13: 10k, Resistor_SMD:R_0603_1608Metric_Pad0.98x0.95mm_HandSolder, symbol Device:R_Small
- removed R17: 0.5R, Resistor_SMD:R_1206_3216Metric_Pad1.30x1.75mm_HandSolder, symbol Device:R
- removed R22, R24, R58, R61, R63, R65, R66, R68, R70: 2k, Resistor_SMD:R_0603_1608Metric_Pad0.98x0.95mm_HandSolder, symbol Device:R_Small
- removed R23, R25: 3k, Resistor_SMD:R_0603_1608Metric_Pad0.98x0.95mm_HandSolder, symbol Device:R_Small
- removed R3, R4, R5, R6: 5.1k, Resistor_SMD:R_0603_1608Metric_Pad0.98x0.95mm_HandSolder, symbol Device:R_Small
- removed RV1: 10k/DNP, Potentiometer_SMD:Potentiometer_Bourns_TC33X_Vertical, symbol Device:R_Potentiometer
- removed SW1: PCM13, Button_Switch_SMD:SW_SP3T_PCM13, symbol Switch:SW_SP3T
- removed SW3: BUT_SMD, Button_Switch_SMD:SW_SPST_TL3342, symbol Switch:SW_Push
- removed TP1, TP2: TestPoint, TestPoint:TestPoint_Pad_D1.0mm, symbol Connector:TestPoint
- removed TP3: ID1_CTRL, TestPoint:TestPoint_Pad_D1.0mm, symbol Connector:TestPoint
- removed TP4: ID1_STATE, TestPoint:TestPoint_Pad_D1.0mm, symbol Connector:TestPoint
- removed TP6: ID2_STATE, TestPoint:TestPoint_Pad_D1.0mm, symbol Connector:TestPoint
- removed TP8: RFUPAD, TestPoint:TestPoint_Pad_D1.0mm, symbol Connector:TestPoint
- removed U10: INA181, Package_TO_SOT_SMD:SOT-23-6, symbol Amplifier_Current:INA181
- removed U11: ADP1612, Package_SO:MSOP-8_3x3mm_P0.65mm, symbol Critbit_lib:ADP1612
- removed U12: MCP6001U, Package_TO_SOT_SMD:SOT-23-5, symbol Amplifier_Operational:MCP6001U
- removed U13, U14, U15, U16: AZ1117-ADJ, Package_TO_SOT_SMD:SOT-223-3_TabPin2, symbol Regulator_Linear:AZ1117-ADJ
- removed U2, U3: USBLC6-2SC6, Package_TO_SOT_SMD:SOT-23-6, symbol Critbit_lib:USBLC6-2SC6
- removed U4: MIC2405x, Critbit_lib:QFN-28-3EP_5x6mm_MIC2045x, symbol Critbit_lib:MIC2405x
- removed U5: FSUSB30MUX, Package_SO:MSOP-10_3x3mm_P0.5mm, symbol Critbit_lib:FSUSB30MUX
- removed U7, U9: LB66200, Critbit_lib:SOT-5x3-8, symbol Critbit_lib:LB66200
- added R?: R, Resistor_SMD:R_0603_1608Metric_Pad1.05x0.95mm_HandSolder, symbol Device:R
- added R? (x3): 1k, Resistor_SMD:R_0603_1608Metric_Pad0.98x0.95mm_HandSolder, symbol Device:R_Small
- added SW?: PCM13, Button_Switch_SMD:SW_SP3T_PCM13, symbol Switch:SW_SP3T
- R60: value 2k -> 1k
Connections:
- net +3V3: now also R?.2
- net GND: now also U21.2 (GND), U21.5 (REF), U22.2 (GND), U22.5 (REF), U23.2 (GND), U23.5 (REF), U24.2 (GND), U24.5 (REF), U25.2 (GND), U25.5 (REF), SW?.4
- net GNDA: no longer U21.2 (GND), U21.5 (REF), U22.2 (GND), U22.5 (REF), U23.2 (GND), U23.5 (REF), U24.2 (GND), U24.5 (REF), U25.2 (GND), U25.5 (REF)
- net STM_LED1: now also R?.2
- net STM_LED2: now also R?.2
- net STM_LED3: now also R?.2
- net VDD: now also SW?.1
- net at D12.2 (A): now also R?.1
- net at D7.2 (A): now also R?.1
- net EXT_5V_ENA: now reaches U1.61 (PB8)
- net at C66.1, SW2.2, U1.7 (NRST): now also R?.1
- net at D9.2 (A): now also R?.1
- new net Input ports and power supplies/USBINx_SEL: SW?.3
- no-connect marks 14 -> 10
Other:
- added sheet Input ports and power supplies (power-supplies.kicad_sch)
- note added: "Manual USB source override"
- note removed: "1.8V output expected to be low current - no step-down needed"
- note removed: "3.3V internal"
- note removed: "3.3V output To be upgraded to step-down when silicon shortage is dealt with"
- note removed: "4.8V - STM 0V 2V - STM 1.9V 0V - STM 1.6V https://tinyurl.com/y2o7nnj4"
- note removed: "From my experience, voltage on USB HUBs tends to sag a lot, in some cases to unacceptable values (like 4.6v)."
- note removed: "Generic SMD pot, like VG039NCHXTB503 Better one on top board"
- note removed: "HSD1* when S=LOW"
- note removed: "LOW when powered from VBUSIN_1 (VIN2 pin)"
- note removed: "Lines crossed for compatibility with FSUSB30MUX"
- note removed: "NRS8030T2R2NJGJ"
- note removed: "PSU section"
- note removed: "Relatively small resistance helps mitigating ripple"
- note removed: "SRF0703-150M SRF0703A-150M"
- note removed: "The multiplexer can be controlled: * via ideal diode status pin * manually overriden by switch * overriden strongly by MCU output"
- note removed: "This signal will probably be useless as we already sample VBUS"
- note removed: "there's already large cap at VSW output"
- moved on the sheet: C11, C12, C13, C15, C16, C18, C21, C22, C24, C25, C42, C43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
