File: rev_1/bread-board/bread-board.kicad_sch (KiCad schematic)
At the start: 133 parts, among them IC1 FE2.1, J10 Conn_01x03, J4 Conn_02x30_Top_Bottom, J5 USB2, J6 USB3, J7 USB4, J8 Screw_Terminal_01x12, J9 USB1, Q1 AO3401A, Q10 BC847, Q11 BC847, Q12 BC847, Q2 AO3401A, Q3 AO3401A, Q4 AO3401A, Q5 AO3401A, Q6 AO3401A, Q7 BC847, Q8 BC847, Q9 BC847, SW2 BUT_SMD, SW4 PCM13, U1 STM32F103RFTx, U17 USBLC6-2SC6, U18 USBLC6-2SC6, U19 USBLC6-2SC6, U20 USBLC6-2SC6, U21 INA181, U22 INA181, U23 INA181, U24 INA181, U25 INA181, U26 INA181, U27 INA181, U28 INA181, U6 24LC00, U8 INA181, Y1 6MHZ 2520, Y2 6MHZ 2520

Commit message: more schematic refactor, minor STM gpio changes
Parts:
- removed C42, C43, C44, C45, C52, C54, C55, C56: 10u, Capacitor_SMD:C_0603_1608Metric, symbol Device:C_Small
- removed C46, C47, C48, C49, C50, C51, C60, C61, C62: 100n, Capacitor_SMD:C_0402_1005Metric, symbol Device:C_Small
- removed C53: 10u/16V, Capacitor_SMD:C_0603_1608Metric, symbol Device:C_Small
- removed F3: 1A, Resistor_SMD:R_1210_3225Metric_Pad1.30x2.65mm_HandSolder, symbol Device:Polyfuse
- removed J5: USB2, Connector_USB:USB_A_Molex_67643_Horizontal, symbol Connector:USB_A
- removed J6: USB3, Connector_USB:USB_A_Molex_67643_Horizontal, symbol Connector:USB_A
- removed J7: USB4, Connector_USB:USB_A_Molex_67643_Horizontal, symbol Connector:USB_A
- removed J8: Screw_Terminal_01x12, TerminalBlock_Phoenix:TerminalBlock_Phoenix_PT-1,5-12-5.0-H_1x12_P5.00mm_Horizontal, symbol Connector:Screw_Terminal_01x12
- removed J9: USB1, Connector_USB:USB_A_Molex_67643_Horizontal, symbol Connector:USB_A
- removed JP1: FUSE_BYP, Jumper:SolderJumper-2_P1.3mm_Open_RoundedPad1.0x1.5mm, symbol Jumper:SolderJumper_2_Open
- removed Q1, Q2, Q3, Q4, Q5, Q6: AO3401A, Package_TO_SOT_SMD:SOT-23, symbol Transistor_FET:AO3401A
- removed Q10, Q11, Q12, Q7, Q8, Q9: BC847, Package_TO_SOT_SMD:SOT-23, symbol Transistor_BJT:BC847
- removed R36, R37, R38, R40: 50mR, Resistor_SMD:R_1206_3216Metric_Pad1.30x1.75mm_HandSolder, symbol Device:R
- removed R39: 200mR, Resistor_SMD:R_1206_3216Metric_Pad1.30x1.75mm_HandSolder, symbol Device:R
- removed R41, R43, R44, R45: 100mR, Resistor_SMD:R_1206_3216Metric_Pad1.30x1.75mm_HandSolder, symbol Device:R
- removed R46, R47, R50, R51, R52, R53: 10k, Resistor_SMD:R_0603_1608Metric_Pad0.98x0.95mm_HandSolder, symbol Device:R_Small
- removed R48, R49, R54, R55, R56, R57: 3k, Resistor_SMD:R_0603_1608Metric_Pad0.98x0.95mm_HandSolder, symbol Device:R_Small
- removed R?: R, Resistor_SMD:R_0603_1608Metric_Pad1.05x0.95mm_HandSolder, symbol Device:R
- removed U17, U18, U19, U20: USBLC6-2SC6, Package_TO_SOT_SMD:SOT-23-6, symbol Critbit_lib:USBLC6-2SC6
- removed U21, U22, U23, U24, U25, U26, U27, U28, U8: INA181, Package_TO_SOT_SMD:SOT-23-6, symbol Amplifier_Current:INA181
- added R?: 100k, Resistor_SMD:R_0603_1608Metric_Pad0.98x0.95mm_HandSolder, symbol Device:R_Small
- U102: renamed from U6; value 24LC00 -> 24LC00/DNP
- gave numbers to parts that had none: 4
- renumbered C64 to C101, C65 to C102, C58 to C103, C59 to C104, C63 to C105, C66 to C106, C2 to C107, C57 to C108, C13 to C109, C15 to C110, C16 to C111, C18 to C112, C21 to C113, C22 to C114, C24 to C115, C25 to C116, C12 to C117, C6 to C118, C8 to C119, C11 to C120, D6 to D101, D8 to D102, D10 to D103, D11 to D104, D4 to D105, D5 to D106, D7 to D107, D9 to D108, D12 to D109, IC1 to IC101, J10 to J101, J4 to J102, JP6 to JP101, JP7 to JP102, JP8 to JP103, R42 to R102, R72 to R103, R73 to R104, R14 to R105, R71 to R106, R20 to R107, R18 to R108, R59 to R109, R62 to R110, R64 to R111, R67 to R112, R69 to R113, R60 to R114, R15 to R118, SW2 to SW102, SW4 to SW103, TP7 to TP101, TP5 to TP102, U1 to U101, Y2 to Y101, Y1 to Y102
Connections:
- net VBUS is gone; now on net +5V: IC101.41 (VBUSM)
- net VDD: now also R?.2
- net at C106.1, SW102.2, U101.7 (NRST): now also R?.1
- net FE21_EEPROM_SCL: no longer names the net of JP103.1 (A), U102.6 (SCL)
- net FE21_EEPROM_SCL: no longer U101.53 (PC12)
- net FE21_EEPROM_SDA: no longer names the net of JP102.1 (A), U102.5 (SDA)
- net FE21_EEPROM_SDA: no longer U101.52 (PC11)
- new net LOADSW_5V_OUT: U101.53 (PC12)
- new net LOADSW_VDC_OUT: U101.52 (PC11)
Other:
- added sheet Output ports (output.kicad_sch)
- note removed: "INA181A2 dI_max = 0.1V R=U/I"
- note removed: "Imax = 1A"
- note removed: "Imax = 2A"
- note removed: "Imax = 500mA"
- note removed: "USB outputs"
- moved on the sheet: C101, C102, C103, C104, C105, C106, C107, C108, C109, C110, C111, C112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
