File: rev_1/bread-board/power-supplies.kicad_sch (KiCad schematic)
At the start: 101 parts

Commit message: more schematic refactor, minor STM gpio changes
Parts:
- added C?: 470uF, symbol Device:C_Polarized_Small
- added D?: D_Schottky, Diode_SMD:D_SMA, symbol Device:D_Schottky
- added R?: 100, Resistor_SMD:R_0603_1608Metric_Pad0.98x0.95mm_HandSolder, symbol Device:R_Small
- gave numbers to parts that had none: 101
Connections:
- net GND: now also C?.2
- net at C205.1, D201.1 (K), D202.1 (K)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: now also D?.1 (K), R?.2
- new net: C?.1, D?.2 (A), R?.1
Other:
- note added: "Backup power in case of 5V rail shortcircuit"
- moved on the sheet: C205, C206, C209, C210, L201, R216, R218, R220, R222, U207, U209
